File: Projects/Voicemeeter/test.sch (KiCad schematic (older format))
At the start: 0 parts

Commit message: boop
Changed lines of the file:
@@
 $Descr A4 11693 8268
 encoding utf-8
-Sheet 1 7
+Sheet 1 6
 Title ""
 Date "2018-04-28"
@@
 Wire Bus Line
 	7750 3100 8100 3100
-$Sheet
-S 4000 1550 1450 750
-U 5AFAE980
-F0 "PSU" 60
-F1 "file5AFAE97F.sch" 60
-$EndSheet
 $EndSCHEMATC
