File: Projects/Voicemeeter/_saved_file5AF36D43.sch (KiCad schematic (older format))
At the start: 0 parts

Commit message: taking a break
Parts:
- added OLED?: 1.5\"OLED, symbol 1.5"OLED
Connections:
- new net +5V: OLED?.10 (+~)
- new net GND: OLED?.11 (GND~)
- new net OLED1: OLED?.2 (CL~)
- new net OLED2: OLED?.7 (SO~)
- new net OLED3: OLED?.1 (SI)
- new net OLED4: OLED?.3 (DC~)
- new net OLED5: OLED?.4 (R~)
- new net OLED6: OLED?.5 (OC~)
- new net OLED7: OLED?.6 (SC~)
- no-connect marks 0 -> 1
Changed lines of the file:
@@
 $Descr A4 11693 8268
 encoding utf-8
-Sheet 1 6
+Sheet 7 7
 Title ""
-Date "2018-04-28"
+Date ""
 Rev ""
 Comp ""
@@
 Comment4 ""
 $EndDescr
-$Sheet
-S 2000 2750 1000 1050
-U 5AE49271
-F0 "Pot" 60
-F1 "file5AE49270.sch" 60
-F2 "HD[11..38]" O R 3000 2850 60
-F3 "DD[11..28]" O R 3000 2950 60
-F4 "OD[11..53]" O R 3000 3050 60
-F5 "OA[1..5]" O R 3000 3150 60
-F6 "DA[11..24]" O R 3000 3250 60
-F7 "HA[11..33]" O R 3000 3350 60
-$EndSheet
-$Sheet
-S 4000 3750 1000 400
-U 5AE5FE22
-F0 "Capacitors" 60
-F1 "file5AE5FE21.sch" 60
-F2 "HA[11..33]" B L 4000 4050 60
-F3 "DA[11..24]" B L 4000 3950 60
-F4 "OA[1..5]" B L 4000 3850 60
-$EndSheet
-$Sheet
-S 4000 2750 1450 700
-U 5AF6330D
-F0 "Mux" 60
-F1 "file5AF6330C.sch" 60
-F2 "HA[11..33]" I L 4000 3350 60
-F3 "OA[1..5]" I L 4000 3150 60
-F4 "DA[11..24]" I L 4000 3250 60
-F5 "M[1..27]" O R 5450 2950 60
-F6 "HD[11..38]" I L 4000 2850 60
-F7 "DD[11..28]" I L 4000 2950 60
-F8 "OD[11..53]" I L 4000 3050 60
-$EndSheet
+Text HLabel 6350 2500 2    60   Input ~ 0
+OLED[1..7]
+$Comp
+L 1.5"OLED OLED?
+U 1 1 5AF3742D
+P 4700 3400
+F 0 "OLED?" H 4700 3250 60  0000 C CNN
+F 1 "1.5\"OLED" H 4700 3550 60  0000 C CNN
+F 2 "" H 4700 3400 60  0001 C CNN
+F 3 "" H 4700 3400 60  0001 C CNN
+	1    4700 3400
+	0    1    1    0
+$EndComp
+Entry Wire Line
+	6050 2900 6150 2800
+Entry Wire Line
+	6050 3000 6150 2900
+Entry Wire Line
+	6050 3100 6150 3000
+Entry Wire Line
+	6050 3200 6150 3100
+Entry Wire Line
+	6050 3300 6150 3200
+Entry Wire Line
+	6050 3400 6150 3300
+Entry Wire Line
+	6050 3500 6150 3400
+Entry Wire Line
+	6050 3600 6150 3500
 Wire Bus Line
-	4000 4050 3100 4050
+	6150 2500 6350 2500
+Wire Wire Line
+	5450 2900 6050 2900
+Wire Wire Line
+	5450 3000 6050 3000
+Wire Wire Line
+	5450 3100 6050 3100
+Wire Wire Line
+	5450 3200 6050 3200
+Wire Wire Line
+	5450 3300 6050 3300
+Wire Wire Line
+	5450 3400 6050 3400
+Wire Wire Line
+	5450 3500 6050 3500
+Wire Wire Line
+	5450 3600 6050 3600
+Text Label 5800 3000 2    60   ~ 0
+OLED1
+Text Label 5800 3500 2    60   ~ 0
+OLED2
+Text Label 5800 2900 2    60   ~ 0
+OLED3
+Text Label 5800 3100 2    60   ~ 0
+OLED4
+Text Label 5800 3200 2    60   ~ 0
+OLED5
+Text Label 5800 3300 2    60   ~ 0
+OLED6
+Text Label 5800 3400 2    60   ~ 0
+OLED7
 Wire Bus Line
-	3100 4050 3100 3350
-Wire Bus Line
-	3000 3350 4000 3350
-Wire Bus Line
-	3000 3250 4000 3250
-Wire Bus Line
-	3200 3250 3200 3950
-Wire Bus Line
-	3200 3950 4000 3950
-Wire Bus Line
-	4000 3850 3300 3850
-Wire Bus Line
-	3300 3850 3300 3150
-Wire Bus Line
-	3000 3150 4000 3150
-Wire Bus Line
-	4000 3050 3000 3050
-Wire Bus Line
-	3000 2850 4000 2850
-Wire Bus Line
-	3000 2950 4000 2950
-$Sheet
-S 6250 2750 1500 700
-U 5AE700A5
-F0 "STM" 60
-F1 "file5AE700A4.sch" 60
-F2 "M[1..27]" I L 6250 2950 60
-F3 "SK[1..2]" O R 7750 3100 60
-$EndSheet
-Connection ~ 3300 3150
-Connection ~ 3200 3250
-Connection ~ 3100 3350
-Wire Bus Line
-	5450 2950 6250 2950
-$Sheet
-S 8100 2900 1050 450
-U 5AE7739C
-F0 "LEDs" 60
-F1 "file5AE7739B.sch" 60
-F2 "SK[1..2]" I L 8100 3100 60
-$EndSheet
-Wire Bus Line
-	7750 3100 8100 3100
+	6150 3500 6150 2500
+NoConn ~ 5450 3700
+$Comp
+L GND #PWR?
+U 1 1 5AF383EF
+P 5450 3900
+F 0 "#PWR?" H 5450 3650 50  0001 C CNN
+F 1 "GND" H 5450 3750 50  0000 C CNN
+F 2 "" H 5450 3900 50  0001 C CNN
+F 3 "" H 5450 3900 50  0001 C CNN
+	1    5450 3900
+	1    0    0    -1
+$EndComp
+$Comp
+L +5V #PWR?
+U 1 1 5AF38417
+P 5450 3800
+F 0 "#PWR?" H 5450 3650 50  0001 C CNN
+F 1 "+5V" V 5450 4000 50  0000 C CNN
+F 2 "" H 5450 3800 50  0001 C CNN
+F 3 "" H 5450 3800 50  0001 C CNN
+	1    5450 3800
+	0    1    1    0
+$EndComp
 $EndSCHEMATC
