File: Projects/Voicemeeter/_saved_file5AE700A4.sch (KiCad schematic (older format))
At the start: 36 parts, among them J1 SPARE, J2 Screw_Terminal_01x02, J3 MIDI OUT, J4 MIDI IN, J5 DIN-5_180degree, J6 DIN-5_180degree, SW56 Rotary_Encoder_Switch, U11 stm32f103-china-MS, U12 PC817

Commit message: stuff
Parts:
- added J?: GS2, Connectors:GS2, symbol GS2
Connections:
- wire segments 128 -> 114
Changed lines of the file:
@@
 $EndComp
 Wire Wire Line
-	7000 2100 7050 2100
-Wire Wire Line
-	7050 2100 7450 2100
+	7000 2100 7450 2100
 Wire Wire Line
 	7000 2500 7450 2500
@@
 	9550 3750 9750 3750
 Wire Wire Line
-	9200 4850 9500 4850
-Wire Wire Line
-	9500 4850 9800 4850
+	9200 4850 9800 4850
 Wire Wire Line
 	9200 4650 9200 4550
 Wire Wire Line
-	9200 4550 9500 4550
-Wire Wire Line
-	9500 4550 9800 4550
-Wire Wire Line
-	8600 4450 8600 4500
-Wire Wire Line
-	8600 4500 8600 4650
+	9200 4550 9800 4550
+Wire Wire Line
+	8600 4450 8600 4650
 Wire Wire Line
 	7000 4500 8600 4500
@@
 	8000 4100 7350 4100
 Wire Bus Line
-	8100 3700 8100 3800
-Wire Bus Line
-	8100 3800 8100 4000
-Wire Bus Line
-	8100 4000 8100 4200
+	8100 3700 8100 4200
 Wire Bus Line
 	8100 3700 8250 3700
 Wire Bus Line
-	3000 1700 3000 2000
-Wire Bus Line
-	3000 2000 3000 2800
-Wire Bus Line
-	3000 2800 3000 3000
-Wire Bus Line
-	3000 3000 3000 3200
-Wire Bus Line
-	3000 3200 3000 3400
-Wire Bus Line
-	3000 3400 3000 3600
-Wire Bus Line
-	3000 3600 3000 3800
+	3000 1700 3000 3800
 Wire Bus Line
 	3000 1700 2850 1700
 Wire Wire Line
-	2500 5500 3250 5500
-Wire Wire Line
-	3250 5500 3650 5500
-Wire Wire Line
-	3650 5500 3800 5500
-Wire Wire Line
-	3650 5500 4000 5500
-Wire Wire Line
-	4000 5500 4600 5500
+	2500 5500 3800 5500
+Wire Wire Line
+	3650 5500 4600 5500
 Wire Wire Line
 	4600 3900 3400 3900
@@
 	3300 4000 3200 4000
 Wire Wire Line
-	3600 5800 4000 5800
-Wire Wire Line
-	4000 5800 4150 5800
+	3600 5800 4150 5800
 Wire Wire Line
 	4150 5800 4150 5700
@@
 	4150 5200 4150 5300
 Wire Wire Line
-	3600 5200 4000 5200
-Wire Wire Line
-	4000 5200 4150 5200
-Wire Wire Line
-	3600 5400 3600 5200
-Wire Wire Line
-	3600 5200 3600 5150
+	3600 5200 4150 5200
+Wire Wire Line
+	3600 5400 3600 5150
 Connection ~ 4000 5200
 Wire Wire Line
-	3600 5600 3600 5800
-Wire Wire Line
-	3600 5800 3600 5850
+	3600 5600 3600 5850
 Connection ~ 4000 5800
 Connection ~ 4000 5500
@@
 Connection ~ 3600 5200
 Wire Wire Line
-	2600 5400 3150 5400
-Wire Wire Line
-	3150 5400 3600 5400
+	2600 5400 3600 5400
 Wire Wire Line
 	3150 5400 3150 5250
@@
 	3700 4500 4600 4500
 Wire Bus Line
-	3900 1500 3900 2000
-Wire Bus Line
-	3900 2000 3900 2200
-Wire Bus Line
-	3900 2200 3900 2400
-Wire Bus Line
-	3900 2400 3900 5000
+	3900 1500 3900 5000
 Wire Wire Line
 	4000 2500 4600 2500
@@
 	2200 5050 2600 5050
 Wire Bus Line
-	1600 3800 1600 4350
-Wire Bus Line
-	1600 4350 1600 4500
-Wire Bus Line
-	1600 4500 1600 4650
+	1600 3800 1600 4650
 Wire Bus Line
 	1600 4500 1600 4350
@@
 	4000 5100 4600 5100
 Wire Bus Line
-	7800 1500 7800 2600
-Wire Bus Line
-	7800 2600 7800 2800
-Wire Bus Line
-	7800 2800 7800 3000
+	7800 1500 7800 3000
 Wire Bus Line
 	2650 1500 7800 1500
 Wire Bus Line
-	7550 3200 7550 3400
+	7550 3200 7550 4600
 Wire Wire Line
 	7000 4700 7450 4700
@@
 	2400 5450 2200 5450
 Wire Bus Line
-	8000 900  8000 1600
-Wire Bus Line
-	8000 1600 8000 2200
-Wire Bus Line
-	8000 2200 8000 3200
+	8000 900  8000 3200
 Wire Wire Line
 	9400 2300 9400 2100
@@
 	8750 2100 9200 2100
 Wire Wire Line
-	8750 1500 8950 1500
-Wire Wire Line
-	8950 1500 9200 1500
+	8750 1500 9200 1500
 Wire Wire Line
 	9400 800  9400 1500
 Wire Wire Line
-	8750 800  8950 800
-Wire Wire Line
-	8950 800  9400 800
+	8750 800  9400 800
 Wire Wire Line
 	9100 1150 8950 1150
 Wire Wire Line
-	8950 1100 8950 1150
-Wire Wire Line
-	8950 1150 8950 1200
+	8950 1100 8950 1200
 Connection ~ 8950 1150
 Wire Bus Line
-	7550 3200 7550 3400
-Wire Bus Line
-	7550 3200 7550 3600
-Wire Bus Line
 	8000 3200 7550 3200
-Wire Bus Line
-	7550 3600 7550 3600
-Wire Bus Line
-	7550 3600 7550 4600
 $Comp
 L 1.5"OLED OLED1
@@
 NoConn ~ 1950 1550
 Wire Bus Line
-	2650 750  2650 850
-Wire Bus Line
-	2650 850  2650 950
-Wire Bus Line
-	2650 950  2650 1050
-Wire Bus Line
-	2650 1050 2650 1150
-Wire Bus Line
-	2650 1150 2650 1250
-Wire Bus Line
-	2650 1250 2650 1350
-Wire Bus Line
-	2650 1350 2650 1500
+	2650 750  2650 1500
 $Comp
 L R R56
@@
 $EndComp
 Wire Wire Line
-	3650 1900 4600 1900
-Wire Wire Line
 	3350 1900 3100 1900
 Wire Wire Line
@@
 Wire Wire Line
 	8100 800  8450 800
+$Comp
+L GS2 J?
+U 1 1 5AF39CAF
+P 4300 1900
+F 0 "J?" H 4400 2050 50  0000 C CNN
+F 1 "GS2" H 4400 1751 50  0000 C CNN
+F 2 "Connectors:GS2" V 4374 1900 50  0001 C CNN
+F 3 "" H 4300 1900 50  0001 C CNN
+	1    4300 1900
+	0    -1   -1   0
+$EndComp
+Wire Wire Line
+	3650 1900 4100 1900
+Wire Wire Line
+	4500 1900 4600 1900
 $EndSCHEMATC
