File: Projects/Voicemeeter/file5AF6330C.sch (KiCad schematic (older format))
At the start: 10 parts, among them U401 74HC4051, U402 74HC4051, U403 74HC4051, U404 74HC4051, U405 74HC4051, U406 74HC4051, U407 74HC4051, U408 74HC4051, U409 74HC4051, U410 74HC4051

Commit message: stuff
Parts:
- renumbered U401 to U1, U410 to U10, U402 to U2, U403 to U3, U404 to U4, U405 to U5, U406 to U6, U407 to U7, U408 to U8, U409 to U9
Changed lines of the file:
@@
 $EndDescr
 $Comp
-L 74HC4051 U401
+L 74HC4051 U1
 U 1 1 5AEAF7C0
 P 3600 1600
-F 0 "U401" H 3200 2350 60  0000 C CNN
+F 0 "U1" H 3200 2350 60  0000 C CNN
 F 1 "74HC4051" H 3250 2250 60  0000 C CNN
 F 2 "Housings_DIP:DIP-16_W7.62mm_LongPads" H 3600 1600 60  0001 C CNN
@@
 	3600 1050 3600 1050
 $Comp
-L GND #PWR022
+L GND #PWR23
 U 1 1 5AEAFE60
 P 3600 2150
-F 0 "#PWR022" H 3600 1900 50  0001 C CNN
+F 0 "#PWR23" H 3600 1900 50  0001 C CNN
 F 1 "GND" H 3600 2000 50  0000 C CNN
 F 2 "" H 3600 2150 50  0001 C CNN
@@
 $EndComp
 $Comp
-L +3.3V #PWR023
+L +3.3V #PWR22
 U 1 1 5AF6738F
 P 3600 1050
-F 0 "#PWR023" H 3600 900 50  0001 C CNN
+F 0 "#PWR22" H 3600 900 50  0001 C CNN
 F 1 "+3.3V" H 3600 1190 50  0000 C CNN
 F 2 "" H 3600 1050 50  0001 C CNN
@@
 	4000 750  4000 1200
 $Comp
-L 74HC4051 U402
+L 74HC4051 U2
 U 1 1 5AED3FF9
 P 3600 3300
-F 0 "U402" H 3200 4050 60  0000 C CNN
+F 0 "U2" H 3200 4050 60  0000 C CNN
 F 1 "74HC4051" H 3250 3950 60  0000 C CNN
 F 2 "Housings_DIP:DIP-16_W7.62mm_LongPads" H 3600 3300 60  0001 C CNN
@@
 	3600 2750 3600 2750
 $Comp
-L GND #PWR024
+L GND #PWR25
 U 1 1 5AED4000
 P 3600 3850
-F 0 "#PWR024" H 3600 3600 50  0001 C CNN
+F 0 "#PWR25" H 3600 3600 50  0001 C CNN
 F 1 "GND" H 3600 3700 50  0000 C CNN
 F 2 "" H 3600 3850 50  0001 C CNN
@@
 $EndComp
 $Comp
-L +3.3V #PWR025
+L +3.3V #PWR24
 U 1 1 5AED4006
 P 3600 2750
-F 0 "#PWR025" H 3600 2600 50  0001 C CNN
+F 0 "#PWR24" H 3600 2600 50  0001 C CNN
 F 1 "+3.3V" H 3600 2890 50  0000 C CNN
 F 2 "" H 3600 2750 50  0001 C CNN
@@
 	4000 2450 4000 2900
 $Comp
-L 74HC4051 U403
+L 74HC4051 U3
 U 1 1 5AED40AA
 P 3600 5000
-F 0 "U403" H 3200 5750 60  0000 C CNN
+F 0 "U3" H 3200 5750 60  0000 C CNN
 F 1 "74HC4051" H 3250 5650 60  0000 C CNN
 F 2 "Housings_DIP:DIP-16_W7.62mm_LongPads" H 3600 5000 60  0001 C CNN
@@
 	3600 4450 3600 4450
 $Comp
-L GND #PWR026
+L GND #PWR27
 U 1 1 5AED40B1
 P 3600 5550
-F 0 "#PWR026" H 3600 5300 50  0001 C CNN
+F 0 "#PWR27" H 3600 5300 50  0001 C CNN
 F 1 "GND" H 3600 5400 50  0000 C CNN
 F 2 "" H 3600 5550 50  0001 C CNN
@@
 $EndComp
 $Comp
-L +3.3V #PWR027
+L +3.3V #PWR26
 U 1 1 5AED40B7
 P 3600 4450
-F 0 "#PWR027" H 3600 4300 50  0001 C CNN
+F 0 "#PWR26" H 3600 4300 50  0001 C CNN
 F 1 "+3.3V" H 3600 4590 50  0000 C CNN
 F 2 "" H 3600 4450 50  0001 C CNN
@@
 	4000 4150 4000 4600
 $Comp
-L 74HC4051 U404
+L 74HC4051 U4
 U 1 1 5AED440D
 P 8350 1600
-F 0 "U404" H 7950 2350 60  0000 C CNN
+F 0 "U4" H 7950 2350 60  0000 C CNN
 F 1 "74HC4051" H 8000 2250 60  0000 C CNN
 F 2 "Housings_DIP:DIP-16_W7.62mm_LongPads" H 8350 1600 60  0001 C CNN
@@
 	8350 1050 8350 1050
 $Comp
-L GND #PWR028
+L GND #PWR29
 U 1 1 5AED4414
 P 8350 2150
-F 0 "#PWR028" H 8350 1900 50  0001 C CNN
+F 0 "#PWR29" H 8350 1900 50  0001 C CNN
 F 1 "GND" H 8350 2000 50  0000 C CNN
 F 2 "" H 8350 2150 50  0001 C CNN
@@
 $EndComp
 $Comp
-L +3.3V #PWR029
+L +3.3V #PWR28
 U 1 1 5AED441A
 P 8350 1050
-F 0 "#PWR029" H 8350 900 50  0001 C CNN
+F 0 "#PWR28" H 8350 900 50  0001 C CNN
 F 1 "+3.3V" H 8350 1190 50  0000 C CNN
 F 2 "" H 8350 1050 50  0001 C CNN
@@
 	7950 750  7950 1200
 $Comp
-L 74HC4051 U405
+L 74HC4051 U5
 U 1 1 5AED4437
 P 8350 3300
-F 0 "U405" H 7950 4050 60  0000 C CNN
+F 0 "U5" H 7950 4050 60  0000 C CNN
 F 1 "74HC4051" H 8000 3950 60  0000 C CNN
 F 2 "Housings_DIP:DIP-16_W7.62mm_LongPads" H 8350 3300 60  0001 C CNN
@@
 	8350 2750 8350 2750
 $Comp
-L GND #PWR030
+L GND #PWR31
 U 1 1 5AED443E
 P 8350 3850
-F 0 "#PWR030" H 8350 3600 50  0001 C CNN
+F 0 "#PWR31" H 8350 3600 50  0001 C CNN
 F 1 "GND" H 8350 3700 50  0000 C CNN
 F 2 "" H 8350 3850 50  0001 C CNN
@@
 $EndComp
 $Comp
-L +3.3V #PWR031
+L +3.3V #PWR30
 U 1 1 5AED4444
 P 8350 2750
-F 0 "#PWR031" H 8350 2600 50  0001 C CNN
+F 0 "#PWR30" H 8350 2600 50  0001 C CNN
 F 1 "+3.3V" H 8350 2890 50  0000 C CNN
 F 2 "" H 8350 2750 50  0001 C CNN
@@
 	7950 2450 7950 2900
 $Comp
-L 74HC4051 U406
+L 74HC4051 U6
 U 1 1 5AED4462
 P 8350 5000
-F 0 "U406" H 7950 5750 60  0000 C CNN
+F 0 "U6" H 7950 5750 60  0000 C CNN
 F 1 "74HC4051" H 8000 5650 60  0000 C CNN
 F 2 "Housings_DIP:DIP-16_W7.62mm_LongPads" H 8350 5000 60  0001 C CNN
@@
 	8350 4450 8350 4450
 $Comp
-L GND #PWR032
+L GND #PWR33
 U 1 1 5AED4469
 P 8350 5550
-F 0 "#PWR032" H 8350 5300 50  0001 C CNN
+F 0 "#PWR33" H 8350 5300 50  0001 C CNN
 F 1 "GND" H 8350 5400 50  0000 C CNN
 F 2 "" H 8350 5550 50  0001 C CNN
@@
 $EndComp
 $Comp
-L +3.3V #PWR033
+L +3.3V #PWR32
 U 1 1 5AED446F
 P 8350 4450
-F 0 "#PWR033" H 8350 4300 50  0001 C CNN
+F 0 "#PWR32" H 8350 4300 50  0001 C CNN
 F 1 "+3.3V" H 8350 4590 50  0000 C CNN
 F 2 "" H 8350 4450 50  0001 C CNN
@@
 	2700 600  9250 600
 $Comp
-L 74HC4051 U407
+L 74HC4051 U7
 U 1 1 5AED4578
 P 8350 6700
-F 0 "U407" H 7950 7450 60  0000 C CNN
+F 0 "U7" H 7950 7450 60  0000 C CNN
 F 1 "74HC4051" H 8000 7350 60  0000 C CNN
 F 2 "Housings_DIP:DIP-16_W7.62mm_LongPads" H 8350 6700 60  0001 C CNN
@@
 	8350 6150 8350 6150
 $Comp
-L GND #PWR034
+L GND #PWR35
 U 1 1 5AED457F
 P 8350 7250
-F 0 "#PWR034" H 8350 7000 50  0001 C CNN
+F 0 "#PWR35" H 8350 7000 50  0001 C CNN
 F 1 "GND" H 8350 7100 50  0000 C CNN
 F 2 "" H 8350 7250 50  0001 C CNN
@@
 $EndComp
 $Comp
-L +3.3V #PWR035
+L +3.3V #PWR34
 U 1 1 5AED4585
 P 8350 6150
-F 0 "#PWR035" H 8350 6000 50  0001 C CNN
+F 0 "#PWR34" H 8350 6000 50  0001 C CNN
 F 1 "+3.3V" H 8350 6290 50  0000 C CNN
 F 2 "" H 8350 6150 50  0001 C CNN
@@
 	7950 5850 7950 6300
 $Comp
-L 74HC4051 U408
+L 74HC4051 U8
 U 1 1 5AED461C
 P 8350 8400
-F 0 "U408" H 7950 9150 60  0000 C CNN
+F 0 "U8" H 7950 9150 60  0000 C CNN
 F 1 "74HC4051" H 8000 9050 60  0000 C CNN
 F 2 "Housings_DIP:DIP-16_W7.62mm_LongPads" H 8350 8400 60  0001 C CNN
@@
 	8350 7850 8350 7850
 $Comp
-L GND #PWR036
+L GND #PWR37
 U 1 1 5AED4623
 P 8350 8950
-F 0 "#PWR036" H 8350 8700 50  0001 C CNN
+F 0 "#PWR37" H 8350 8700 50  0001 C CNN
 F 1 "GND" H 8350 8800 50  0000 C CNN
 F 2 "" H 8350 8950 50  0001 C CNN
@@
 $EndComp
 $Comp
-L +3.3V #PWR037
+L +3.3V #PWR36
 U 1 1 5AED4629
 P 8350 7850
-F 0 "#PWR037" H 8350 7700 50  0001 C CNN
+F 0 "#PWR36" H 8350 7700 50  0001 C CNN
 F 1 "+3.3V" H 8350 7990 50  0000 C CNN
 F 2 "" H 8350 7850 50  0001 C CNN
@@
 	7950 7550 7950 8000
 $Comp
-L 74HC4051 U409
+L 74HC4051 U9
 U 1 1 5AED477E
 P 8350 10100
-F 0 "U409" H 7950 10850 60  0000 C CNN
+F 0 "U9" H 7950 10850 60  0000 C CNN
 F 1 "74HC4051" H 8000 10750 60  0000 C CNN
 F 2 "Housings_DIP:DIP-16_W7.62mm_LongPads" H 8350 10100 60  0001 C CNN
@@
 	8350 9550 8350 9550
 $Comp
-L GND #PWR038
+L GND #PWR39
 U 1 1 5AED4785
 P 8350 10650
-F 0 "#PWR038" H 8350 10400 50  0001 C CNN
+F 0 "#PWR39" H 8350 10400 50  0001 C CNN
 F 1 "GND" H 8350 10500 50  0000 C CNN
 F 2 "" H 8350 10650 50  0001 C CNN
@@
 $EndComp
 $Comp
-L +3.3V #PWR039
+L +3.3V #PWR38
 U 1 1 5AED478B
 P 8350 9550
-F 0 "#PWR039" H 8350 9400 50  0001 C CNN
+F 0 "#PWR38" H 8350 9400 50  0001 C CNN
 F 1 "+3.3V" H 8350 9690 50  0000 C CNN
 F 2 "" H 8350 9550 50  0001 C CNN
@@
 	7950 9250 7950 9700
 $Comp
-L 74HC4051 U410
+L 74HC4051 U10
 U 1 1 5AED4882
 P 8350 11800
-F 0 "U410" H 7950 12550 60  0000 C CNN
+F 0 "U10" H 7950 12550 60  0000 C CNN
 F 1 "74HC4051" H 8000 12450 60  0000 C CNN
 F 2 "Housings_DIP:DIP-16_W7.62mm_LongPads" H 8350 11800 60  0001 C CNN
@@
 	8350 11250 8350 11250
 $Comp
-L GND #PWR040
+L GND #PWR41
 U 1 1 5AED4889
 P 8350 12350
-F 0 "#PWR040" H 8350 12100 50  0001 C CNN
+F 0 "#PWR41" H 8350 12100 50  0001 C CNN
 F 1 "GND" H 8350 12200 50  0000 C CNN
 F 2 "" H 8350 12350 50  0001 C CNN
@@
 $EndComp
 $Comp
-L +3.3V #PWR041
+L +3.3V #PWR40
 U 1 1 5AED488F
 P 8350 11250
-F 0 "#PWR041" H 8350 11100 50  0001 C CNN
+F 0 "#PWR40" H 8350 11100 50  0001 C CNN
 F 1 "+3.3V" H 8350 11390 50  0000 C CNN
 F 2 "" H 8350 11250 50  0001 C CNN

Commit message: Zzzzz
Parts:
- renumbered U1 to U401, U2 to U402, U3 to U403, U4 to U404, U5 to U405, U6 to U406, U7 to U407, U8 to U408, U9 to U409, U10 to U410
Changed lines of the file:
@@
 $EndDescr
 $Comp
-L 74HC4051 U1
+L 74HC4051 U401
 U 1 1 5AEAF7C0
 P 3600 1600
-F 0 "U1" H 3200 2350 60  0000 C CNN
+F 0 "U401" H 3200 2350 60  0000 C CNN
 F 1 "74HC4051" H 3250 2250 60  0000 C CNN
 F 2 "Housings_DIP:DIP-16_W7.62mm_LongPads" H 3600 1600 60  0001 C CNN
@@
 	3600 1050 3600 1050
 $Comp
-L GND #PWR23
+L GND #PWR022
 U 1 1 5AEAFE60
 P 3600 2150
-F 0 "#PWR23" H 3600 1900 50  0001 C CNN
+F 0 "#PWR022" H 3600 1900 50  0001 C CNN
 F 1 "GND" H 3600 2000 50  0000 C CNN
 F 2 "" H 3600 2150 50  0001 C CNN
@@
 $EndComp
 $Comp
-L +3.3V #PWR22
+L +3.3V #PWR023
 U 1 1 5AF6738F
 P 3600 1050
-F 0 "#PWR22" H 3600 900 50  0001 C CNN
+F 0 "#PWR023" H 3600 900 50  0001 C CNN
 F 1 "+3.3V" H 3600 1190 50  0000 C CNN
 F 2 "" H 3600 1050 50  0001 C CNN
@@
 	4000 750  4000 1200
 $Comp
-L 74HC4051 U2
+L 74HC4051 U402
 U 1 1 5AED3FF9
 P 3600 3300
-F 0 "U2" H 3200 4050 60  0000 C CNN
+F 0 "U402" H 3200 4050 60  0000 C CNN
 F 1 "74HC4051" H 3250 3950 60  0000 C CNN
 F 2 "Housings_DIP:DIP-16_W7.62mm_LongPads" H 3600 3300 60  0001 C CNN
@@
 	3600 2750 3600 2750
 $Comp
-L GND #PWR25
+L GND #PWR024
 U 1 1 5AED4000
 P 3600 3850
-F 0 "#PWR25" H 3600 3600 50  0001 C CNN
+F 0 "#PWR024" H 3600 3600 50  0001 C CNN
 F 1 "GND" H 3600 3700 50  0000 C CNN
 F 2 "" H 3600 3850 50  0001 C CNN
@@
 $EndComp
 $Comp
-L +3.3V #PWR24
+L +3.3V #PWR025
 U 1 1 5AED4006
 P 3600 2750
-F 0 "#PWR24" H 3600 2600 50  0001 C CNN
+F 0 "#PWR025" H 3600 2600 50  0001 C CNN
 F 1 "+3.3V" H 3600 2890 50  0000 C CNN
 F 2 "" H 3600 2750 50  0001 C CNN
@@
 	4000 2450 4000 2900
 $Comp
-L 74HC4051 U3
+L 74HC4051 U403
 U 1 1 5AED40AA
 P 3600 5000
-F 0 "U3" H 3200 5750 60  0000 C CNN
+F 0 "U403" H 3200 5750 60  0000 C CNN
 F 1 "74HC4051" H 3250 5650 60  0000 C CNN
 F 2 "Housings_DIP:DIP-16_W7.62mm_LongPads" H 3600 5000 60  0001 C CNN
@@
 	3600 4450 3600 4450
 $Comp
-L GND #PWR27
+L GND #PWR026
 U 1 1 5AED40B1
 P 3600 5550
-F 0 "#PWR27" H 3600 5300 50  0001 C CNN
+F 0 "#PWR026" H 3600 5300 50  0001 C CNN
 F 1 "GND" H 3600 5400 50  0000 C CNN
 F 2 "" H 3600 5550 50  0001 C CNN
@@
 $EndComp
 $Comp
-L +3.3V #PWR26
+L +3.3V #PWR027
 U 1 1 5AED40B7
 P 3600 4450
-F 0 "#PWR26" H 3600 4300 50  0001 C CNN
+F 0 "#PWR027" H 3600 4300 50  0001 C CNN
 F 1 "+3.3V" H 3600 4590 50  0000 C CNN
 F 2 "" H 3600 4450 50  0001 C CNN
@@
 	4000 4150 4000 4600
 $Comp
-L 74HC4051 U4
+L 74HC4051 U404
 U 1 1 5AED440D
 P 8350 1600
-F 0 "U4" H 7950 2350 60  0000 C CNN
+F 0 "U404" H 7950 2350 60  0000 C CNN
 F 1 "74HC4051" H 8000 2250 60  0000 C CNN
 F 2 "Housings_DIP:DIP-16_W7.62mm_LongPads" H 8350 1600 60  0001 C CNN
@@
 	8350 1050 8350 1050
 $Comp
-L GND #PWR29
+L GND #PWR028
 U 1 1 5AED4414
 P 8350 2150
-F 0 "#PWR29" H 8350 1900 50  0001 C CNN
+F 0 "#PWR028" H 8350 1900 50  0001 C CNN
 F 1 "GND" H 8350 2000 50  0000 C CNN
 F 2 "" H 8350 2150 50  0001 C CNN
@@
 $EndComp
 $Comp
-L +3.3V #PWR28
+L +3.3V #PWR029
 U 1 1 5AED441A
 P 8350 1050
-F 0 "#PWR28" H 8350 900 50  0001 C CNN
+F 0 "#PWR029" H 8350 900 50  0001 C CNN
 F 1 "+3.3V" H 8350 1190 50  0000 C CNN
 F 2 "" H 8350 1050 50  0001 C CNN
@@
 	7950 750  7950 1200
 $Comp
-L 74HC4051 U5
+L 74HC4051 U405
 U 1 1 5AED4437
 P 8350 3300
-F 0 "U5" H 7950 4050 60  0000 C CNN
+F 0 "U405" H 7950 4050 60  0000 C CNN
 F 1 "74HC4051" H 8000 3950 60  0000 C CNN
 F 2 "Housings_DIP:DIP-16_W7.62mm_LongPads" H 8350 3300 60  0001 C CNN
@@
 	8350 2750 8350 2750
 $Comp
-L GND #PWR31
+L GND #PWR030
 U 1 1 5AED443E
 P 8350 3850
-F 0 "#PWR31" H 8350 3600 50  0001 C CNN
+F 0 "#PWR030" H 8350 3600 50  0001 C CNN
 F 1 "GND" H 8350 3700 50  0000 C CNN
 F 2 "" H 8350 3850 50  0001 C CNN
@@
 $EndComp
 $Comp
-L +3.3V #PWR30
+L +3.3V #PWR031
 U 1 1 5AED4444
 P 8350 2750
-F 0 "#PWR30" H 8350 2600 50  0001 C CNN
+F 0 "#PWR031" H 8350 2600 50  0001 C CNN
 F 1 "+3.3V" H 8350 2890 50  0000 C CNN
 F 2 "" H 8350 2750 50  0001 C CNN
@@
 	7950 2450 7950 2900
 $Comp
-L 74HC4051 U6
+L 74HC4051 U406
 U 1 1 5AED4462
 P 8350 5000
-F 0 "U6" H 7950 5750 60  0000 C CNN
+F 0 "U406" H 7950 5750 60  0000 C CNN
 F 1 "74HC4051" H 8000 5650 60  0000 C CNN
 F 2 "Housings_DIP:DIP-16_W7.62mm_LongPads" H 8350 5000 60  0001 C CNN
@@
 	8350 4450 8350 4450
 $Comp
-L GND #PWR33
+L GND #PWR032
 U 1 1 5AED4469
 P 8350 5550
-F 0 "#PWR33" H 8350 5300 50  0001 C CNN
+F 0 "#PWR032" H 8350 5300 50  0001 C CNN
 F 1 "GND" H 8350 5400 50  0000 C CNN
 F 2 "" H 8350 5550 50  0001 C CNN
@@
 $EndComp
 $Comp
-L +3.3V #PWR32
+L +3.3V #PWR033
 U 1 1 5AED446F
 P 8350 4450
-F 0 "#PWR32" H 8350 4300 50  0001 C CNN
+F 0 "#PWR033" H 8350 4300 50  0001 C CNN
 F 1 "+3.3V" H 8350 4590 50  0000 C CNN
 F 2 "" H 8350 4450 50  0001 C CNN
@@
 	2700 600  9250 600
 $Comp
-L 74HC4051 U7
+L 74HC4051 U407
 U 1 1 5AED4578
 P 8350 6700
-F 0 "U7" H 7950 7450 60  0000 C CNN
+F 0 "U407" H 7950 7450 60  0000 C CNN
 F 1 "74HC4051" H 8000 7350 60  0000 C CNN
 F 2 "Housings_DIP:DIP-16_W7.62mm_LongPads" H 8350 6700 60  0001 C CNN
@@
 	8350 6150 8350 6150
 $Comp
-L GND #PWR35
+L GND #PWR034
 U 1 1 5AED457F
 P 8350 7250
-F 0 "#PWR35" H 8350 7000 50  0001 C CNN
+F 0 "#PWR034" H 8350 7000 50  0001 C CNN
 F 1 "GND" H 8350 7100 50  0000 C CNN
 F 2 "" H 8350 7250 50  0001 C CNN
@@
 $EndComp
 $Comp
-L +3.3V #PWR34
+L +3.3V #PWR035
 U 1 1 5AED4585
 P 8350 6150
-F 0 "#PWR34" H 8350 6000 50  0001 C CNN
+F 0 "#PWR035" H 8350 6000 50  0001 C CNN
 F 1 "+3.3V" H 8350 6290 50  0000 C CNN
 F 2 "" H 8350 6150 50  0001 C CNN
@@
 	7950 5850 7950 6300
 $Comp
-L 74HC4051 U8
+L 74HC4051 U408
 U 1 1 5AED461C
 P 8350 8400
-F 0 "U8" H 7950 9150 60  0000 C CNN
+F 0 "U408" H 7950 9150 60  0000 C CNN
 F 1 "74HC4051" H 8000 9050 60  0000 C CNN
 F 2 "Housings_DIP:DIP-16_W7.62mm_LongPads" H 8350 8400 60  0001 C CNN
@@
 	8350 7850 8350 7850
 $Comp
-L GND #PWR37
+L GND #PWR036
 U 1 1 5AED4623
 P 8350 8950
-F 0 "#PWR37" H 8350 8700 50  0001 C CNN
+F 0 "#PWR036" H 8350 8700 50  0001 C CNN
 F 1 "GND" H 8350 8800 50  0000 C CNN
 F 2 "" H 8350 8950 50  0001 C CNN
@@
 $EndComp
 $Comp
-L +3.3V #PWR36
+L +3.3V #PWR037
 U 1 1 5AED4629
 P 8350 7850
-F 0 "#PWR36" H 8350 7700 50  0001 C CNN
+F 0 "#PWR037" H 8350 7700 50  0001 C CNN
 F 1 "+3.3V" H 8350 7990 50  0000 C CNN
 F 2 "" H 8350 7850 50  0001 C CNN
@@
 	7950 7550 7950 8000
 $Comp
-L 74HC4051 U9
+L 74HC4051 U409
 U 1 1 5AED477E
 P 8350 10100
-F 0 "U9" H 7950 10850 60  0000 C CNN
+F 0 "U409" H 7950 10850 60  0000 C CNN
 F 1 "74HC4051" H 8000 10750 60  0000 C CNN
 F 2 "Housings_DIP:DIP-16_W7.62mm_LongPads" H 8350 10100 60  0001 C CNN
@@
 	8350 9550 8350 9550
 $Comp
-L GND #PWR39
+L GND #PWR038
 U 1 1 5AED4785
 P 8350 10650
-F 0 "#PWR39" H 8350 10400 50  0001 C CNN
+F 0 "#PWR038" H 8350 10400 50  0001 C CNN
 F 1 "GND" H 8350 10500 50  0000 C CNN
 F 2 "" H 8350 10650 50  0001 C CNN
@@
 $EndComp
 $Comp
-L +3.3V #PWR38
+L +3.3V #PWR039
 U 1 1 5AED478B
 P 8350 9550
-F 0 "#PWR38" H 8350 9400 50  0001 C CNN
+F 0 "#PWR039" H 8350 9400 50  0001 C CNN
 F 1 "+3.3V" H 8350 9690 50  0000 C CNN
 F 2 "" H 8350 9550 50  0001 C CNN
@@
 	7950 9250 7950 9700
 $Comp
-L 74HC4051 U10
+L 74HC4051 U410
 U 1 1 5AED4882
 P 8350 11800
-F 0 "U10" H 7950 12550 60  0000 C CNN
+F 0 "U410" H 7950 12550 60  0000 C CNN
 F 1 "74HC4051" H 8000 12450 60  0000 C CNN
 F 2 "Housings_DIP:DIP-16_W7.62mm_LongPads" H 8350 11800 60  0001 C CNN
@@
 	8350 11250 8350 11250
 $Comp
-L GND #PWR41
+L GND #PWR040
 U 1 1 5AED4889
 P 8350 12350
-F 0 "#PWR41" H 8350 12100 50  0001 C CNN
+F 0 "#PWR040" H 8350 12100 50  0001 C CNN
 F 1 "GND" H 8350 12200 50  0000 C CNN
 F 2 "" H 8350 12350 50  0001 C CNN
@@
 $EndComp
 $Comp
-L +3.3V #PWR40
+L +3.3V #PWR041
 U 1 1 5AED488F
 P 8350 11250
-F 0 "#PWR40" H 8350 11100 50  0001 C CNN
+F 0 "#PWR041" H 8350 11100 50  0001 C CNN
 F 1 "+3.3V" H 8350 11390 50  0000 C CNN
 F 2 "" H 8350 11250 50  0001 C CNN
