File: Projects/Voicemeeter/file5AF6330C.sch (KiCad schematic (older format))
At the start: 10 parts

Commit message: why did a lock file sneak in? <.<
Parts:
- U401, U402, U403, U404, U405, U406, U407, U408, U409, U410: renamed from U?; footprint (none) -> Housings_DIP:DIP-16_W7.62mm_LongPads
Changed lines of the file:
@@
 NoConn ~ 4000 3400
 $Comp
-L 74HC4051 U?
+L 74HC4051 U401
 U 1 1 5AF5E23A
 P 3600 1600
-F 0 "U?" H 3200 2350 60  0000 C CNN
+F 0 "U401" H 3200 2350 60  0000 C CNN
 F 1 "74HC4051" H 3250 2250 60  0000 C CNN
-F 2 "" H 3600 1600 60  0000 C CNN
+F 2 "Housings_DIP:DIP-16_W7.62mm_LongPads" H 3600 1600 60  0001 C CNN
 F 3 "" H 3600 1600 60  0000 C CNN
 F 4 "CD74HC4051E" H 3300 2450 60  0001 C CNN "part_num"
@@
 $EndComp
 $Comp
-L 74HC4051 U?
+L 74HC4051 U402
 U 1 1 5AF5E29D
 P 3600 3300
-F 0 "U?" H 3200 4050 60  0000 C CNN
+F 0 "U402" H 3200 4050 60  0000 C CNN
 F 1 "74HC4051" H 3250 3950 60  0000 C CNN
-F 2 "" H 3600 3300 60  0000 C CNN
+F 2 "Housings_DIP:DIP-16_W7.62mm_LongPads" H 3600 3300 60  0001 C CNN
 F 3 "" H 3600 3300 60  0000 C CNN
 F 4 "CD74HC4051E" H 3300 4150 60  0001 C CNN "part_num"
@@
 $EndComp
 $Comp
-L 74HC4051 U?
+L 74HC4051 U403
 U 1 1 5AF5E2FB
 P 3600 5000
-F 0 "U?" H 3200 5750 60  0000 C CNN
+F 0 "U403" H 3200 5750 60  0000 C CNN
 F 1 "74HC4051" H 3250 5650 60  0000 C CNN
-F 2 "" H 3600 5000 60  0000 C CNN
+F 2 "Housings_DIP:DIP-16_W7.62mm_LongPads" H 3600 5000 60  0001 C CNN
 F 3 "" H 3600 5000 60  0000 C CNN
 F 4 "CD74HC4051E" H 3300 5850 60  0001 C CNN "part_num"
@@
 $EndComp
 $Comp
-L 74HC4051 U?
+L 74HC4051 U404
 U 1 1 5AF5E356
 P 8350 1600
-F 0 "U?" H 7950 2350 60  0000 C CNN
+F 0 "U404" H 7950 2350 60  0000 C CNN
 F 1 "74HC4051" H 8000 2250 60  0000 C CNN
-F 2 "" H 8350 1600 60  0000 C CNN
+F 2 "Housings_DIP:DIP-16_W7.62mm_LongPads" H 8350 1600 60  0001 C CNN
 F 3 "" H 8350 1600 60  0000 C CNN
 F 4 "CD74HC4051E" H 8050 2450 60  0001 C CNN "part_num"
@@
 $EndComp
 $Comp
-L 74HC4051 U?
+L 74HC4051 U405
 U 1 1 5AF5E45E
 P 8350 3300
-F 0 "U?" H 7950 4050 60  0000 C CNN
+F 0 "U405" H 7950 4050 60  0000 C CNN
 F 1 "74HC4051" H 8000 3950 60  0000 C CNN
-F 2 "" H 8350 3300 60  0000 C CNN
+F 2 "Housings_DIP:DIP-16_W7.62mm_LongPads" H 8350 3300 60  0001 C CNN
 F 3 "" H 8350 3300 60  0000 C CNN
 F 4 "CD74HC4051E" H 8050 4150 60  0001 C CNN "part_num"
@@
 $EndComp
 $Comp
-L 74HC4051 U?
+L 74HC4051 U406
 U 1 1 5AF5E4AD
 P 8350 5000
-F 0 "U?" H 7950 5750 60  0000 C CNN
+F 0 "U406" H 7950 5750 60  0000 C CNN
 F 1 "74HC4051" H 8000 5650 60  0000 C CNN
-F 2 "" H 8350 5000 60  0000 C CNN
+F 2 "Housings_DIP:DIP-16_W7.62mm_LongPads" H 8350 5000 60  0001 C CNN
 F 3 "" H 8350 5000 60  0000 C CNN
 F 4 "CD74HC4051E" H 8050 5850 60  0001 C CNN "part_num"
@@
 $EndComp
 $Comp
-L 74HC4051 U?
+L 74HC4051 U407
 U 1 1 5AF5E5A9
 P 8350 6700
-F 0 "U?" H 7950 7450 60  0000 C CNN
+F 0 "U407" H 7950 7450 60  0000 C CNN
 F 1 "74HC4051" H 8000 7350 60  0000 C CNN
-F 2 "" H 8350 6700 60  0000 C CNN
+F 2 "Housings_DIP:DIP-16_W7.62mm_LongPads" H 8350 6700 60  0001 C CNN
 F 3 "" H 8350 6700 60  0000 C CNN
 F 4 "CD74HC4051E" H 8050 7550 60  0001 C CNN "part_num"
@@
 $EndComp
 $Comp
-L 74HC4051 U?
+L 74HC4051 U408
 U 1 1 5AF5E600
 P 8350 8400
-F 0 "U?" H 7950 9150 60  0000 C CNN
+F 0 "U408" H 7950 9150 60  0000 C CNN
 F 1 "74HC4051" H 8000 9050 60  0000 C CNN
-F 2 "" H 8350 8400 60  0000 C CNN
+F 2 "Housings_DIP:DIP-16_W7.62mm_LongPads" H 8350 8400 60  0001 C CNN
 F 3 "" H 8350 8400 60  0000 C CNN
 F 4 "CD74HC4051E" H 8050 9250 60  0001 C CNN "part_num"
@@
 $EndComp
 $Comp
-L 74HC4051 U?
+L 74HC4051 U409
 U 1 1 5AF5E6C0
 P 8350 10100
-F 0 "U?" H 7950 10850 60  0000 C CNN
+F 0 "U409" H 7950 10850 60  0000 C CNN
 F 1 "74HC4051" H 8000 10750 60  0000 C CNN
-F 2 "" H 8350 10100 60  0000 C CNN
+F 2 "Housings_DIP:DIP-16_W7.62mm_LongPads" H 8350 10100 60  0001 C CNN
 F 3 "" H 8350 10100 60  0000 C CNN
 F 4 "CD74HC4051E" H 8050 10950 60  0001 C CNN "part_num"
@@
 $EndComp
 $Comp
-L 74HC4051 U?
+L 74HC4051 U410
 U 1 1 5AF5E727
 P 8350 11800
-F 0 "U?" H 7950 12550 60  0000 C CNN
+F 0 "U410" H 7950 12550 60  0000 C CNN
 F 1 "74HC4051" H 8000 12450 60  0000 C CNN
-F 2 "" H 8350 11800 60  0000 C CNN
+F 2 "Housings_DIP:DIP-16_W7.62mm_LongPads" H 8350 11800 60  0001 C CNN
 F 3 "" H 8350 11800 60  0000 C CNN
 F 4 "CD74HC4051E" H 8050 12650 60  0001 C CNN "part_num"

Commit message: in case of emergency
Connections:
- net +3V3: now also U401.6 (~EN), U402.6 (~EN), U403.6 (~EN), U404.6 (~EN), U405.6 (~EN), U406.6 (~EN), U407.6 (~EN), U408.6 (~EN), U409.6 (~EN), U410.6 (~EN)
- no-connect marks 23 -> 13
Changed lines of the file:
@@
 	3600 1050 3600 1050
 $Comp
-L GND #PWR403
+L GND #PWR022
 U 1 1 5AEAFE60
 P 3600 2150
-F 0 "#PWR403" H 3600 1900 50  0001 C CNN
+F 0 "#PWR022" H 3600 1900 50  0001 C CNN
 F 1 "GND" H 3600 2000 50  0000 C CNN
 F 2 "" H 3600 2150 50  0001 C CNN
@@
 $EndComp
 $Comp
-L +3.3V #PWR401
+L +3.3V #PWR023
 U 1 1 5AF6738F
 P 3600 1050
-F 0 "#PWR401" H 3600 900 50  0001 C CNN
+F 0 "#PWR023" H 3600 900 50  0001 C CNN
 F 1 "+3.3V" H 3600 1190 50  0000 C CNN
 F 2 "" H 3600 1050 50  0001 C CNN
@@
 Wire Wire Line
 	4000 1600 4650 1600
-NoConn ~ 3200 1700
 NoConn ~ 3200 1900
 Wire Wire Line
@@
 	3600 2750 3600 2750
 $Comp
-L GND #PWR407
+L GND #PWR024
 U 1 1 5AED4000
 P 3600 3850
-F 0 "#PWR407" H 3600 3600 50  0001 C CNN
+F 0 "#PWR024" H 3600 3600 50  0001 C CNN
 F 1 "GND" H 3600 3700 50  0000 C CNN
 F 2 "" H 3600 3850 50  0001 C CNN
@@
 $EndComp
 $Comp
-L +3.3V #PWR405
+L +3.3V #PWR025
 U 1 1 5AED4006
 P 3600 2750
-F 0 "#PWR405" H 3600 2600 50  0001 C CNN
+F 0 "#PWR025" H 3600 2600 50  0001 C CNN
 F 1 "+3.3V" H 3600 2890 50  0000 C CNN
 F 2 "" H 3600 2750 50  0001 C CNN
@@
 Wire Wire Line
 	4000 3300 4650 3300
-NoConn ~ 3200 3400
 NoConn ~ 3200 3600
 Wire Wire Line
@@
 	3600 4450 3600 4450
 $Comp
-L GND #PWR411
+L GND #PWR026
 U 1 1 5AED40B1
 P 3600 5550
-F 0 "#PWR411" H 3600 5300 50  0001 C CNN
+F 0 "#PWR026" H 3600 5300 50  0001 C CNN
 F 1 "GND" H 3600 5400 50  0000 C CNN
 F 2 "" H 3600 5550 50  0001 C CNN
@@
 $EndComp
 $Comp
-L +3.3V #PWR409
+L +3.3V #PWR027
 U 1 1 5AED40B7
 P 3600 4450
-F 0 "#PWR409" H 3600 4300 50  0001 C CNN
+F 0 "#PWR027" H 3600 4300 50  0001 C CNN
 F 1 "+3.3V" H 3600 4590 50  0000 C CNN
 F 2 "" H 3600 4450 50  0001 C CNN
@@
 Wire Wire Line
 	4000 5000 4650 5000
-NoConn ~ 3200 5100
 NoConn ~ 3200 5300
 Wire Wire Line
@@
 	8350 1050 8350 1050
 $Comp
-L GND #PWR404
+L GND #PWR028
 U 1 1 5AED4414
 P 8350 2150
-F 0 "#PWR404" H 8350 1900 50  0001 C CNN
+F 0 "#PWR028" H 8350 1900 50  0001 C CNN
 F 1 "GND" H 8350 2000 50  0000 C CNN
 F 2 "" H 8350 2150 50  0001 C CNN
@@
 $EndComp
 $Comp
-L +3.3V #PWR402
+L +3.3V #PWR029
 U 1 1 5AED441A
 P 8350 1050
-F 0 "#PWR402" H 8350 900 50  0001 C CNN
+F 0 "#PWR029" H 8350 900 50  0001 C CNN
 F 1 "+3.3V" H 8350 1190 50  0000 C CNN
 F 2 "" H 8350 1050 50  0001 C CNN
@@
 Wire Wire Line
 	7950 1600 7300 1600
-NoConn ~ 8750 1700
 NoConn ~ 8750 1900
 Wire Wire Line
@@
 	8350 2750 8350 2750
 $Comp
-L GND #PWR408
+L GND #PWR030
 U 1 1 5AED443E
 P 8350 3850
-F 0 "#PWR408" H 8350 3600 50  0001 C CNN
+F 0 "#PWR030" H 8350 3600 50  0001 C CNN
 F 1 "GND" H 8350 3700 50  0000 C CNN
 F 2 "" H 8350 3850 50  0001 C CNN
@@
 $EndComp
 $Comp
-L +3.3V #PWR406
+L +3.3V #PWR031
 U 1 1 5AED4444
 P 8350 2750
-F 0 "#PWR406" H 8350 2600 50  0001 C CNN
+F 0 "#PWR031" H 8350 2600 50  0001 C CNN
 F 1 "+3.3V" H 8350 2890 50  0000 C CNN
 F 2 "" H 8350 2750 50  0001 C CNN
@@
 Wire Wire Line
 	7950 3300 7300 3300
-NoConn ~ 8750 3400
 NoConn ~ 8750 3600
 Wire Wire Line
@@
 	8350 4450 8350 4450
 $Comp
-L GND #PWR412
+L GND #PWR032
 U 1 1 5AED4469
 P 8350 5550
-F 0 "#PWR412" H 8350 5300 50  0001 C CNN
+F 0 "#PWR032" H 8350 5300 50  0001 C CNN
 F 1 "GND" H 8350 5400 50  0000 C CNN
 F 2 "" H 8350 5550 50  0001 C CNN
@@
 $EndComp
 $Comp
-L +3.3V #PWR410
+L +3.3V #PWR033
 U 1 1 5AED446F
 P 8350 4450
-F 0 "#PWR410" H 8350 4300 50  0001 C CNN
+F 0 "#PWR033" H 8350 4300 50  0001 C CNN
 F 1 "+3.3V" H 8350 4590 50  0000 C CNN
 F 2 "" H 8350 4450 50  0001 C CNN
@@
 Wire Wire Line
 	7950 5000 7300 5000
-NoConn ~ 8750 5100
 NoConn ~ 8750 5300
 Wire Wire Line
@@
 	8350 6150 8350 6150
 $Comp
-L GND #PWR414
+L GND #PWR034
 U 1 1 5AED457F
 P 8350 7250
-F 0 "#PWR414" H 8350 7000 50  0001 C CNN
+F 0 "#PWR034" H 8350 7000 50  0001 C CNN
 F 1 "GND" H 8350 7100 50  0000 C CNN
 F 2 "" H 8350 7250 50  0001 C CNN
@@
 $EndComp
 $Comp
-L +3.3V #PWR413
+L +3.3V #PWR035
 U 1 1 5AED4585
 P 8350 6150
-F 0 "#PWR413" H 8350 6000 50  0001 C CNN
+F 0 "#PWR035" H 8350 6000 50  0001 C CNN
 F 1 "+3.3V" H 8350 6290 50  0000 C CNN
 F 2 "" H 8350 6150 50  0001 C CNN
@@
 Wire Wire Line
 	7950 6700 7300 6700
-NoConn ~ 8750 6800
 NoConn ~ 8750 7000
 Wire Wire Line
@@
 	8350 7850 8350 7850
 $Comp
-L GND #PWR416
+L GND #PWR036
 U 1 1 5AED4623
 P 8350 8950
-F 0 "#PWR416" H 8350 8700 50  0001 C CNN
+F 0 "#PWR036" H 8350 8700 50  0001 C CNN
 F 1 "GND" H 8350 8800 50  0000 C CNN
 F 2 "" H 8350 8950 50  0001 C CNN
@@
 $EndComp
 $Comp
-L +3.3V #PWR415
+L +3.3V #PWR037
 U 1 1 5AED4629
 P 8350 7850
-F 0 "#PWR415" H 8350 7700 50  0001 C CNN
+F 0 "#PWR037" H 8350 7700 50  0001 C CNN
 F 1 "+3.3V" H 8350 7990 50  0000 C CNN
 F 2 "" H 8350 7850 50  0001 C CNN
@@
 Wire Wire Line
 	7950 8400 7300 8400
-NoConn ~ 8750 8500
 NoConn ~ 8750 8700
 Wire Wire Line
@@
 	8350 9550 8350 9550
 $Comp
-L GND #PWR418
+L GND #PWR038
 U 1 1 5AED4785
 P 8350 10650
-F 0 "#PWR418" H 8350 10400 50  0001 C CNN
+F 0 "#PWR038" H 8350 10400 50  0001 C CNN
 F 1 "GND" H 8350 10500 50  0000 C CNN
 F 2 "" H 8350 10650 50  0001 C CNN
@@
 $EndComp
 $Comp
-L +3.3V #PWR417
+L +3.3V #PWR039
 U 1 1 5AED478B
 P 8350 9550
-F 0 "#PWR417" H 8350 9400 50  0001 C CNN
+F 0 "#PWR039" H 8350 9400 50  0001 C CNN
 F 1 "+3.3V" H 8350 9690 50  0000 C CNN
 F 2 "" H 8350 9550 50  0001 C CNN
@@
 Wire Wire Line
 	7950 10100 7300 10100
-NoConn ~ 8750 10200
 NoConn ~ 8750 10400
 Wire Wire Line
@@
 	8350 11250 8350 11250
 $Comp
-L GND #PWR420
+L GND #PWR040
 U 1 1 5AED4889
 P 8350 12350
-F 0 "#PWR420" H 8350 12100 50  0001 C CNN
+F 0 "#PWR040" H 8350 12100 50  0001 C CNN
 F 1 "GND" H 8350 12200 50  0000 C CNN
 F 2 "" H 8350 12350 50  0001 C CNN
@@
 $EndComp
 $Comp
-L +3.3V #PWR419
+L +3.3V #PWR041
 U 1 1 5AED488F
 P 8350 11250
-F 0 "#PWR419" H 8350 11100 50  0001 C CNN
+F 0 "#PWR041" H 8350 11100 50  0001 C CNN
 F 1 "+3.3V" H 8350 11390 50  0000 C CNN
 F 2 "" H 8350 11250 50  0001 C CNN
@@
 Wire Wire Line
 	7950 12100 7300 12100
-NoConn ~ 8750 11900
 NoConn ~ 8750 12100
 Wire Wire Line
@@
 	-1   0    0    -1
 $EndComp
+$Comp
+L +3.3V #PWR042
+U 1 1 5AFBA642
+P 3150 3350
+F 0 "#PWR042" H 3150 3200 50  0001 C CNN
+F 1 "+3.3V" H 3150 3490 50  0000 C CNN
+F 2 "" H 3150 3350 50  0001 C CNN
+F 3 "" H 3150 3350 50  0001 C CNN
+	1    3150 3350
+	1    0    0    -1
+$EndComp
+Wire Wire Line
+	3150 3350 3150 3400
+Wire Wire Line
+	3150 3400 3200 3400
+$Comp
+L +3.3V #PWR043
+U 1 1 5AFBA8F5
+P 3150 5050
+F 0 "#PWR043" H 3150 4900 50  0001 C CNN
+F 1 "+3.3V" H 3150 5190 50  0000 C CNN
+F 2 "" H 3150 5050 50  0001 C CNN
+F 3 "" H 3150 5050 50  0001 C CNN
+	1    3150 5050
+	1    0    0    -1
+$EndComp
+Wire Wire Line
+	3150 5050 3150 5100
+Wire Wire Line
+	3150 5100 3200 5100
+$Comp
+L +3.3V #PWR044
+U 1 1 5AFBAA1F
+P 3150 1650
+F 0 "#PWR044" H 3150 1500 50  0001 C CNN
+F 1 "+3.3V" H 3150 1790 50  0000 C CNN
+F 2 "" H 3150 1650 50  0001 C CNN
+F 3 "" H 3150 1650 50  0001 C CNN
+	1    3150 1650
+	1    0    0    -1
+$EndComp
+Wire Wire Line
+	3150 1650 3150 1700
+Wire Wire Line
+	3150 1700 3200 1700
+$Comp
+L +3.3V #PWR045
+U 1 1 5AFBAC7F
+P 8800 1650
+F 0 "#PWR045" H 8800 1500 50  0001 C CNN
+F 1 "+3.3V" H 8800 1790 50  0000 C CNN
+F 2 "" H 8800 1650 50  0001 C CNN
+F 3 "" H 8800 1650 50  0001 C CNN
+	1    8800 1650
+	-1   0    0    -1
+$EndComp
+Wire Wire Line
+	8750 1700 8800 1700
+Wire Wire Line
+	8800 1700 8800 1650
+$Comp
+L +3.3V #PWR046
+U 1 1 5AFBAE0A
+P 8800 3350
+F 0 "#PWR046" H 8800 3200 50  0001 C CNN
+F 1 "+3.3V" H 8800 3490 50  0000 C CNN
+F 2 "" H 8800 3350 50  0001 C CNN
+F 3 "" H 8800 3350 50  0001 C CNN
+	1    8800 3350
+	-1   0    0    -1
+$EndComp
+Wire Wire Line
+	8750 3400 8800 3400
+Wire Wire Line
+	8800 3400 8800 3350
+$Comp
+L +3.3V #PWR047
+U 1 1 5AFBAF8E
+P 8800 5050
+F 0 "#PWR047" H 8800 4900 50  0001 C CNN
+F 1 "+3.3V" H 8800 5190 50  0000 C CNN
+F 2 "" H 8800 5050 50  0001 C CNN
+F 3 "" H 8800 5050 50  0001 C CNN
+	1    8800 5050
+	-1   0    0    -1
+$EndComp
+Wire Wire Line
+	8750 5100 8800 5100
+Wire Wire Line
+	8800 5100 8800 5050
+$Comp
+L +3.3V #PWR048
+U 1 1 5AFBB202
+P 8800 6750
+F 0 "#PWR048" H 8800 6600 50  0001 C CNN
+F 1 "+3.3V" H 8800 6890 50  0000 C CNN
+F 2 "" H 8800 6750 50  0001 C CNN
+F 3 "" H 8800 6750 50  0001 C CNN
+	1    8800 6750
+	-1   0    0    -1
+$EndComp
+Wire Wire Line
+	8750 6800 8800 6800
+Wire Wire Line
+	8800 6800 8800 6750
+$Comp
+L +3.3V #PWR049
+U 1 1 5AFBB2FA
+P 8800 10150
+F 0 "#PWR049" H 8800 10000 50  0001 C CNN
+F 1 "+3.3V" H 8800 10290 50  0000 C CNN
+F 2 "" H 8800 10150 50  0001 C CNN
+F 3 "" H 8800 10150 50  0001 C CNN
+	1    8800 10150
+	-1   0    0    -1
+$EndComp
+Wire Wire Line
+	8750 10200 8800 10200
+Wire Wire Line
+	8800 10200 8800 10150
+$Comp
+L +3.3V #PWR050
+U 1 1 5AFBB35C
+P 8800 8450
+F 0 "#PWR050" H 8800 8300 50  0001 C CNN
+F 1 "+3.3V" H 8800 8590 50  0000 C CNN
+F 2 "" H 8800 8450 50  0001 C CNN
+F 3 "" H 8800 8450 50  0001 C CNN
+	1    8800 8450
+	-1   0    0    -1
+$EndComp
+Wire Wire Line
+	8750 8500 8800 8500
+Wire Wire Line
+	8800 8500 8800 8450
+$Comp
+L +3.3V #PWR051
+U 1 1 5AFBB490
+P 8800 11850
+F 0 "#PWR051" H 8800 11700 50  0001 C CNN
+F 1 "+3.3V" H 8800 11990 50  0000 C CNN
+F 2 "" H 8800 11850 50  0001 C CNN
+F 3 "" H 8800 11850 50  0001 C CNN
+	1    8800 11850
+	-1   0    0    -1
+$EndComp
+Wire Wire Line
+	8750 11900 8800 11900
+Wire Wire Line
+	8800 11900 8800 11850
 $EndSCHEMATC

Commit message: gtg
Connections:
- net HD17: now also U404.13 (X0); no longer U404.12 (X3)
- net HD18: now also U404.12 (X3); no longer U404.13 (X0)
Changed lines of the file:
@@
 Text Label 7300 1400 0    60   ~ 0
 HD16
+Text Label 7300 1300 0    60   ~ 0
+HD17
 Text Label 7300 1600 0    60   ~ 0
-HD17
-Text Label 7300 1300 0    60   ~ 0
 HD18
 Text Label 7300 3500 0    60   ~ 0

Commit message: boop
Connections:
- net DA13: now also U403.15 (X2); no longer U403.13 (X0)
- net DA14: now also U403.13 (X0); no longer U403.14 (X1)
- net DA22: now also U403.5 (X5); no longer U403.15 (X2)
- net HA12: now also U401.1 (X4); no longer U401.2 (X6)
- net HA13: now also U401.2 (X6); no longer U401.1 (X4)
- net HA33: now also U403.14 (X1); no longer U403.5 (X5)
- net HD27: now also U405.13 (X0); no longer U405.12 (X3)
- net HD28: now also U405.12 (X3); no longer U405.13 (X0)
Changed lines of the file:
@@
 Text Label 4400 1500 0    60   ~ 0
 HA11
-Text Label 4400 1900 0    60   ~ 0
+Text Label 4100 1700 0    60   ~ 0
 HA12
-Text Label 4400 1700 0    60   ~ 0
+Text Label 4100 1900 0    60   ~ 0
 HA13
 Text Label 4400 2000 0    60   ~ 0
@@
 Text Label 4400 1600 0    60   ~ 0
 HA32
-Text Label 4400 5200 0    60   ~ 0
+Text Label 4100 4800 0    60   ~ 0
 HA33
 Text Label 4400 3500 0    60   ~ 0
@@
 Text Label 4400 5000 0    60   ~ 0
 DA12
-Text Label 4400 4700 0    60   ~ 0
+Text Label 4100 4900 0    60   ~ 0
 DA13
-Text Label 4400 4800 0    60   ~ 0
+Text Label 4100 4700 0    60   ~ 0
 DA14
 Text Label 4400 3600 0    60   ~ 0
 DA21
-Text Label 4400 4900 0    60   ~ 0
+Text Label 4100 5200 0    60   ~ 0
 DA22
 Text Label 4400 5100 0    60   ~ 0
@@
 Text Label 7300 3100 0    60   ~ 0
 HD26
-Text Label 7300 3300 0    60   ~ 0
+Text Label 7550 3000 0    60   ~ 0
 HD27
-Text Label 7300 3000 0    60   ~ 0
+Text Label 7550 3300 0    60   ~ 0
 HD28
 Text Label 7300 5200 0    60   ~ 0

Commit message: starting to get bored
Connections:
- net DA22: now also U403.1 (X4); no longer U403.5 (X5)
- net DA23: now also U403.5 (X5); no longer U403.1 (X4)
- net DD17: now also U407.13 (X0); no longer U407.12 (X3)
- net DD18: now also U407.12 (X3); no longer U407.13 (X0)
- net DD27: now also U408.13 (X0); no longer U408.12 (X3)
- net DD28: now also U408.12 (X3); no longer U408.13 (X0)
- net HD37: now also U406.13 (X0); no longer U406.12 (X3)
- net HD38: now also U406.12 (X3); no longer U406.13 (X0)
- net OD51: now also U410.5 (X5); no longer U410.2 (X6)
- net OD52: now also U410.4 (X7); no longer U410.5 (X5)
- net OD53: now also U410.2 (X6); no longer U410.4 (X7)
Changed lines of the file:
@@
 Text Label 4400 1600 0    60   ~ 0
 HA32
-Text Label 4100 4800 0    60   ~ 0
+Text Label 4400 4800 0    60   ~ 0
 HA33
 Text Label 4400 3500 0    60   ~ 0
@@
 Text Label 4400 5000 0    60   ~ 0
 DA12
-Text Label 4100 4900 0    60   ~ 0
+Text Label 4400 4900 0    60   ~ 0
 DA13
-Text Label 4100 4700 0    60   ~ 0
+Text Label 4400 4700 0    60   ~ 0
 DA14
 Text Label 4400 3600 0    60   ~ 0
 DA21
+Text Label 4400 5100 0    60   ~ 0
+DA22
 Text Label 4100 5200 0    60   ~ 0
-DA22
-Text Label 4400 5100 0    60   ~ 0
 DA23
 Text Label 4400 5300 0    60   ~ 0
@@
 Text Label 7300 4800 0    60   ~ 0
 HD36
-Text Label 7300 5000 0    60   ~ 0
+Text Label 7600 4700 0    60   ~ 0
 HD37
-Text Label 7300 4700 0    60   ~ 0
+Text Label 7600 5000 0    60   ~ 0
 HD38
 Text Label 7300 6900 0    60   ~ 0
@@
 Text Label 7300 6500 0    60   ~ 0
 DD16
-Text Label 7300 6700 0    60   ~ 0
+Text Label 7650 6400 0    60   ~ 0
 DD17
-Text Label 7300 6400 0    60   ~ 0
+Text Label 7550 6700 0    60   ~ 0
 DD18
 Text Label 7300 8600 0    60   ~ 0
@@
 Text Label 7300 8200 0    60   ~ 0
 DD26
+Text Label 7300 8100 0    60   ~ 0
+DD27
 Text Label 7300 8400 0    60   ~ 0
-DD27
-Text Label 7300 8100 0    60   ~ 0
 DD28
 Text Label 7300 10500 0    60   ~ 0
@@
 Text Label 7300 11500 0    60   ~ 0
 OD43
-Text Label 7300 12100 0    60   ~ 0
+Text Label 7650 12000 0    60   ~ 0
 OD51
-Text Label 7300 12000 0    60   ~ 0
+Text Label 7600 12200 0    60   ~ 0
 OD52
-Text Label 7300 12200 0    60   ~ 0
+Text Label 7600 12100 0    60   ~ 0
 OD53
 Wire Bus Line

Commit message: before it's too late
Connections:
- net DA13: now also U403.5 (X5); no longer U403.15 (X2)
- net DA22: now also U403.15 (X2); no longer U403.1 (X4)
- net DA23: now also U403.2 (X6); no longer U403.5 (X5)
- net DA24: now also U403.1 (X4); no longer U403.2 (X6)
Changed lines of the file:
@@
 	7200 12000 7300 12100
 Wire Bus Line
-	4750 3500 4750 5300
+	4750 3500 4750 5200
 Wire Bus Line
 	4750 2900 4850 2900
@@
 Text Label 4400 5000 0    60   ~ 0
 DA12
-Text Label 4400 4900 0    60   ~ 0
+Text Label 4400 5200 0    60   ~ 0
 DA13
 Text Label 4400 4700 0    60   ~ 0
@@
 Text Label 4400 3600 0    60   ~ 0
 DA21
-Text Label 4400 5100 0    60   ~ 0
+Text Label 4150 4900 0    60   ~ 0
 DA22
-Text Label 4100 5200 0    60   ~ 0
+Text Label 4150 5300 0    60   ~ 0
 DA23
-Text Label 4400 5300 0    60   ~ 0
+Text Label 4150 5100 0    60   ~ 0
 DA24
 Text Label 7300 1800 0    60   ~ 0
