File: Projects/Voicemeeter/_saved_file5AF6330C.sch (KiCad schematic (older format))
At the start: 10 parts

Commit message: dvcvcv
Parts:
- gave numbers to parts that had none: 10
Changed lines of the file:
@@
 NoConn ~ 4000 3400
 $Comp
-L 74HC4051 U?
+L 74HC4051 U401
 U 1 1 5AF5E23A
 P 3600 1600
-F 0 "U?" H 3200 2350 60  0000 C CNN
+F 0 "U401" H 3200 2350 60  0000 C CNN
 F 1 "74HC4051" H 3250 2250 60  0000 C CNN
 F 2 "" H 3600 1600 60  0000 C CNN
@@
 $EndComp
 $Comp
-L 74HC4051 U?
+L 74HC4051 U402
 U 1 1 5AF5E29D
 P 3600 3300
-F 0 "U?" H 3200 4050 60  0000 C CNN
+F 0 "U402" H 3200 4050 60  0000 C CNN
 F 1 "74HC4051" H 3250 3950 60  0000 C CNN
 F 2 "" H 3600 3300 60  0000 C CNN
@@
 $EndComp
 $Comp
-L 74HC4051 U?
+L 74HC4051 U403
 U 1 1 5AF5E2FB
 P 3600 5000
-F 0 "U?" H 3200 5750 60  0000 C CNN
+F 0 "U403" H 3200 5750 60  0000 C CNN
 F 1 "74HC4051" H 3250 5650 60  0000 C CNN
 F 2 "" H 3600 5000 60  0000 C CNN
@@
 $EndComp
 $Comp
-L 74HC4051 U?
+L 74HC4051 U404
 U 1 1 5AF5E356
 P 8350 1600
-F 0 "U?" H 7950 2350 60  0000 C CNN
+F 0 "U404" H 7950 2350 60  0000 C CNN
 F 1 "74HC4051" H 8000 2250 60  0000 C CNN
 F 2 "" H 8350 1600 60  0000 C CNN
@@
 $EndComp
 $Comp
-L 74HC4051 U?
+L 74HC4051 U405
 U 1 1 5AF5E45E
 P 8350 3300
-F 0 "U?" H 7950 4050 60  0000 C CNN
+F 0 "U405" H 7950 4050 60  0000 C CNN
 F 1 "74HC4051" H 8000 3950 60  0000 C CNN
 F 2 "" H 8350 3300 60  0000 C CNN
@@
 $EndComp
 $Comp
-L 74HC4051 U?
+L 74HC4051 U406
 U 1 1 5AF5E4AD
 P 8350 5000
-F 0 "U?" H 7950 5750 60  0000 C CNN
+F 0 "U406" H 7950 5750 60  0000 C CNN
 F 1 "74HC4051" H 8000 5650 60  0000 C CNN
 F 2 "" H 8350 5000 60  0000 C CNN
@@
 $EndComp
 $Comp
-L 74HC4051 U?
+L 74HC4051 U407
 U 1 1 5AF5E5A9
 P 8350 6700
-F 0 "U?" H 7950 7450 60  0000 C CNN
+F 0 "U407" H 7950 7450 60  0000 C CNN
 F 1 "74HC4051" H 8000 7350 60  0000 C CNN
 F 2 "" H 8350 6700 60  0000 C CNN
@@
 $EndComp
 $Comp
-L 74HC4051 U?
+L 74HC4051 U408
 U 1 1 5AF5E600
 P 8350 8400
-F 0 "U?" H 7950 9150 60  0000 C CNN
+F 0 "U408" H 7950 9150 60  0000 C CNN
 F 1 "74HC4051" H 8000 9050 60  0000 C CNN
 F 2 "" H 8350 8400 60  0000 C CNN
@@
 $EndComp
 $Comp
-L 74HC4051 U?
+L 74HC4051 U409
 U 1 1 5AF5E6C0
 P 8350 10100
-F 0 "U?" H 7950 10850 60  0000 C CNN
+F 0 "U409" H 7950 10850 60  0000 C CNN
 F 1 "74HC4051" H 8000 10750 60  0000 C CNN
 F 2 "" H 8350 10100 60  0000 C CNN
@@
 $EndComp
 $Comp
-L 74HC4051 U?
+L 74HC4051 U410
 U 1 1 5AF5E727
 P 8350 11800
-F 0 "U?" H 7950 12550 60  0000 C CNN
+F 0 "U410" H 7950 12550 60  0000 C CNN
 F 1 "74HC4051" H 8000 12450 60  0000 C CNN
 F 2 "" H 8350 11800 60  0000 C CNN
