File: Projects/Voicemeeter/file5AE49270.sch (KiCad schematic (older format))
At the start: 132 parts, among them SW201 SW_SPDT_6pin, SW202 SW_SPDT_6pin, SW203 SW_SPDT_6pin, SW204 SW_SPDT_6pin, SW205 SW_SPDT_6pin, SW206 SW_SPDT_6pin, SW207 SW_SPDT_6pin, SW208 SW_SPDT_6pin, SW209 SW_SPDT_6pin, SW210 SW_SPDT_6pin, SW211 SW_SPDT_6pin, SW212 SW_SPDT_6pin, SW213 SW_SPDT_6pin, SW214 SW_SPDT_6pin, SW215 SW_SPDT_6pin, SW216 SW_SPDT_6pin, SW217 SW_SPDT_6pin, SW218 SW_SPDT_6pin, SW219 SW_SPDT_6pin, SW220 SW_SPDT_6pin, SW221 SW_SPDT_6pin, SW222 SW_SPDT_6pin, SW223 SW_SPDT_6pin, SW224 SW_SPDT_6pin, SW225 SW_SPDT_6pin, SW226 SW_SPDT_6pin, SW227 SW_SPDT_6pin, SW228 SW_SPDT_6pin, SW229 SW_SPDT_6pin, SW230 SW_SPDT_6pin, SW231 SW_SPDT_6pin, SW232 SW_SPDT_6pin, SW233 SW_SPDT_6pin, SW234 SW_SPDT_6pin, SW235 SW_SPDT_6pin, SW236 SW_SPDT_6pin, SW237 SW_SPDT_6pin, SW238 SW_SPDT_6pin, SW239 SW_SPDT_6pin, SW240 SW_SPDT_6pin, SW241 SW_SPDT_6pin, SW242 SW_SPDT_6pin, SW243 SW_SPDT_6pin, SW244 SW_SPDT_6pin, SW245 SW_SPDT_6pin, SW246 SW_SPDT_6pin, SW247 SW_SPDT_6pin, SW248 SW_SPDT_6pin, SW249 SW_SPDT_6pin, SW250 SW_SPDT_6pin, SW251 SW_SPDT_6pin, SW252 SW_SPDT_6pin, SW253 SW_SPDT_6pin, SW254 SW_SPDT_6pin, SW255 SW_SPDT_6pin

Commit message: stuff
Parts:
- renumbered R201 to R1, R210 to R10, R211 to R11, R212 to R12, R213 to R13, R214 to R14, R215 to R15, R216 to R16, R217 to R17, R218 to R18, R219 to R19, R202 to R2, R220 to R20, R221 to R21, R222 to R22, R223 to R23, R224 to R24, R225 to R25, R226 to R26, R227 to R27, R228 to R28, R229 to R29, R203 to R3, R230 to R30, R231 to R31, R232 to R32, R233 to R33, R234 to R34, R235 to R35, R236 to R36, R237 to R37, R238 to R38, R239 to R39, R204 to R4, R240 to R40, R241 to R41, R242 to R42, R243 to R43, R244 to R44, R245 to R45, R246 to R46, R247 to R47, R248 to R48, R249 to R49, R205 to R5, R250 to R50, R251 to R51, R252 to R52, R253 to R53, R254 to R54, R255 to R55, R206 to R6, R207 to R7, R208 to R8, R209 to R9, RV201 to RV1, RV210 to RV10, RV211 to RV11, RV212 to RV12, RV213 to RV13, RV214 to RV14, RV215 to RV15, RV216 to RV16, RV217 to RV17, RV218 to RV18, RV219 to RV19, RV202 to RV2, RV220 to RV20, RV221 to RV21, RV222 to RV22, RV203 to RV3, RV204 to RV4, RV205 to RV5, RV206 to RV6, RV207 to RV7, RV208 to RV8, RV209 to RV9, SW201 to SW1, SW210 to SW10, SW211 to SW11, SW212 to SW12, SW213 to SW13, SW214 to SW14, SW215 to SW15, SW216 to SW16, SW217 to SW17, SW218 to SW18, SW219 to SW19, SW202 to SW2, SW220 to SW20, SW221 to SW21, SW222 to SW22, SW223 to SW23, SW224 to SW24, SW225 to SW25, SW226 to SW26, SW227 to SW27, SW228 to SW28, SW229 to SW29, SW203 to SW3, SW230 to SW30, SW231 to SW31, SW232 to SW32, SW233 to SW33, SW234 to SW34, SW235 to SW35, SW236 to SW36, SW237 to SW37, SW238 to SW38, SW239 to SW39, SW204 to SW4, SW240 to SW40, SW241 to SW41, SW242 to SW42, SW243 to SW43, SW244 to SW44, SW245 to SW45, SW246 to SW46, SW247 to SW47, SW248 to SW48, SW249 to SW49, SW205 to SW5, SW250 to SW50, SW251 to SW51, SW252 to SW52, SW253 to SW53, SW254 to SW54, SW255 to SW55, SW206 to SW6, SW207 to SW7, SW208 to SW8, SW209 to SW9

Commit message: stuff
Parts:
- RV10, RV14, RV18, RV19, RV2, RV20, RV21, RV22, RV5, RV8: footprint pots:slidepot -> MATHSTERK:slidepot
- SW1, SW10, SW11, SW12, SW13, SW14, SW15, SW16, SW17, SW18, SW19, SW2, SW20, SW21, SW22, SW23, SW24, SW25, SW26, SW27, SW28, SW29, SW3, SW30, SW31, SW32, SW33, SW34, SW35, SW36, SW37, SW38, SW39, SW4, SW40, SW41, SW42, SW43, SW44, SW45, SW46, SW47, SW48, SW49, SW5, SW50, SW51, SW52, SW53, SW54, SW55, SW6, SW7, SW8, SW9: footprint switches:8mm_push_button -> MATHSTERK:8mm_push_button

Commit message: Zzzzz
Parts:
- renumbered R1 to R201, R2 to R202, R3 to R203, R4 to R204, R5 to R205, R6 to R206, R7 to R207, R8 to R208, R9 to R209, R10 to R210, R11 to R211, R12 to R212, R13 to R213, R14 to R214, R15 to R215, R16 to R216, R17 to R217, R18 to R218, R19 to R219, R20 to R220, R21 to R221, R22 to R222, R23 to R223, R24 to R224, R25 to R225, R26 to R226, R27 to R227, R28 to R228, R29 to R229, R30 to R230, R31 to R231, R32 to R232, R33 to R233, R34 to R234, R35 to R235, R36 to R236, R37 to R237, R38 to R238, R39 to R239, R40 to R240, R41 to R241, R42 to R242, R43 to R243, R44 to R244, R45 to R245, R46 to R246, R47 to R247, R48 to R248, R49 to R249, R50 to R250, R51 to R251, R52 to R252, R53 to R253, R54 to R254, R55 to R255, RV1 to RV201, RV2 to RV202, RV3 to RV203, RV4 to RV204, RV5 to RV205, RV6 to RV206, RV7 to RV207, RV8 to RV208, RV9 to RV209, RV10 to RV210, RV11 to RV211, RV12 to RV212, RV13 to RV213, RV14 to RV214, RV15 to RV215, RV16 to RV216, RV17 to RV217, RV18 to RV218, RV19 to RV219, RV20 to RV220, RV21 to RV221, RV22 to RV222, SW1 to SW201, SW2 to SW202, SW3 to SW203, SW4 to SW204, SW5 to SW205, SW6 to SW206, SW7 to SW207, SW8 to SW208, SW9 to SW209, SW10 to SW210, SW11 to SW211, SW12 to SW212, SW13 to SW213, SW14 to SW214, SW15 to SW215, SW16 to SW216, SW17 to SW217, SW18 to SW218, SW19 to SW219, SW20 to SW220, SW21 to SW221, SW22 to SW222, SW23 to SW223, SW24 to SW224, SW25 to SW225, SW26 to SW226, SW27 to SW227, SW28 to SW228, SW29 to SW229, SW30 to SW230, SW31 to SW231, SW32 to SW232, SW33 to SW233, SW34 to SW234, SW35 to SW235, SW36 to SW236, SW37 to SW237, SW38 to SW238, SW39 to SW239, SW40 to SW240, SW41 to SW241, SW42 to SW242, SW43 to SW243, SW44 to SW244, SW45 to SW245, SW46 to SW246, SW47 to SW247, SW48 to SW248, SW49 to SW249, SW50 to SW250, SW51 to SW251, SW52 to SW252, SW53 to SW253, SW54 to SW254, SW55 to SW255

Commit message: why did a lock file sneak in? <.<
Parts:
- removed RV201, RV203, RV204, RV206, RV207, RV209, RV211, RV212, RV213, RV215, RV216, RV217: POT, Potentiometers:Potentiometer_Omeg_PC16PU_Horizontal, symbol POT
- removed RV202, RV205, RV208, RV210, RV214, RV218, RV219, RV220, RV221, RV222: SLIDEPOT, MATHSTERK:slidepot, symbol POT
- added RV? (x22): POT, symbol POT
Connections:
- net +3V3: now also RV?.1, RV?.1, RV?.1, RV?.1, RV?.1, RV?.1, RV?.1, RV?.1, RV?.1, RV?.1, RV?.1, RV?.1, RV?.1, RV?.1, RV?.1, RV?.1, RV?.1, RV?.1, RV?.1, RV?.1, RV?.1, RV?.1
- net DA11: now also RV?.2
- net DA12: now also RV?.2
- net DA13: now also RV?.2
- net DA14: now also RV?.2
- net DA21: now also RV?.2
- net DA22: now also RV?.2
- net DA23: now also RV?.2
- net DA24: now also RV?.2
- net GND: now also RV?.3, RV?.3, RV?.3, RV?.3, RV?.3, RV?.3, RV?.3, RV?.3, RV?.3, RV?.3, RV?.3, RV?.3, RV?.3, RV?.3, RV?.3, RV?.3, RV?.3, RV?.3, RV?.3, RV?.3, RV?.3, RV?.3
- net HA11: now also RV?.2
- net HA12: now also RV?.2
- net HA13: now also RV?.2
- net HA21: now also RV?.2
- net HA22: now also RV?.2
- net HA23: now also RV?.2
- net HA31: now also RV?.2
- net HA32: now also RV?.2
- net HA33: now also RV?.2
- net OA1: now also RV?.2
- net OA2: now also RV?.2
- net OA3: now also RV?.2
- net OA4: now also RV?.2
- net OA5: now also RV?.2
