File: Projects/Voicemeeter/file5AE49270.sch (KiCad schematic (older format))
At the start: 132 parts, among them SW201 SW_SPDT_6pin, SW202 SW_SPDT_6pin, SW203 SW_SPDT_6pin, SW204 SW_SPDT_6pin, SW205 SW_SPDT_6pin, SW206 SW_SPDT_6pin, SW207 SW_SPDT_6pin, SW208 SW_SPDT_6pin, SW209 SW_SPDT_6pin, SW210 SW_SPDT_6pin, SW211 SW_SPDT_6pin, SW212 SW_SPDT_6pin, SW213 SW_SPDT_6pin, SW214 SW_SPDT_6pin, SW215 SW_SPDT_6pin, SW216 SW_SPDT_6pin, SW217 SW_SPDT_6pin, SW218 SW_SPDT_6pin, SW219 SW_SPDT_6pin, SW220 SW_SPDT_6pin, SW221 SW_SPDT_6pin, SW222 SW_SPDT_6pin, SW223 SW_SPDT_6pin, SW224 SW_SPDT_6pin, SW225 SW_SPDT_6pin, SW226 SW_SPDT_6pin, SW227 SW_SPDT_6pin, SW228 SW_SPDT_6pin, SW229 SW_SPDT_6pin, SW230 SW_SPDT_6pin, SW231 SW_SPDT_6pin, SW232 SW_SPDT_6pin, SW233 SW_SPDT_6pin, SW234 SW_SPDT_6pin, SW235 SW_SPDT_6pin, SW236 SW_SPDT_6pin, SW237 SW_SPDT_6pin, SW238 SW_SPDT_6pin, SW239 SW_SPDT_6pin, SW240 SW_SPDT_6pin, SW241 SW_SPDT_6pin, SW242 SW_SPDT_6pin, SW243 SW_SPDT_6pin, SW244 SW_SPDT_6pin, SW245 SW_SPDT_6pin, SW246 SW_SPDT_6pin, SW247 SW_SPDT_6pin, SW248 SW_SPDT_6pin, SW249 SW_SPDT_6pin, SW250 SW_SPDT_6pin, SW251 SW_SPDT_6pin, SW252 SW_SPDT_6pin, SW253 SW_SPDT_6pin, SW254 SW_SPDT_6pin, SW255 SW_SPDT_6pin

Commit message: considering stuff
Parts:
- gave numbers to parts that had none: 22
Changed lines of the file:
@@
 $EndComp
 $Comp
-L POT RV?
+L POT RV201
 U 1 1 5AF6EA0A
 P 1800 2000
-F 0 "RV?" V 1625 2000 50  0000 C CNN
+F 0 "RV201" V 1625 2000 50  0000 C CNN
 F 1 "POT" V 1700 2000 50  0000 C CNN
 F 2 "" H 1800 2000 50  0001 C CNN
@@
 $EndComp
 $Comp
-L POT RV?
+L POT RV203
 U 1 1 5AF705D6
 P 2900 2000
-F 0 "RV?" V 2725 2000 50  0000 C CNN
+F 0 "RV203" V 2725 2000 50  0000 C CNN
 F 1 "POT" V 2800 2000 50  0000 C CNN
 F 2 "" H 2900 2000 50  0001 C CNN
@@
 $EndComp
 $Comp
-L POT RV?
+L POT RV206
 U 1 1 5AF70976
 P 4500 2000
-F 0 "RV?" V 4325 2000 50  0000 C CNN
+F 0 "RV206" V 4325 2000 50  0000 C CNN
 F 1 "POT" V 4400 2000 50  0000 C CNN
 F 2 "" H 4500 2000 50  0001 C CNN
@@
 $EndComp
 $Comp
-L POT RV?
+L POT RV209
 U 1 1 5AF70F89
 P 6100 2000
-F 0 "RV?" V 5925 2000 50  0000 C CNN
+F 0 "RV209" V 5925 2000 50  0000 C CNN
 F 1 "POT" V 6000 2000 50  0000 C CNN
 F 2 "" H 6100 2000 50  0001 C CNN
@@
 $EndComp
 $Comp
-L POT RV?
+L POT RV204
 U 1 1 5AF713D7
 P 3400 2000
-F 0 "RV?" V 3225 2000 50  0000 C CNN
+F 0 "RV204" V 3225 2000 50  0000 C CNN
 F 1 "POT" V 3300 2000 50  0000 C CNN
 F 2 "" H 3400 2000 50  0001 C CNN
@@
 $EndComp
 $Comp
-L POT RV?
+L POT RV207
 U 1 1 5AF71615
 P 5000 2000
-F 0 "RV?" V 4825 2000 50  0000 C CNN
+F 0 "RV207" V 4825 2000 50  0000 C CNN
 F 1 "POT" V 4900 2000 50  0000 C CNN
 F 2 "" H 5000 2000 50  0001 C CNN
@@
 $EndComp
 $Comp
-L POT RV?
+L POT RV211
 U 1 1 5AF724A8
 P 6600 2000
-F 0 "RV?" V 6425 2000 50  0000 C CNN
+F 0 "RV211" V 6425 2000 50  0000 C CNN
 F 1 "POT" V 6500 2000 50  0000 C CNN
 F 2 "" H 6600 2000 50  0001 C CNN
@@
 $EndComp
 $Comp
-L POT RV?
+L POT RV213
 U 1 1 5AF727E2
 P 7500 2000
-F 0 "RV?" V 7325 2000 50  0000 C CNN
+F 0 "RV213" V 7325 2000 50  0000 C CNN
 F 1 "POT" V 7400 2000 50  0000 C CNN
 F 2 "" H 7500 2000 50  0001 C CNN
@@
 $EndComp
 $Comp
-L POT RV?
+L POT RV212
 U 1 1 5AF72990
 P 7450 1500
-F 0 "RV?" V 7275 1500 50  0000 C CNN
+F 0 "RV212" V 7275 1500 50  0000 C CNN
 F 1 "POT" V 7350 1500 50  0000 C CNN
 F 2 "" H 7450 1500 50  0001 C CNN
@@
 $EndComp
 $Comp
-L POT RV?
+L POT RV216
 U 1 1 5AF72B35
 P 9050 1500
-F 0 "RV?" V 8875 1500 50  0000 C CNN
+F 0 "RV216" V 8875 1500 50  0000 C CNN
 F 1 "POT" V 8950 1500 50  0000 C CNN
 F 2 "" H 9050 1500 50  0001 C CNN
@@
 $EndComp
 $Comp
-L POT RV?
+L POT RV217
 U 1 1 5AF72CF3
 P 9100 2000
-F 0 "RV?" V 8925 2000 50  0000 C CNN
+F 0 "RV217" V 8925 2000 50  0000 C CNN
 F 1 "POT" V 9000 2000 50  0000 C CNN
 F 2 "" H 9100 2000 50  0001 C CNN
@@
 $EndComp
 $Comp
-L POT RV?
+L POT RV215
 U 1 1 5AF72F27
 P 8200 2000
-F 0 "RV?" V 8025 2000 50  0000 C CNN
+F 0 "RV215" V 8025 2000 50  0000 C CNN
 F 1 "POT" V 8100 2000 50  0000 C CNN
 F 2 "" H 8200 2000 50  0001 C CNN
@@
 $EndComp
 $Comp
-L POT RV?
+L POT RV202
 U 1 1 5AF789D8
 P 1800 2600
-F 0 "RV?" V 1625 2600 50  0000 C CNN
+F 0 "RV202" V 1625 2600 50  0000 C CNN
 F 1 "POT" V 1700 2600 50  0000 C CNN
 F 2 "" H 1800 2600 50  0001 C CNN
@@
 $EndComp
 $Comp
-L POT RV?
+L POT RV205
 U 1 1 5AF7AE42
 P 3400 2600
-F 0 "RV?" V 3225 2600 50  0000 C CNN
+F 0 "RV205" V 3225 2600 50  0000 C CNN
 F 1 "POT" V 3300 2600 50  0000 C CNN
 F 2 "" H 3400 2600 50  0001 C CNN
@@
 $EndComp
 $Comp
-L POT RV?
+L POT RV208
 U 1 1 5AF7B004
 P 5000 2600
-F 0 "RV?" V 4825 2600 50  0000 C CNN
+F 0 "RV208" V 4825 2600 50  0000 C CNN
 F 1 "POT" V 4900 2600 50  0000 C CNN
 F 2 "" H 5000 2600 50  0001 C CNN
@@
 $EndComp
 $Comp
-L POT RV?
+L POT RV210
 U 1 1 5AF7B1AD
 P 6550 2600
-F 0 "RV?" V 6375 2600 50  0000 C CNN
+F 0 "RV210" V 6375 2600 50  0000 C CNN
 F 1 "POT" V 6450 2600 50  0000 C CNN
 F 2 "" H 6550 2600 50  0001 C CNN
@@
 $EndComp
 $Comp
-L POT RV?
+L POT RV214
 U 1 1 5AF7BCBB
 P 8150 2600
-F 0 "RV?" V 7975 2600 50  0000 C CNN
+F 0 "RV214" V 7975 2600 50  0000 C CNN
 F 1 "POT" V 8050 2600 50  0000 C CNN
 F 2 "" H 8150 2600 50  0001 C CNN
@@
 $EndComp
 $Comp
-L POT RV?
+L POT RV218
 U 1 1 5AF7BE86
 P 9750 2600
-F 0 "RV?" V 9575 2600 50  0000 C CNN
+F 0 "RV218" V 9575 2600 50  0000 C CNN
 F 1 "POT" V 9650 2600 50  0000 C CNN
 F 2 "" H 9750 2600 50  0001 C CNN
@@
 $EndComp
 $Comp
-L POT RV?
+L POT RV219
 U 1 1 5AF7C04E
 P 10950 2600
-F 0 "RV?" V 10775 2600 50  0000 C CNN
+F 0 "RV219" V 10775 2600 50  0000 C CNN
 F 1 "POT" V 10850 2600 50  0000 C CNN
 F 2 "" H 10950 2600 50  0001 C CNN
@@
 $EndComp
 $Comp
-L POT RV?
+L POT RV220
 U 1 1 5AF7C20F
 P 12150 2600
-F 0 "RV?" V 11975 2600 50  0000 C CNN
+F 0 "RV220" V 11975 2600 50  0000 C CNN
 F 1 "POT" V 12050 2600 50  0000 C CNN
 F 2 "" H 12150 2600 50  0001 C CNN
@@
 $EndComp
 $Comp
-L POT RV?
+L POT RV221
 U 1 1 5AF7C3C7
 P 13350 2600
-F 0 "RV?" V 13175 2600 50  0000 C CNN
+F 0 "RV221" V 13175 2600 50  0000 C CNN
 F 1 "POT" V 13250 2600 50  0000 C CNN
 F 2 "" H 13350 2600 50  0001 C CNN
@@
 $EndComp
 $Comp
-L POT RV?
+L POT RV222
 U 1 1 5AF7C582
 P 14550 2600
-F 0 "RV?" V 14375 2600 50  0000 C CNN
+F 0 "RV222" V 14375 2600 50  0000 C CNN
 F 1 "POT" V 14450 2600 50  0000 C CNN
 F 2 "" H 14550 2600 50  0001 C CNN

Commit message: need to do stuff elsewhere
Parts:
- RV202, RV205, RV208, RV210, RV214, RV218, RV219, RV220, RV221, RV222: footprint (none) -> MATHSTERK:slidepot
Changed lines of the file:
@@
 F 0 "RV202" V 1625 2600 50  0000 C CNN
 F 1 "POT" V 1700 2600 50  0000 C CNN
-F 2 "" H 1800 2600 50  0001 C CNN
+F 2 "MATHSTERK:slidepot" H 1800 2600 50  0001 C CNN
 F 3 "" V 1625 2600 50  0001 C CNN
 F 4 "RS6011YA6009" V 1725 2700 60  0001 C CNN "part_num"
@@
 F 0 "RV205" V 3225 2600 50  0000 C CNN
 F 1 "POT" V 3300 2600 50  0000 C CNN
-F 2 "" H 3400 2600 50  0001 C CNN
+F 2 "MATHSTERK:slidepot" H 3400 2600 50  0001 C CNN
 F 3 "" V 3225 2600 50  0001 C CNN
 F 4 "RS6011YA6009" V 3325 2700 60  0001 C CNN "part_num"
@@
 F 0 "RV208" V 4825 2600 50  0000 C CNN
 F 1 "POT" V 4900 2600 50  0000 C CNN
-F 2 "" H 5000 2600 50  0001 C CNN
+F 2 "MATHSTERK:slidepot" H 5000 2600 50  0001 C CNN
 F 3 "" V 4825 2600 50  0001 C CNN
 F 4 "RS6011YA6009" V 4925 2700 60  0001 C CNN "part_num"
@@
 F 0 "RV210" V 6375 2600 50  0000 C CNN
 F 1 "POT" V 6450 2600 50  0000 C CNN
-F 2 "" H 6550 2600 50  0001 C CNN
+F 2 "MATHSTERK:slidepot" H 6550 2600 50  0001 C CNN
 F 3 "" V 6375 2600 50  0001 C CNN
 F 4 "RS6011YA6009" V 6475 2700 60  0001 C CNN "part_num"
@@
 F 0 "RV214" V 7975 2600 50  0000 C CNN
 F 1 "POT" V 8050 2600 50  0000 C CNN
-F 2 "" H 8150 2600 50  0001 C CNN
+F 2 "MATHSTERK:slidepot" H 8150 2600 50  0001 C CNN
 F 3 "" V 7975 2600 50  0001 C CNN
 F 4 "RS6011YA6009" V 8075 2700 60  0001 C CNN "part_num"
@@
 F 0 "RV218" V 9575 2600 50  0000 C CNN
 F 1 "POT" V 9650 2600 50  0000 C CNN
-F 2 "" H 9750 2600 50  0001 C CNN
+F 2 "MATHSTERK:slidepot" H 9750 2600 50  0001 C CNN
 F 3 "" V 9575 2600 50  0001 C CNN
 F 4 "RS6011YA6009" V 9675 2700 60  0001 C CNN "part_num"
@@
 F 0 "RV219" V 10775 2600 50  0000 C CNN
 F 1 "POT" V 10850 2600 50  0000 C CNN
-F 2 "" H 10950 2600 50  0001 C CNN
+F 2 "MATHSTERK:slidepot" H 10950 2600 50  0001 C CNN
 F 3 "" V 10775 2600 50  0001 C CNN
 F 4 "RS6011YA6009" V 10875 2700 60  0001 C CNN "part_num"
@@
 F 0 "RV220" V 11975 2600 50  0000 C CNN
 F 1 "POT" V 12050 2600 50  0000 C CNN
-F 2 "" H 12150 2600 50  0001 C CNN
+F 2 "MATHSTERK:slidepot" H 12150 2600 50  0001 C CNN
 F 3 "" V 11975 2600 50  0001 C CNN
 F 4 "RS6011YA6009" V 12075 2700 60  0001 C CNN "part_num"
@@
 F 0 "RV221" V 13175 2600 50  0000 C CNN
 F 1 "POT" V 13250 2600 50  0000 C CNN
-F 2 "" H 13350 2600 50  0001 C CNN
+F 2 "MATHSTERK:slidepot" H 13350 2600 50  0001 C CNN
 F 3 "" V 13175 2600 50  0001 C CNN
 F 4 "RS6011YA6009" V 13275 2700 60  0001 C CNN "part_num"
@@
 F 0 "RV222" V 14375 2600 50  0000 C CNN
 F 1 "POT" V 14450 2600 50  0000 C CNN
-F 2 "" H 14550 2600 50  0001 C CNN
+F 2 "MATHSTERK:slidepot" H 14550 2600 50  0001 C CNN
 F 3 "" V 14375 2600 50  0001 C CNN
 F 4 "RS6011YA6009" V 14475 2700 60  0001 C CNN "part_num"

Commit message: uuuuuugh
Parts:
- RV201, RV203, RV204, RV206, RV207, RV209, RV211, RV212, RV213, RV215, RV216, RV217: footprint (none) -> MATHSTERK:Pot
Connections:
- net GND: now also RV201.4 (GND), RV202.4 (GND), RV203.4 (GND), RV204.4 (GND), RV205.4 (GND), RV206.4 (GND), RV207.4 (GND), RV208.4 (GND), RV209.4 (GND), RV210.4 (GND), RV211.4 (GND), RV212.4 (GND), RV213.4 (GND), RV214.4 (GND), RV215.4 (GND), RV216.4 (GND), RV217.4 (GND), RV218.4 (GND), RV219.4 (GND), RV220.4 (GND), RV221.4 (GND), RV222.4 (GND)
Changed lines of the file:
@@
 $Descr A3 16535 11693
 encoding utf-8
-Sheet 2 6
+Sheet 2 7
 Title ""
 Date ""
@@
 	11950 4750 12050 4650
 Wire Wire Line
-	1800 2750 2900 2750
+	1750 2750 2900 2750
 Wire Wire Line
 	1500 2450 1800 2450
@@
 	2350 7850 2350 7950
 Wire Wire Line
-	1800 2150 2900 2150
+	1750 2150 2950 2150
 Connection ~ 2900 2150
 Wire Bus Line
@@
 Connection ~ 2900 2750
 Wire Wire Line
-	3400 2750 4500 2750
+	3350 2750 4500 2750
 Wire Wire Line
 	3100 2450 3400 2450
@@
 	3950 7850 3950 7950
 Wire Wire Line
-	3400 2150 4500 2150
+	3350 2150 4550 2150
 Connection ~ 4500 2150
 Wire Bus Line
@@
 Connection ~ 4500 2750
 Wire Wire Line
-	5000 2750 6100 2750
+	4950 2750 6100 2750
 Wire Wire Line
 	4700 2450 5000 2450
@@
 	5550 7850 5550 7950
 Wire Wire Line
-	5000 2150 6100 2150
+	4950 2150 6150 2150
 Connection ~ 6100 2150
 Wire Wire Line
@@
 Connection ~ 6100 2750
 Wire Wire Line
-	9300 2750 8150 2750
+	8100 2750 9300 2750
 Wire Wire Line
 	7900 2450 8150 2450
@@
 	8750 7850 8750 7950
 Wire Wire Line
-	8200 2150 9300 2150
+	8150 2150 9300 2150
 Connection ~ 9100 2150
 Wire Wire Line
@@
 Connection ~ 8200 1850
 Wire Wire Line
-	7700 2750 6550 2750
+	6500 2750 7700 2750
 Wire Wire Line
 	6300 2450 6550 2450
@@
 	7150 7850 7150 7950
 Wire Wire Line
-	6600 2150 7700 2150
+	6550 2150 7700 2150
 Connection ~ 7500 2150
 Wire Wire Line
@@
 	10500 2750 10500 4750
 Wire Wire Line
-	10500 2750 9750 2750
+	9700 2750 10500 2750
 Wire Wire Line
 	9750 2450 9500 2450
@@
 	11700 2750 11700 4750
 Wire Wire Line
-	11700 2750 10950 2750
+	10900 2750 11700 2750
 Wire Wire Line
 	10950 2450 10700 2450
@@
 	12900 2750 12900 4750
 Wire Wire Line
-	12900 2750 12150 2750
+	12100 2750 12900 2750
 Wire Wire Line
 	12150 2450 11900 2450
@@
 	14100 2750 14100 4750
 Wire Wire Line
-	14100 2750 13350 2750
+	13300 2750 14100 2750
 Wire Wire Line
 	13350 2450 13100 2450
@@
 	15300 2750 15300 4750
 Wire Wire Line
-	15300 2750 14550 2750
+	14500 2750 15300 2750
 Wire Wire Line
 	14550 2450 14300 2450
@@
 F 0 "RV201" V 1625 2000 50  0000 C CNN
 F 1 "POT" V 1700 2000 50  0000 C CNN
-F 2 "" H 1800 2000 50  0001 C CNN
+F 2 "MATHSTERK:Pot" H 1800 2000 50  0001 C CNN
 F 3 "" V 1625 2000 50  0001 C CNN
 F 4 "RK09D1130A1L" V 1725 2100 60  0001 C CNN "part_num"
@@
 F 0 "RV203" V 2725 2000 50  0000 C CNN
 F 1 "POT" V 2800 2000 50  0000 C CNN
-F 2 "" H 2900 2000 50  0001 C CNN
+F 2 "MATHSTERK:Pot" H 2900 2000 50  0001 C CNN
 F 3 "" V 2725 2000 50  0001 C CNN
 F 4 "RK09D1130A1L" V 2825 2100 60  0001 C CNN "part_num"
@@
 F 0 "RV206" V 4325 2000 50  0000 C CNN
 F 1 "POT" V 4400 2000 50  0000 C CNN
-F 2 "" H 4500 2000 50  0001 C CNN
+F 2 "MATHSTERK:Pot" H 4500 2000 50  0001 C CNN
 F 3 "" V 4325 2000 50  0001 C CNN
 F 4 "RK09D1130A1L" V 4425 2100 60  0001 C CNN "part_num"
@@
 F 0 "RV209" V 5925 2000 50  0000 C CNN
 F 1 "POT" V 6000 2000 50  0000 C CNN
-F 2 "" H 6100 2000 50  0001 C CNN
+F 2 "MATHSTERK:Pot" H 6100 2000 50  0001 C CNN
 F 3 "" V 5925 2000 50  0001 C CNN
 F 4 "RK09D1130A1L" V 6025 2100 60  0001 C CNN "part_num"
@@
 F 0 "RV204" V 3225 2000 50  0000 C CNN
 F 1 "POT" V 3300 2000 50  0000 C CNN
-F 2 "" H 3400 2000 50  0001 C CNN
+F 2 "MATHSTERK:Pot" H 3400 2000 50  0001 C CNN
 F 3 "" V 3225 2000 50  0001 C CNN
 F 4 "RK09D1130A1L" V 3325 2100 60  0001 C CNN "part_num"
@@
 F 0 "RV207" V 4825 2000 50  0000 C CNN
 F 1 "POT" V 4900 2000 50  0000 C CNN
-F 2 "" H 5000 2000 50  0001 C CNN
+F 2 "MATHSTERK:Pot" H 5000 2000 50  0001 C CNN
 F 3 "" V 4825 2000 50  0001 C CNN
 F 4 "RK09D1130A1L" V 4925 2100 60  0001 C CNN "part_num"
@@
 F 0 "RV211" V 6425 2000 50  0000 C CNN
 F 1 "POT" V 6500 2000 50  0000 C CNN
-F 2 "" H 6600 2000 50  0001 C CNN
+F 2 "MATHSTERK:Pot" H 6600 2000 50  0001 C CNN
 F 3 "" V 6425 2000 50  0001 C CNN
 F 4 "RK09D1130A1L" V 6525 2100 60  0001 C CNN "part_num"
@@
 F 0 "RV213" V 7325 2000 50  0000 C CNN
 F 1 "POT" V 7400 2000 50  0000 C CNN
-F 2 "" H 7500 2000 50  0001 C CNN
+F 2 "MATHSTERK:Pot" H 7500 2000 50  0001 C CNN
 F 3 "" V 7325 2000 50  0001 C CNN
 F 4 "RK09D1130A1L" V 7425 2100 60  0001 C CNN "part_num"
@@
 F 0 "RV212" V 7275 1500 50  0000 C CNN
 F 1 "POT" V 7350 1500 50  0000 C CNN
-F 2 "" H 7450 1500 50  0001 C CNN
+F 2 "MATHSTERK:Pot" H 7450 1500 50  0001 C CNN
 F 3 "" V 7275 1500 50  0001 C CNN
 F 4 "RK09D1130A1L" V 7375 1600 60  0001 C CNN "part_num"
@@
 F 0 "RV216" V 8875 1500 50  0000 C CNN
 F 1 "POT" V 8950 1500 50  0000 C CNN
-F 2 "" H 9050 1500 50  0001 C CNN
+F 2 "MATHSTERK:Pot" H 9050 1500 50  0001 C CNN
 F 3 "" V 8875 1500 50  0001 C CNN
 F 4 "RK09D1130A1L" V 8975 1600 60  0001 C CNN "part_num"
@@
 F 0 "RV217" V 8925 2000 50  0000 C CNN
 F 1 "POT" V 9000 2000 50  0000 C CNN
-F 2 "" H 9100 2000 50  0001 C CNN
+F 2 "MATHSTERK:Pot" H 9100 2000 50  0001 C CNN
 F 3 "" V 8925 2000 50  0001 C CNN
 F 4 "RK09D1130A1L" V 9025 2100 60  0001 C CNN "part_num"
@@
 F 0 "RV215" V 8025 2000 50  0000 C CNN
 F 1 "POT" V 8100 2000 50  0000 C CNN
-F 2 "" H 8200 2000 50  0001 C CNN
+F 2 "MATHSTERK:Pot" H 8200 2000 50  0001 C CNN
 F 3 "" V 8025 2000 50  0001 C CNN
 F 4 "RK09D1130A1L" V 8125 2100 60  0001 C CNN "part_num"
@@
 	1    0    0    -1
 $EndComp
+Connection ~ 1800 2150
+Connection ~ 1800 2750
+Connection ~ 3400 2750
+Connection ~ 3400 2150
+Connection ~ 5000 2150
+Connection ~ 5000 2750
+Connection ~ 6600 2150
+Connection ~ 6550 2750
+Connection ~ 7550 2150
+Connection ~ 7500 1650
+Connection ~ 9150 2150
+Connection ~ 9100 1650
+Connection ~ 8200 2150
+Connection ~ 8150 2750
+Connection ~ 9750 2750
+Connection ~ 10950 2750
+Connection ~ 12150 2750
+Connection ~ 13350 2750
+Connection ~ 14550 2750
 $EndSCHEMATC

Commit message: testing
Parts:
- SW201, SW202, SW203, SW204, SW205, SW206, SW207, SW208, SW209, SW210, SW211, SW212, SW213, SW214, SW215, SW216, SW217, SW218, SW219, SW220, SW221, SW222, SW223, SW224, SW225, SW226, SW227, SW228, SW229, SW230, SW231, SW232, SW233, SW234, SW235, SW236, SW237, SW238, SW239, SW240, SW241, SW242, SW243, SW244, SW245, SW246, SW247, SW248, SW249, SW250, SW251, SW252, SW253, SW254, SW255: part_num (none) -> MHPS2285
