File: Projects/Voicemeeter/file5AE5FE21.sch (KiCad schematic (older format))
At the start: 22 parts

Commit message: stuff
Parts:
- renumbered C301 to C1, C310 to C10, C311 to C11, C312 to C12, C313 to C13, C314 to C14, C315 to C15, C316 to C16, C317 to C17, C318 to C18, C319 to C19, C302 to C2, C320 to C20, C321 to C21, C322 to C22, C303 to C3, C304 to C4, C305 to C5, C306 to C6, C307 to C7, C308 to C8, C309 to C9
Changed lines of the file:
@@
 Connection ~ 5850 1150
 $Comp
-L C C302
+L C C2
 U 1 1 5AE99D8A
 P 5450 1150
-F 0 "C302" H 5475 1250 50  0000 L CNN
+F 0 "C2" H 5475 1250 50  0000 L CNN
 F 1 "10uF" H 5475 1050 50  0000 L CNN
 F 2 "Capacitors_SMD:C_1206_HandSoldering" H 5488 1000 50  0001 C CNN
@@
 $EndComp
 $Comp
-L C C301
+L C C1
 U 1 1 5AE99D90
 P 5450 850
-F 0 "C301" H 5475 950 50  0000 L CNN
+F 0 "C1" H 5475 950 50  0000 L CNN
 F 1 "10uF" H 5475 750 50  0000 L CNN
 F 2 "Capacitors_SMD:C_1206_HandSoldering" H 5488 700 50  0001 C CNN
@@
 Connection ~ 5850 1750
 $Comp
-L C C304
+L C C4
 U 1 1 5AEBEF8D
 P 5450 1750
-F 0 "C304" H 5475 1850 50  0000 L CNN
+F 0 "C4" H 5475 1850 50  0000 L CNN
 F 1 "10uF" H 5475 1650 50  0000 L CNN
 F 2 "Capacitors_SMD:C_1206_HandSoldering" H 5488 1600 50  0001 C CNN
@@
 $EndComp
 $Comp
-L C C303
+L C C3
 U 1 1 5AEBEF93
 P 5450 1450
-F 0 "C303" H 5475 1550 50  0000 L CNN
+F 0 "C3" H 5475 1550 50  0000 L CNN
 F 1 "10uF" H 5475 1350 50  0000 L CNN
 F 2 "Capacitors_SMD:C_1206_HandSoldering" H 5488 1300 50  0001 C CNN
@@
 Connection ~ 5850 2350
 $Comp
-L C C306
+L C C6
 U 1 1 5AEBF031
 P 5450 2350
-F 0 "C306" H 5475 2450 50  0000 L CNN
+F 0 "C6" H 5475 2450 50  0000 L CNN
 F 1 "10uF" H 5475 2250 50  0000 L CNN
 F 2 "Capacitors_SMD:C_1206_HandSoldering" H 5488 2200 50  0001 C CNN
@@
 $EndComp
 $Comp
-L C C305
+L C C5
 U 1 1 5AEBF037
 P 5450 2050
-F 0 "C305" H 5475 2150 50  0000 L CNN
+F 0 "C5" H 5475 2150 50  0000 L CNN
 F 1 "10uF" H 5475 1950 50  0000 L CNN
 F 2 "Capacitors_SMD:C_1206_HandSoldering" H 5488 1900 50  0001 C CNN
@@
 Connection ~ 5850 2650
 $Comp
-L C C307
+L C C7
 U 1 1 5AEBF1CC
 P 5450 2650
-F 0 "C307" H 5475 2750 50  0000 L CNN
+F 0 "C7" H 5475 2750 50  0000 L CNN
 F 1 "10uF" H 5475 2550 50  0000 L CNN
 F 2 "Capacitors_SMD:C_1206_HandSoldering" H 5488 2500 50  0001 C CNN
@@
 Connection ~ 5850 3250
 $Comp
-L C C309
+L C C9
 U 1 1 5AEBF1D7
 P 5450 3250
-F 0 "C309" H 5475 3350 50  0000 L CNN
+F 0 "C9" H 5475 3350 50  0000 L CNN
 F 1 "10uF" H 5475 3150 50  0000 L CNN
 F 2 "Capacitors_SMD:C_1206_HandSoldering" H 5488 3100 50  0001 C CNN
@@
 $EndComp
 $Comp
-L C C308
+L C C8
 U 1 1 5AEBF1DD
 P 5450 2950
-F 0 "C308" H 5475 3050 50  0000 L CNN
+F 0 "C8" H 5475 3050 50  0000 L CNN
 F 1 "10uF" H 5475 2850 50  0000 L CNN
 F 2 "Capacitors_SMD:C_1206_HandSoldering" H 5488 2800 50  0001 C CNN
@@
 Connection ~ 5850 3850
 $Comp
-L C C311
+L C C11
 U 1 1 5AEBF1EA
 P 5450 3850
-F 0 "C311" H 5475 3950 50  0000 L CNN
+F 0 "C11" H 5475 3950 50  0000 L CNN
 F 1 "10uF" H 5475 3750 50  0000 L CNN
 F 2 "Capacitors_SMD:C_1206_HandSoldering" H 5488 3700 50  0001 C CNN
@@
 $EndComp
 $Comp
-L C C310
+L C C10
 U 1 1 5AEBF1F0
 P 5450 3550
-F 0 "C310" H 5475 3650 50  0000 L CNN
+F 0 "C10" H 5475 3650 50  0000 L CNN
 F 1 "10uF" H 5475 3450 50  0000 L CNN
 F 2 "Capacitors_SMD:C_1206_HandSoldering" H 5488 3400 50  0001 C CNN
@@
 Connection ~ 5850 4150
 $Comp
-L C C312
+L C C12
 U 1 1 5AEBF4BD
 P 5450 4150
-F 0 "C312" H 5475 4250 50  0000 L CNN
+F 0 "C12" H 5475 4250 50  0000 L CNN
 F 1 "10uF" H 5475 4050 50  0000 L CNN
 F 2 "Capacitors_SMD:C_1206_HandSoldering" H 5488 4000 50  0001 C CNN
@@
 Connection ~ 5850 4750
 $Comp
-L C C314
+L C C14
 U 1 1 5AEBF4C8
 P 5450 4750
-F 0 "C314" H 5475 4850 50  0000 L CNN
+F 0 "C14" H 5475 4850 50  0000 L CNN
 F 1 "10uF" H 5475 4650 50  0000 L CNN
 F 2 "Capacitors_SMD:C_1206_HandSoldering" H 5488 4600 50  0001 C CNN
@@
 $EndComp
 $Comp
-L C C313
+L C C13
 U 1 1 5AEBF4CE
 P 5450 4450
-F 0 "C313" H 5475 4550 50  0000 L CNN
+F 0 "C13" H 5475 4550 50  0000 L CNN
 F 1 "10uF" H 5475 4350 50  0000 L CNN
 F 2 "Capacitors_SMD:C_1206_HandSoldering" H 5488 4300 50  0001 C CNN
@@
 Connection ~ 5850 5350
 $Comp
-L C C316
+L C C16
 U 1 1 5AEBF4DB
 P 5450 5350
-F 0 "C316" H 5475 5450 50  0000 L CNN
+F 0 "C16" H 5475 5450 50  0000 L CNN
 F 1 "10uF" H 5475 5250 50  0000 L CNN
 F 2 "Capacitors_SMD:C_1206_HandSoldering" H 5488 5200 50  0001 C CNN
@@
 $EndComp
 $Comp
-L C C315
+L C C15
 U 1 1 5AEBF4E1
 P 5450 5050
-F 0 "C315" H 5475 5150 50  0000 L CNN
+F 0 "C15" H 5475 5150 50  0000 L CNN
 F 1 "10uF" H 5475 4950 50  0000 L CNN
 F 2 "Capacitors_SMD:C_1206_HandSoldering" H 5488 4900 50  0001 C CNN
@@
 Connection ~ 5850 5650
 $Comp
-L C C317
+L C C17
 U 1 1 5AEBF4EC
 P 5450 5650
-F 0 "C317" H 5475 5750 50  0000 L CNN
+F 0 "C17" H 5475 5750 50  0000 L CNN
 F 1 "10uF" H 5475 5550 50  0000 L CNN
 F 2 "Capacitors_SMD:C_1206_HandSoldering" H 5488 5500 50  0001 C CNN
@@
 Connection ~ 5850 6250
 $Comp
-L C C319
+L C C19
 U 1 1 5AEBF4F7
 P 5450 6250
-F 0 "C319" H 5475 6350 50  0000 L CNN
+F 0 "C19" H 5475 6350 50  0000 L CNN
 F 1 "10uF" H 5475 6150 50  0000 L CNN
 F 2 "Capacitors_SMD:C_1206_HandSoldering" H 5488 6100 50  0001 C CNN
@@
 $EndComp
 $Comp
-L C C318
+L C C18
 U 1 1 5AEBF4FD
 P 5450 5950
-F 0 "C318" H 5475 6050 50  0000 L CNN
+F 0 "C18" H 5475 6050 50  0000 L CNN
 F 1 "10uF" H 5475 5850 50  0000 L CNN
 F 2 "Capacitors_SMD:C_1206_HandSoldering" H 5488 5800 50  0001 C CNN
@@
 Connection ~ 5850 6850
 $Comp
-L C C321
+L C C21
 U 1 1 5AEBF50A
 P 5450 6850
-F 0 "C321" H 5475 6950 50  0000 L CNN
+F 0 "C21" H 5475 6950 50  0000 L CNN
 F 1 "10uF" H 5475 6750 50  0000 L CNN
 F 2 "Capacitors_SMD:C_1206_HandSoldering" H 5488 6700 50  0001 C CNN
@@
 $EndComp
 $Comp
-L C C320
+L C C20
 U 1 1 5AEBF510
 P 5450 6550
-F 0 "C320" H 5475 6650 50  0000 L CNN
+F 0 "C20" H 5475 6650 50  0000 L CNN
 F 1 "10uF" H 5475 6450 50  0000 L CNN
 F 2 "Capacitors_SMD:C_1206_HandSoldering" H 5488 6400 50  0001 C CNN
@@
 Connection ~ 5850 6550
 $Comp
-L C C322
+L C C22
 U 1 1 5AEBF8EB
 P 5450 7150
-F 0 "C322" H 5475 7250 50  0000 L CNN
+F 0 "C22" H 5475 7250 50  0000 L CNN
 F 1 "10uF" H 5475 7050 50  0000 L CNN
 F 2 "Capacitors_SMD:C_1206_HandSoldering" H 5488 7000 50  0001 C CNN
@@
 	5300 7150 4400 7150
 $Comp
-L GND #PWR021
+L GND #PWR21
 U 1 1 5AEC0528
 P 5850 7200
-F 0 "#PWR021" H 5850 6950 50  0001 C CNN
+F 0 "#PWR21" H 5850 6950 50  0001 C CNN
 F 1 "GND" H 5850 7050 50  0000 C CNN
 F 2 "" H 5850 7200 50  0001 C CNN

Commit message: Zzzzz
Parts:
- renumbered C1 to C301, C2 to C302, C3 to C303, C4 to C304, C5 to C305, C6 to C306, C7 to C307, C8 to C308, C9 to C309, C10 to C310, C11 to C311, C12 to C312, C13 to C313, C14 to C314, C15 to C315, C16 to C316, C17 to C317, C18 to C318, C19 to C319, C20 to C320, C21 to C321, C22 to C322
Changed lines of the file:
@@
 Connection ~ 5850 1150
 $Comp
-L C C2
+L C C302
 U 1 1 5AE99D8A
 P 5450 1150
-F 0 "C2" H 5475 1250 50  0000 L CNN
+F 0 "C302" H 5475 1250 50  0000 L CNN
 F 1 "10uF" H 5475 1050 50  0000 L CNN
 F 2 "Capacitors_SMD:C_1206_HandSoldering" H 5488 1000 50  0001 C CNN
@@
 $EndComp
 $Comp
-L C C1
+L C C301
 U 1 1 5AE99D90
 P 5450 850
-F 0 "C1" H 5475 950 50  0000 L CNN
+F 0 "C301" H 5475 950 50  0000 L CNN
 F 1 "10uF" H 5475 750 50  0000 L CNN
 F 2 "Capacitors_SMD:C_1206_HandSoldering" H 5488 700 50  0001 C CNN
@@
 Connection ~ 5850 1750
 $Comp
-L C C4
+L C C304
 U 1 1 5AEBEF8D
 P 5450 1750
-F 0 "C4" H 5475 1850 50  0000 L CNN
+F 0 "C304" H 5475 1850 50  0000 L CNN
 F 1 "10uF" H 5475 1650 50  0000 L CNN
 F 2 "Capacitors_SMD:C_1206_HandSoldering" H 5488 1600 50  0001 C CNN
@@
 $EndComp
 $Comp
-L C C3
+L C C303
 U 1 1 5AEBEF93
 P 5450 1450
-F 0 "C3" H 5475 1550 50  0000 L CNN
+F 0 "C303" H 5475 1550 50  0000 L CNN
 F 1 "10uF" H 5475 1350 50  0000 L CNN
 F 2 "Capacitors_SMD:C_1206_HandSoldering" H 5488 1300 50  0001 C CNN
@@
 Connection ~ 5850 2350
 $Comp
-L C C6
+L C C306
 U 1 1 5AEBF031
 P 5450 2350
-F 0 "C6" H 5475 2450 50  0000 L CNN
+F 0 "C306" H 5475 2450 50  0000 L CNN
 F 1 "10uF" H 5475 2250 50  0000 L CNN
 F 2 "Capacitors_SMD:C_1206_HandSoldering" H 5488 2200 50  0001 C CNN
@@
 $EndComp
 $Comp
-L C C5
+L C C305
 U 1 1 5AEBF037
 P 5450 2050
-F 0 "C5" H 5475 2150 50  0000 L CNN
+F 0 "C305" H 5475 2150 50  0000 L CNN
 F 1 "10uF" H 5475 1950 50  0000 L CNN
 F 2 "Capacitors_SMD:C_1206_HandSoldering" H 5488 1900 50  0001 C CNN
@@
 Connection ~ 5850 2650
 $Comp
-L C C7
+L C C307
 U 1 1 5AEBF1CC
 P 5450 2650
-F 0 "C7" H 5475 2750 50  0000 L CNN
+F 0 "C307" H 5475 2750 50  0000 L CNN
 F 1 "10uF" H 5475 2550 50  0000 L CNN
 F 2 "Capacitors_SMD:C_1206_HandSoldering" H 5488 2500 50  0001 C CNN
@@
 Connection ~ 5850 3250
 $Comp
-L C C9
+L C C309
 U 1 1 5AEBF1D7
 P 5450 3250
-F 0 "C9" H 5475 3350 50  0000 L CNN
+F 0 "C309" H 5475 3350 50  0000 L CNN
 F 1 "10uF" H 5475 3150 50  0000 L CNN
 F 2 "Capacitors_SMD:C_1206_HandSoldering" H 5488 3100 50  0001 C CNN
@@
 $EndComp
 $Comp
-L C C8
+L C C308
 U 1 1 5AEBF1DD
 P 5450 2950
-F 0 "C8" H 5475 3050 50  0000 L CNN
+F 0 "C308" H 5475 3050 50  0000 L CNN
 F 1 "10uF" H 5475 2850 50  0000 L CNN
 F 2 "Capacitors_SMD:C_1206_HandSoldering" H 5488 2800 50  0001 C CNN
@@
 Connection ~ 5850 3850
 $Comp
-L C C11
+L C C311
 U 1 1 5AEBF1EA
 P 5450 3850
-F 0 "C11" H 5475 3950 50  0000 L CNN
+F 0 "C311" H 5475 3950 50  0000 L CNN
 F 1 "10uF" H 5475 3750 50  0000 L CNN
 F 2 "Capacitors_SMD:C_1206_HandSoldering" H 5488 3700 50  0001 C CNN
@@
 $EndComp
 $Comp
-L C C10
+L C C310
 U 1 1 5AEBF1F0
 P 5450 3550
-F 0 "C10" H 5475 3650 50  0000 L CNN
+F 0 "C310" H 5475 3650 50  0000 L CNN
 F 1 "10uF" H 5475 3450 50  0000 L CNN
 F 2 "Capacitors_SMD:C_1206_HandSoldering" H 5488 3400 50  0001 C CNN
@@
 Connection ~ 5850 4150
 $Comp
-L C C12
+L C C312
 U 1 1 5AEBF4BD
 P 5450 4150
-F 0 "C12" H 5475 4250 50  0000 L CNN
+F 0 "C312" H 5475 4250 50  0000 L CNN
 F 1 "10uF" H 5475 4050 50  0000 L CNN
 F 2 "Capacitors_SMD:C_1206_HandSoldering" H 5488 4000 50  0001 C CNN
@@
 Connection ~ 5850 4750
 $Comp
-L C C14
+L C C314
 U 1 1 5AEBF4C8
 P 5450 4750
-F 0 "C14" H 5475 4850 50  0000 L CNN
+F 0 "C314" H 5475 4850 50  0000 L CNN
 F 1 "10uF" H 5475 4650 50  0000 L CNN
 F 2 "Capacitors_SMD:C_1206_HandSoldering" H 5488 4600 50  0001 C CNN
@@
 $EndComp
 $Comp
-L C C13
+L C C313
 U 1 1 5AEBF4CE
 P 5450 4450
-F 0 "C13" H 5475 4550 50  0000 L CNN
+F 0 "C313" H 5475 4550 50  0000 L CNN
 F 1 "10uF" H 5475 4350 50  0000 L CNN
 F 2 "Capacitors_SMD:C_1206_HandSoldering" H 5488 4300 50  0001 C CNN
@@
 Connection ~ 5850 5350
 $Comp
-L C C16
+L C C316
 U 1 1 5AEBF4DB
 P 5450 5350
-F 0 "C16" H 5475 5450 50  0000 L CNN
+F 0 "C316" H 5475 5450 50  0000 L CNN
 F 1 "10uF" H 5475 5250 50  0000 L CNN
 F 2 "Capacitors_SMD:C_1206_HandSoldering" H 5488 5200 50  0001 C CNN
@@
 $EndComp
 $Comp
-L C C15
+L C C315
 U 1 1 5AEBF4E1
 P 5450 5050
-F 0 "C15" H 5475 5150 50  0000 L CNN
+F 0 "C315" H 5475 5150 50  0000 L CNN
 F 1 "10uF" H 5475 4950 50  0000 L CNN
 F 2 "Capacitors_SMD:C_1206_HandSoldering" H 5488 4900 50  0001 C CNN
@@
 Connection ~ 5850 5650
 $Comp
-L C C17
+L C C317
 U 1 1 5AEBF4EC
 P 5450 5650
-F 0 "C17" H 5475 5750 50  0000 L CNN
+F 0 "C317" H 5475 5750 50  0000 L CNN
 F 1 "10uF" H 5475 5550 50  0000 L CNN
 F 2 "Capacitors_SMD:C_1206_HandSoldering" H 5488 5500 50  0001 C CNN
@@
 Connection ~ 5850 6250
 $Comp
-L C C19
+L C C319
 U 1 1 5AEBF4F7
 P 5450 6250
-F 0 "C19" H 5475 6350 50  0000 L CNN
+F 0 "C319" H 5475 6350 50  0000 L CNN
 F 1 "10uF" H 5475 6150 50  0000 L CNN
 F 2 "Capacitors_SMD:C_1206_HandSoldering" H 5488 6100 50  0001 C CNN
@@
 $EndComp
 $Comp
-L C C18
+L C C318
 U 1 1 5AEBF4FD
 P 5450 5950
-F 0 "C18" H 5475 6050 50  0000 L CNN
+F 0 "C318" H 5475 6050 50  0000 L CNN
 F 1 "10uF" H 5475 5850 50  0000 L CNN
 F 2 "Capacitors_SMD:C_1206_HandSoldering" H 5488 5800 50  0001 C CNN
@@
 Connection ~ 5850 6850
 $Comp
-L C C21
+L C C321
 U 1 1 5AEBF50A
 P 5450 6850
-F 0 "C21" H 5475 6950 50  0000 L CNN
+F 0 "C321" H 5475 6950 50  0000 L CNN
 F 1 "10uF" H 5475 6750 50  0000 L CNN
 F 2 "Capacitors_SMD:C_1206_HandSoldering" H 5488 6700 50  0001 C CNN
@@
 $EndComp
 $Comp
-L C C20
+L C C320
 U 1 1 5AEBF510
 P 5450 6550
-F 0 "C20" H 5475 6650 50  0000 L CNN
+F 0 "C320" H 5475 6650 50  0000 L CNN
 F 1 "10uF" H 5475 6450 50  0000 L CNN
 F 2 "Capacitors_SMD:C_1206_HandSoldering" H 5488 6400 50  0001 C CNN
@@
 Connection ~ 5850 6550
 $Comp
-L C C22
+L C C322
 U 1 1 5AEBF8EB
 P 5450 7150
-F 0 "C22" H 5475 7250 50  0000 L CNN
+F 0 "C322" H 5475 7250 50  0000 L CNN
 F 1 "10uF" H 5475 7050 50  0000 L CNN
 F 2 "Capacitors_SMD:C_1206_HandSoldering" H 5488 7000 50  0001 C CNN
@@
 	5300 7150 4400 7150
 $Comp
-L GND #PWR21
+L GND #PWR021
 U 1 1 5AEC0528
 P 5850 7200
-F 0 "#PWR21" H 5850 6950 50  0001 C CNN
+F 0 "#PWR021" H 5850 6950 50  0001 C CNN
 F 1 "GND" H 5850 7050 50  0000 C CNN
 F 2 "" H 5850 7200 50  0001 C CNN

Commit message: ASDASD
Parts:
- C301, C302, C303, C304, C305, C306, C307, C308, C309, C310, C311, C312, C313, C314, C315, C316, C317, C318, C319, C320, C321, C322: footprint Capacitors_SMD:C_1206_HandSoldering -> (none); part_num (none) -> C0603C106M8PACTU

Commit message: why did a lock file sneak in? <.<
Parts:
- C301, C302, C303, C304, C305, C306, C307, C308, C309, C310, C311, C312, C313, C314, C315, C316, C317, C318, C319, C320, C321, C322: footprint (none) -> Capacitors_SMD:C_0603_HandSoldering
Changed lines of the file:
@@
 F 0 "C301" H 5475 950 50  0000 L CNN
 F 1 "10uF" H 5475 750 50  0000 L CNN
-F 2 "" H 5488 700 50  0001 C CNN
+F 2 "Capacitors_SMD:C_0603_HandSoldering" H 5488 700 50  0001 C CNN
 F 3 "" H 5475 950 50  0001 C CNN
 F 4 "C0603C106M8PACTU" H 5575 1050 60  0001 C CNN "part_num"
@@
 F 0 "C302" H 5475 1250 50  0000 L CNN
 F 1 "10uF" H 5475 1050 50  0000 L CNN
-F 2 "" H 5488 1000 50  0001 C CNN
+F 2 "Capacitors_SMD:C_0603_HandSoldering" H 5488 1000 50  0001 C CNN
 F 3 "" H 5475 1250 50  0001 C CNN
 F 4 "C0603C106M8PACTU" H 5575 1350 60  0001 C CNN "part_num"
@@
 F 0 "C303" H 5475 1550 50  0000 L CNN
 F 1 "10uF" H 5475 1350 50  0000 L CNN
-F 2 "" H 5488 1300 50  0001 C CNN
+F 2 "Capacitors_SMD:C_0603_HandSoldering" H 5488 1300 50  0001 C CNN
 F 3 "" H 5475 1550 50  0001 C CNN
 F 4 "C0603C106M8PACTU" H 5575 1650 60  0001 C CNN "part_num"
@@
 F 0 "C304" H 5475 1850 50  0000 L CNN
 F 1 "10uF" H 5475 1650 50  0000 L CNN
-F 2 "" H 5488 1600 50  0001 C CNN
+F 2 "Capacitors_SMD:C_0603_HandSoldering" H 5488 1600 50  0001 C CNN
 F 3 "" H 5475 1850 50  0001 C CNN
 F 4 "C0603C106M8PACTU" H 5575 1950 60  0001 C CNN "part_num"
@@
 F 0 "C305" H 5475 2150 50  0000 L CNN
 F 1 "10uF" H 5475 1950 50  0000 L CNN
-F 2 "" H 5488 1900 50  0001 C CNN
+F 2 "Capacitors_SMD:C_0603_HandSoldering" H 5488 1900 50  0001 C CNN
 F 3 "" H 5475 2150 50  0001 C CNN
 F 4 "C0603C106M8PACTU" H 5575 2250 60  0001 C CNN "part_num"
@@
 F 0 "C306" H 5475 2450 50  0000 L CNN
 F 1 "10uF" H 5475 2250 50  0000 L CNN
-F 2 "" H 5488 2200 50  0001 C CNN
+F 2 "Capacitors_SMD:C_0603_HandSoldering" H 5488 2200 50  0001 C CNN
 F 3 "" H 5475 2450 50  0001 C CNN
 F 4 "C0603C106M8PACTU" H 5575 2550 60  0001 C CNN "part_num"
@@
 F 0 "C307" H 5475 2750 50  0000 L CNN
 F 1 "10uF" H 5475 2550 50  0000 L CNN
-F 2 "" H 5488 2500 50  0001 C CNN
+F 2 "Capacitors_SMD:C_0603_HandSoldering" H 5488 2500 50  0001 C CNN
 F 3 "" H 5475 2750 50  0001 C CNN
 F 4 "C0603C106M8PACTU" H 5575 2850 60  0001 C CNN "part_num"
@@
 F 0 "C308" H 5475 3050 50  0000 L CNN
 F 1 "10uF" H 5475 2850 50  0000 L CNN
-F 2 "" H 5488 2800 50  0001 C CNN
+F 2 "Capacitors_SMD:C_0603_HandSoldering" H 5488 2800 50  0001 C CNN
 F 3 "" H 5475 3050 50  0001 C CNN
 F 4 "C0603C106M8PACTU" H 5575 3150 60  0001 C CNN "part_num"
@@
 F 0 "C309" H 5475 3350 50  0000 L CNN
 F 1 "10uF" H 5475 3150 50  0000 L CNN
-F 2 "" H 5488 3100 50  0001 C CNN
+F 2 "Capacitors_SMD:C_0603_HandSoldering" H 5488 3100 50  0001 C CNN
 F 3 "" H 5475 3350 50  0001 C CNN
 F 4 "C0603C106M8PACTU" H 5575 3450 60  0001 C CNN "part_num"
@@
 F 0 "C310" H 5475 3650 50  0000 L CNN
 F 1 "10uF" H 5475 3450 50  0000 L CNN
-F 2 "" H 5488 3400 50  0001 C CNN
+F 2 "Capacitors_SMD:C_0603_HandSoldering" H 5488 3400 50  0001 C CNN
 F 3 "" H 5475 3650 50  0001 C CNN
 F 4 "C0603C106M8PACTU" H 5575 3750 60  0001 C CNN "part_num"
@@
 F 0 "C311" H 5475 3950 50  0000 L CNN
 F 1 "10uF" H 5475 3750 50  0000 L CNN
-F 2 "" H 5488 3700 50  0001 C CNN
+F 2 "Capacitors_SMD:C_0603_HandSoldering" H 5488 3700 50  0001 C CNN
 F 3 "" H 5475 3950 50  0001 C CNN
 F 4 "C0603C106M8PACTU" H 5575 4050 60  0001 C CNN "part_num"
@@
 F 0 "C312" H 5475 4250 50  0000 L CNN
 F 1 "10uF" H 5475 4050 50  0000 L CNN
-F 2 "" H 5488 4000 50  0001 C CNN
+F 2 "Capacitors_SMD:C_0603_HandSoldering" H 5488 4000 50  0001 C CNN
 F 3 "" H 5475 4250 50  0001 C CNN
 F 4 "C0603C106M8PACTU" H 5575 4350 60  0001 C CNN "part_num"
@@
 F 0 "C313" H 5475 4550 50  0000 L CNN
 F 1 "10uF" H 5475 4350 50  0000 L CNN
-F 2 "" H 5488 4300 50  0001 C CNN
+F 2 "Capacitors_SMD:C_0603_HandSoldering" H 5488 4300 50  0001 C CNN
 F 3 "" H 5475 4550 50  0001 C CNN
 F 4 "C0603C106M8PACTU" H 5575 4650 60  0001 C CNN "part_num"
@@
 F 0 "C314" H 5475 4850 50  0000 L CNN
 F 1 "10uF" H 5475 4650 50  0000 L CNN
-F 2 "" H 5488 4600 50  0001 C CNN
+F 2 "Capacitors_SMD:C_0603_HandSoldering" H 5488 4600 50  0001 C CNN
 F 3 "" H 5475 4850 50  0001 C CNN
 F 4 "C0603C106M8PACTU" H 5575 4950 60  0001 C CNN "part_num"
@@
 F 0 "C315" H 5475 5150 50  0000 L CNN
 F 1 "10uF" H 5475 4950 50  0000 L CNN
-F 2 "" H 5488 4900 50  0001 C CNN
+F 2 "Capacitors_SMD:C_0603_HandSoldering" H 5488 4900 50  0001 C CNN
 F 3 "" H 5475 5150 50  0001 C CNN
 F 4 "C0603C106M8PACTU" H 5575 5250 60  0001 C CNN "part_num"
@@
 F 0 "C316" H 5475 5450 50  0000 L CNN
 F 1 "10uF" H 5475 5250 50  0000 L CNN
-F 2 "" H 5488 5200 50  0001 C CNN
+F 2 "Capacitors_SMD:C_0603_HandSoldering" H 5488 5200 50  0001 C CNN
 F 3 "" H 5475 5450 50  0001 C CNN
 F 4 "C0603C106M8PACTU" H 5575 5550 60  0001 C CNN "part_num"
@@
 F 0 "C317" H 5475 5750 50  0000 L CNN
 F 1 "10uF" H 5475 5550 50  0000 L CNN
-F 2 "" H 5488 5500 50  0001 C CNN
+F 2 "Capacitors_SMD:C_0603_HandSoldering" H 5488 5500 50  0001 C CNN
 F 3 "" H 5475 5750 50  0001 C CNN
 F 4 "C0603C106M8PACTU" H 5575 5850 60  0001 C CNN "part_num"
@@
 F 0 "C318" H 5475 6050 50  0000 L CNN
 F 1 "10uF" H 5475 5850 50  0000 L CNN
-F 2 "" H 5488 5800 50  0001 C CNN
+F 2 "Capacitors_SMD:C_0603_HandSoldering" H 5488 5800 50  0001 C CNN
 F 3 "" H 5475 6050 50  0001 C CNN
 F 4 "C0603C106M8PACTU" H 5575 6150 60  0001 C CNN "part_num"
@@
 F 0 "C319" H 5475 6350 50  0000 L CNN
 F 1 "10uF" H 5475 6150 50  0000 L CNN
-F 2 "" H 5488 6100 50  0001 C CNN
+F 2 "Capacitors_SMD:C_0603_HandSoldering" H 5488 6100 50  0001 C CNN
 F 3 "" H 5475 6350 50  0001 C CNN
 F 4 "C0603C106M8PACTU" H 5575 6450 60  0001 C CNN "part_num"
@@
 F 0 "C320" H 5475 6650 50  0000 L CNN
 F 1 "10uF" H 5475 6450 50  0000 L CNN
-F 2 "" H 5488 6400 50  0001 C CNN
+F 2 "Capacitors_SMD:C_0603_HandSoldering" H 5488 6400 50  0001 C CNN
 F 3 "" H 5475 6650 50  0001 C CNN
 F 4 "C0603C106M8PACTU" H 5575 6750 60  0001 C CNN "part_num"
@@
 F 0 "C321" H 5475 6950 50  0000 L CNN
 F 1 "10uF" H 5475 6750 50  0000 L CNN
-F 2 "" H 5488 6700 50  0001 C CNN
+F 2 "Capacitors_SMD:C_0603_HandSoldering" H 5488 6700 50  0001 C CNN
 F 3 "" H 5475 6950 50  0001 C CNN
 F 4 "C0603C106M8PACTU" H 5575 7050 60  0001 C CNN "part_num"
@@
 F 0 "C322" H 5475 7250 50  0000 L CNN
 F 1 "10uF" H 5475 7050 50  0000 L CNN
-F 2 "" H 5488 7000 50  0001 C CNN
+F 2 "Capacitors_SMD:C_0603_HandSoldering" H 5488 7000 50  0001 C CNN
 F 3 "" H 5475 7250 50  0001 C CNN
 F 4 "C0603C106M8PACTU" H 5575 7350 60  0001 C CNN "part_num"
