File: Projects/Voicemeeter/file5AE700A4.sch (KiCad schematic (older format))
At the start: 38 parts, among them J501 SPARE, J502 GS2, J503 Screw_Terminal_01x02, J504 GS2, J505 MIDI OUT, J506 MIDI IN, J507 DIN-5_180degree, J508 DIN-5_180degree, SW501 PEC11R-4215F-S0024, U501 stm32f103-china-MS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

Commit message: uuuuuugh
Parts:
- removed J503: Screw_Terminal_01x02, Connectors_Terminal_Blocks:TerminalBlock_Altech_AK300-2_P5.00mm, symbol Screw_Terminal_01x02
- added J503: GS2, MATHSTERK:SB2, symbol GS2
Connections:
- net at J501.5 (Pin_5): now also J503.2 (G2); no longer U501.12 (PB4)
- new net: J503.1 (G1), U501.12 (PB4)
Changed lines of the file:
@@
 $Descr A4 11693 8268
 encoding utf-8
-Sheet 5 6
+Sheet 5 7
 Title ""
 Date ""
@@
 	-1   0    0    1
 $EndComp
-$Comp
-L Screw_Terminal_01x02 J503
-U 1 1 5AF33E17
-P 3150 5050
-F 0 "J503" V 3150 5150 50  0000 C CNN
-F 1 "Screw_Terminal_01x02" V 3350 5050 50  0000 C CNN
-F 2 "Connectors_Terminal_Blocks:TerminalBlock_Altech_AK300-2_P5.00mm" H 3150 5050 50  0001 C CNN
-F 3 "" H 3150 5050 50  0001 C CNN
-	1    3150 5050
-	0    -1   -1   0
-$EndComp
 Entry Wire Line
 	2550 850  2650 750
@@
 	2600 5400 3600 5400
 Wire Wire Line
-	3150 5400 3150 5250
-Connection ~ 3150 5400
-Wire Wire Line
-	3250 5250 3250 5500
-Connection ~ 3250 5500
-Wire Wire Line
 	2400 5600 3600 5600
 Wire Wire Line
@@
 Wire Wire Line
 	3600 4750 3600 4900
-Wire Wire Line
-	2500 4100 4600 4100
 Wire Bus Line
 	3000 3800 1600 3800
@@
 	-1   0    0    1
 $EndComp
+$Comp
+L GS2 J503
+U 1 1 5AFB0685
+P 2800 4100
+F 0 "J503" H 2900 4250 50  0000 C CNN
+F 1 "GS2" H 2900 3951 50  0000 C CNN
+F 2 "MATHSTERK:SB2" V 2874 4100 50  0001 C CNN
+F 3 "" H 2800 4100 50  0001 C CNN
+	1    2800 4100
+	0    1    1    0
+$EndComp
+Wire Wire Line
+	2500 4100 2600 4100
+Wire Wire Line
+	3000 4100 4600 4100
 $EndSCHEMATC

Commit message: yes
Parts:
- removed RESET501: SW_Push, Buttons_Switches_THT:SW_PUSH-12mm, symbol SW_Push
Connections:
- net GND: now also U502.3; no longer U502.2
- net at D501.1 (K), J506.1 (Pin_1): now also U502.1; no longer U502.4
- net at D501.2 (A), J506.2 (Pin_2): now also U502.2; no longer U502.3
- net at R519.1, U501.27 (PA2): now also U502.4; no longer U502.1
- no-connect marks 16 -> 17
Changed lines of the file:
@@
 NoConn ~ 7000 5100
-$Comp
-L SW_Push RESET501
-U 1 1 5AE70367
-P 7450 2300
-F 0 "RESET501" V 7650 2350 50  0000 L CNN
-F 1 "SW_Push" H 7450 2240 50  0000 C CNN
-F 2 "Buttons_Switches_THT:SW_PUSH-12mm" H 7450 2500 50  0001 C CNN
-F 3 "" H 7450 2500 50  0001 C CNN
-	1    7450 2300
-	0    1    1    0
-$EndComp
 $Comp
 L +3V3 #PWR042
@@
 $EndComp
 Wire Wire Line
-	7000 2100 7450 2100
-Wire Wire Line
-	7000 2500 7450 2500
-Wire Wire Line
 	7000 2700 7700 2700
 Wire Wire Line
@@
 Wire Wire Line
 	7050 1900 7050 2100
-Connection ~ 7050 2100
 Wire Wire Line
 	8000 3700 7350 3700
@@
 F 4 "PC817X1NSZ1B" H 8800 5050 60  0001 C CNN "part_num"
 	1    8900 4750
-	1    0    0    -1
+	-1   0    0    -1
 $EndComp
 $Comp
@@
 Wire Wire Line
 	3000 4100 4600 4100
+NoConn ~ 7000 2500
+Wire Wire Line
+	7050 2100 7000 2100
 $EndSCHEMATC

Commit message: boop
Parts:
- added J?: Screw_Terminal_01x06, Connectors_Terminal_Blocks:TerminalBlock_bornier-6_P5.08mm, symbol Screw_Terminal_01x06
- added PSU?: IRM-45, MATHSTERK:IRM-45, symbol IRM-45
Connections:
- net +5V: now also PSU?.3 (5V)
- net GND: now also PSU?.4 (GND)
- new net: J?.6 (Pin_6), PSU?.1 (Live)
- new net: J?.5 (Pin_5), PSU?.2 (Neutral)
- new net: J?.1 (Pin_1), J?.4 (Pin_4)
- new net: J?.2 (Pin_2), J?.3 (Pin_3)
Changed lines of the file:
@@
 $Descr A4 11693 8268
 encoding utf-8
-Sheet 5 7
+Sheet 5 6
 Title ""
 Date ""
@@
 Wire Wire Line
 	7050 2100 7000 2100
+$Comp
+L IRM-45 PSU?
+U 1 1 5AF9DFFD
+P 3300 6850
+F 0 "PSU?" H 3200 6800 60  0000 C CNN
+F 1 "IRM-45" H 3200 6700 60  0000 C CNN
+F 2 "MATHSTERK:IRM-45" H 3300 6850 60  0001 C CNN
+F 3 "" H 3300 6850 60  0001 C CNN
+	1    3300 6850
+	1    0    0    -1
+$EndComp
+$Comp
+L +5V #PWR?
+U 1 1 5AF9E004
+P 3900 6950
+F 0 "#PWR?" H 3900 6800 50  0001 C CNN
+F 1 "+5V" H 3900 7090 50  0000 C CNN
+F 2 "" H 3900 6950 50  0001 C CNN
+F 3 "" H 3900 6950 50  0001 C CNN
+	1    3900 6950
+	1    0    0    -1
+$EndComp
+Wire Wire Line
+	3900 6950 3900 7000
+Wire Wire Line
+	3900 7000 3850 7000
+$Comp
+L GND #PWR?
+U 1 1 5AF9E00C
+P 3900 7150
+F 0 "#PWR?" H 3900 6900 50  0001 C CNN
+F 1 "GND" H 3900 7000 50  0000 C CNN
+F 2 "" H 3900 7150 50  0001 C CNN
+F 3 "" H 3900 7150 50  0001 C CNN
+	1    3900 7150
+	1    0    0    -1
+$EndComp
+Wire Wire Line
+	3850 7100 3900 7100
+Wire Wire Line
+	3900 7100 3900 7150
+$Comp
+L Screw_Terminal_01x06 J?
+U 1 1 5AF9E014
+P 2200 6950
+F 0 "J?" H 2200 7250 50  0000 C CNN
+F 1 "Screw_Terminal_01x06" H 2200 6550 50  0000 C CNN
+F 2 "Connectors_Terminal_Blocks:TerminalBlock_bornier-6_P5.08mm" H 2200 6950 50  0001 C CNN
+F 3 "" H 2200 6950 50  0001 C CNN
+	1    2200 6950
+	-1   0    0    1
+$EndComp
+Wire Wire Line
+	2400 6650 2750 6650
+Wire Wire Line
+	2750 6750 2400 6750
+Wire Wire Line
+	2400 7150 2600 7150
+Wire Wire Line
+	2600 7150 2600 6850
+Wire Wire Line
+	2600 6850 2400 6850
+Wire Wire Line
+	2400 6950 2500 6950
+Wire Wire Line
+	2500 6950 2500 7050
+Wire Wire Line
+	2500 7050 2400 7050
 $EndSCHEMATC

Commit message: before something dies
Parts:
- removed J?: Screw_Terminal_01x06, Connectors_Terminal_Blocks:TerminalBlock_bornier-6_P5.08mm, symbol Screw_Terminal_01x06
- added J1: Screw_Terminal_01x02, Connectors_Terminal_Blocks:TerminalBlock_bornier-2_P5.08mm, symbol Screw_Terminal_01x02
- gave numbers to parts that had none: 1
Connections:
- net at PSU1.1 (Live): now also J1.2 (Pin_2)
- net at PSU1.2 (Neutral): now also J1.1 (Pin_1)
Changed lines of the file:
@@
 	7050 2100 7000 2100
 $Comp
-L IRM-45 PSU?
+L IRM-45 PSU1
 U 1 1 5AF9DFFD
 P 3300 6850
-F 0 "PSU?" H 3200 6800 60  0000 C CNN
+F 0 "PSU1" H 3200 6800 60  0000 C CNN
 F 1 "IRM-45" H 3200 6700 60  0000 C CNN
 F 2 "MATHSTERK:IRM-45" H 3300 6850 60  0001 C CNN
@@
 $EndComp
 $Comp
-L +5V #PWR?
+L +5V #PWR055
 U 1 1 5AF9E004
 P 3900 6950
-F 0 "#PWR?" H 3900 6800 50  0001 C CNN
+F 0 "#PWR055" H 3900 6800 50  0001 C CNN
 F 1 "+5V" H 3900 7090 50  0000 C CNN
 F 2 "" H 3900 6950 50  0001 C CNN
@@
 	3900 7000 3850 7000
 $Comp
-L GND #PWR?
+L GND #PWR056
 U 1 1 5AF9E00C
 P 3900 7150
-F 0 "#PWR?" H 3900 6900 50  0001 C CNN
+F 0 "#PWR056" H 3900 6900 50  0001 C CNN
 F 1 "GND" H 3900 7000 50  0000 C CNN
 F 2 "" H 3900 7150 50  0001 C CNN
@@
 Wire Wire Line
 	3900 7100 3900 7150
-$Comp
-L Screw_Terminal_01x06 J?
-U 1 1 5AF9E014
-P 2200 6950
-F 0 "J?" H 2200 7250 50  0000 C CNN
-F 1 "Screw_Terminal_01x06" H 2200 6550 50  0000 C CNN
-F 2 "Connectors_Terminal_Blocks:TerminalBlock_bornier-6_P5.08mm" H 2200 6950 50  0001 C CNN
-F 3 "" H 2200 6950 50  0001 C CNN
-	1    2200 6950
-	-1   0    0    1
-$EndComp
 Wire Wire Line
 	2400 6650 2750 6650
 Wire Wire Line
 	2750 6750 2400 6750
-Wire Wire Line
-	2400 7150 2600 7150
-Wire Wire Line
-	2600 7150 2600 6850
-Wire Wire Line
-	2600 6850 2400 6850
-Wire Wire Line
-	2400 6950 2500 6950
-Wire Wire Line
-	2500 6950 2500 7050
-Wire Wire Line
-	2500 7050 2400 7050
+$Comp
+L Screw_Terminal_01x02 J1
+U 1 1 5AFA544F
+P 2200 6750
+F 0 "J1" H 2200 6850 50  0000 C CNN
+F 1 "Screw_Terminal_01x02" H 2200 6550 50  0000 C CNN
+F 2 "Connectors_Terminal_Blocks:TerminalBlock_bornier-2_P5.08mm" H 2200 6750 50  0001 C CNN
+F 3 "" H 2200 6750 50  0001 C CNN
+	1    2200 6750
+	-1   0    0    1
+$EndComp
 $EndSCHEMATC

Commit message: lol
Parts:
- PSU1: footprint MATHSTERK:IRM-45 -> (none); part_num (none) -> IRM-45-5
Changed lines of the file:
@@
 	7050 2100 7000 2100
-$Comp
-L IRM-45 PSU1
-U 1 1 5AF9DFFD
-P 3300 6850
-F 0 "PSU1" H 3200 6800 60  0000 C CNN
-F 1 "IRM-45" H 3200 6700 60  0000 C CNN
-F 2 "MATHSTERK:IRM-45" H 3300 6850 60  0001 C CNN
-F 3 "" H 3300 6850 60  0001 C CNN
-	1    3300 6850
-	1    0    0    -1
-$EndComp
 $Comp
 L +5V #PWR065
@@
 	-1   0    0    1
 $EndComp
+$Comp
+L IRM-45 PSU1
+U 1 1 5AFB63D9
+P 3300 6850
+F 0 "PSU1" H 3200 6800 60  0000 C CNN
+F 1 "IRM-45" H 3200 6700 60  0000 C CNN
+F 2 "" H 3300 6850 60  0001 C CNN
+F 3 "" H 3300 6850 60  0001 C CNN
+F 4 "IRM-45-5" H 3300 6900 60  0001 C CNN "part_num"
+	1    3300 6850
+	1    0    0    -1
+$EndComp
 $EndSCHEMATC

Commit message: boop
Parts:
- PSU1: footprint (none) -> MATHSTERK:IRM-45
Changed lines of the file:
@@
 F 0 "PSU1" H 3200 6800 60  0000 C CNN
 F 1 "IRM-45" H 3200 6700 60  0000 C CNN
-F 2 "" H 3300 6850 60  0001 C CNN
+F 2 "MATHSTERK:IRM-45" H 3300 6850 60  0001 C CNN
 F 3 "" H 3300 6850 60  0001 C CNN
 F 4 "IRM-45-5" H 3300 6900 60  0001 C CNN "part_num"
