File: Projects/Voicemeeter/file5AE700A4.sch (KiCad schematic (older format))
At the start: 39 parts, among them J1 Screw_Terminal_01x02, J501 SPARE, J502 GS2, J503 GS2, J504 GS2, J505 MIDI OUT, J506 MIDI IN, J507 DIN-5_180degree, J508 DIN-5_180degree, SW501 PEC11R-4215F-S0024, U501 stm32f103-china-MS, U502 PC817

Commit message: before it's too late
Parts:
- J1: footprint Connectors_Terminal_Blocks:TerminalBlock_bornier-2_P5.08mm -> Connectors_Molex:Molex_Sabre_43160-0X02_02x7.49mm_Vertical
Changed lines of the file:
@@
 F 0 "J1" H 2200 6850 50  0000 C CNN
 F 1 "Screw_Terminal_01x02" H 2200 6550 50  0000 C CNN
-F 2 "Connectors_Terminal_Blocks:TerminalBlock_bornier-2_P5.08mm" H 2200 6750 50  0001 C CNN
+F 2 "Connectors_Molex:Molex_Sabre_43160-0X02_02x7.49mm_Vertical" H 2200 6750 50  0001 C CNN
 F 3 "" H 2200 6750 50  0001 C CNN
 	1    2200 6750

Commit message: boop
Parts:
- D501: footprint Diodes_THT:D_DO-41_SOD81_P12.70mm_Horizontal -> Diodes_THT:D_DO-41_SOD81_P7.62mm_Horizontal
Changed lines of the file:
@@
 F 0 "D501" H 9500 4800 50  0000 C CNN
 F 1 "D" H 9500 4600 50  0000 C CNN
-F 2 "Diodes_THT:D_DO-41_SOD81_P12.70mm_Horizontal" H 9500 4700 50  0001 C CNN
+F 2 "Diodes_THT:D_DO-41_SOD81_P7.62mm_Horizontal" H 9500 4700 50  0001 C CNN
 F 3 "" H 9500 4700 50  0001 C CNN
 	1    9500 4700

Commit message: testing
Parts:
- renumbered J1 to J502, J502 to J503, J503 to J504, J504 to J505, J505 to J506, J506 to J507, J507 to J508, J508 to J509, PSU1 to PSU501
Changed lines of the file:
@@
 $EndComp
 $Comp
-L Conn_01x02 J506
+L Conn_01x02 J507
 U 1 1 5AE75593
 P 10000 4750
-F 0 "J506" H 10000 4900 50  0000 C CNN
+F 0 "J507" H 10000 4900 50  0000 C CNN
 F 1 "MIDI IN" H 10200 4650 50  0000 C CNN
 F 2 "Pin_Headers:Pin_Header_Straight_1x02_Pitch2.54mm" H 10000 4750 50  0001 C CNN
@@
 $EndComp
 $Comp
-L Conn_01x03 J505
+L Conn_01x03 J506
 U 1 1 5AE7562E
 P 9400 3000
-F 0 "J505" H 9400 3200 50  0000 C CNN
+F 0 "J506" H 9400 3200 50  0000 C CNN
 F 1 "MIDI OUT" V 9500 3000 50  0000 C CNN
 F 2 "Pin_Headers:Pin_Header_Straight_1x03_Pitch2.54mm" H 9400 3000 50  0001 C CNN
@@
 ROT3
 $Comp
-L DIN-5_180degree J507
+L DIN-5_180degree J508
 U 1 1 5AF30E9D
 P 10050 2350
-F 0 "J507" H 10175 2575 50  0000 C CNN
+F 0 "J508" H 10175 2575 50  0000 C CNN
 F 1 "DIN-5_180degree" H 10050 2100 50  0000 C CNN
 F 2 "" H 10050 2350 50  0001 C CNN
@@
 NoConn ~ 1950 1550
 $Comp
-L GS2 J504
+L GS2 J505
 U 1 1 5AF39CAF
 P 4300 1900
-F 0 "J504" H 4400 2050 50  0000 C CNN
+F 0 "J505" H 4400 2050 50  0000 C CNN
 F 1 "GS2" H 4400 1751 50  0000 C CNN
 F 2 "MATHSTERK:SB2" V 4374 1900 50  0001 C CNN
@@
 $EndComp
 $Comp
-L GS2 J502
+L GS2 J503
 U 1 1 5AF36E78
 P 2750 5150
-F 0 "J502" H 2850 5300 50  0000 C CNN
+F 0 "J503" H 2850 5300 50  0000 C CNN
 F 1 "GS2" H 2850 5001 50  0000 C CNN
 F 2 "MATHSTERK:SB2" V 2824 5150 50  0001 C CNN
@@
 $EndComp
 $Comp
-L DIN-5_180degree J508
+L DIN-5_180degree J509
 U 1 1 5AF63B2F
 P 10050 3650
-F 0 "J508" H 10175 3875 50  0000 C CNN
+F 0 "J509" H 10175 3875 50  0000 C CNN
 F 1 "DIN-5_180degree" H 10050 3400 50  0000 C CNN
 F 2 "" H 10050 3650 50  0001 C CNN
@@
 $EndComp
 $Comp
-L GS2 J503
+L GS2 J504
 U 1 1 5AFB0685
 P 2800 4100
-F 0 "J503" H 2900 4250 50  0000 C CNN
+F 0 "J504" H 2900 4250 50  0000 C CNN
 F 1 "GS2" H 2900 3951 50  0000 C CNN
 F 2 "MATHSTERK:SB2" V 2874 4100 50  0001 C CNN
@@
 	2750 6750 2400 6750
 $Comp
-L Screw_Terminal_01x02 J1
+L Screw_Terminal_01x02 J502
 U 1 1 5AFA544F
 P 2200 6750
-F 0 "J1" H 2200 6850 50  0000 C CNN
+F 0 "J502" H 2200 6850 50  0000 C CNN
 F 1 "Screw_Terminal_01x02" H 2200 6550 50  0000 C CNN
 F 2 "Connectors_Molex:Molex_Sabre_43160-0X02_02x7.49mm_Vertical" H 2200 6750 50  0001 C CNN
@@
 $EndComp
 $Comp
-L IRM-45 PSU1
+L IRM-45 PSU501
 U 1 1 5AFB63D9
 P 3300 6850
-F 0 "PSU1" H 3200 6800 60  0000 C CNN
+F 0 "PSU501" H 3200 6800 60  0000 C CNN
 F 1 "IRM-45" H 3200 6700 60  0000 C CNN
 F 2 "MATHSTERK:IRM-45" H 3300 6850 60  0001 C CNN
