File: Projects/Voicemeeter/file5AE7739B.sch (KiCad schematic (older format))
At the start: 32 parts

Commit message: stuff
Parts:
- renumbered LED601 to LED1, LED611 to LED10, LED619 to LED11, LED627 to LED12, LED604 to LED13, LED612 to LED14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

Commit message: Zzzzz
Parts:
- renumbered LED1 to LED601, LED5 to LED602, LED9 to LED603, LED13 to LED604, LED17 to LED605, LED21 to LED606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
