File: Projects/Voicemeeter/file5AE7739B.sch (KiCad schematic (older format))
At the start: 32 parts

Commit message: yes
Parts:
- added LED100, LED33, LED34, LED35, LED36, LED37, LED38, LED39, LED40, LED41, LED42, LED43, LED44, LED45, LED46, LED47, LED48, LED49, LED50, LED51, LED52, LED53, LED54, LED55, LED56, LED57, LED58, LED59, LED60, LED61, LED62, LED63, LED64, LED65, LED66, LED67, LED68, LED69, LED70, LED71, LED72, LED73, LED74, LED75, LED76, LED77, LED78, LED79, LED80, LED81, LED82, LED83, LED84, LED85, LED86, LED87, LED88, LED89, LED90, LED91, LED92, LED93, LED94, LED95, LED96, LED97, LED98, LED99: SK9822, LEDs:LED_RGB_5050-6, symbol SK9822
- renumbered LED601 to LED1, LED610 to LED10, LED611 to LED11, LED612 to LED12, LED613 to LED13, LED614 to LED14, LED615 to LED15, LED616 to LED16, LED617 to LED17, LED618 to LED18, LED619 to LED19, LED602 to LED2, LED620 to LED20, LED621 to LED21, LED622 to LED22, LED623 to LED23, LED624 to LED24, LED625 to LED25, LED626 to LED26, LED627 to LED27, LED628 to LED28, LED629 to LED29, LED603 to LED3, LED630 to LED30, LED631 to LED31, LED632 to LED32, LED604 to LED4, LED605 to LED5, LED606 to LED6, LED607 to LED7, LED608 to LED8, LED609 to LED9
Connections:
- net +5V: now also LED100.4 (VCC), LED33.4 (VCC), LED34.4 (VCC), LED35.4 (VCC), LED36.4 (VCC), LED37.4 (VCC), LED38.4 (VCC), LED39.4 (VCC), LED40.4 (VCC), LED41.4 (VCC), LED42.4 (VCC), LED43.4 (VCC), LED44.4 (VCC), LED45.4 (VCC), LED46.4 (VCC), LED47.4 (VCC), LED48.4 (VCC), LED49.4 (VCC), LED50.4 (VCC), LED51.4 (VCC), LED52.4 (VCC), LED53.4 (VCC), LED54.4 (VCC), LED55.4 (VCC), LED56.4 (VCC), LED57.4 (VCC), LED58.4 (VCC), LED59.4 (VCC), LED60.4 (VCC), LED61.4 (VCC), LED62.4 (VCC), LED63.4 (VCC), LED64.4 (VCC), LED65.4 (VCC), LED66.4 (VCC), LED67.4 (VCC), LED68.4 (VCC), LED69.4 (VCC), LED70.4 (VCC), LED71.4 (VCC), LED72.4 (VCC), LED73.4 (VCC), LED74.4 (VCC), LED75.4 (VCC), LED76.4 (VCC), LED77.4 (VCC), LED78.4 (VCC), LED79.4 (VCC), LED80.4 (VCC), LED81.4 (VCC), LED82.4 (VCC), LED83.4 (VCC), LED84.4 (VCC), LED85.4 (VCC), LED86.4 (VCC), LED87.4 (VCC), LED88.4 (VCC), LED89.4 (VCC), LED90.4 (VCC), LED91.4 (VCC), LED92.4 (VCC), LED93.4 (VCC), LED94.4 (VCC), LED95.4 (VCC), LED96.4 (VCC), LED97.4 (VCC), LED98.4 (VCC), LED99.4 (VCC)
- net GND: now also LED100.3 (GND), LED33.3 (GND), LED34.3 (GND), LED35.3 (GND), LED36.3 (GND), LED37.3 (GND), LED38.3 (GND), LED39.3 (GND), LED40.3 (GND), LED41.3 (GND), LED42.3 (GND), LED43.3 (GND), LED44.3 (GND), LED45.3 (GND), LED46.3 (GND), LED47.3 (GND), LED48.3 (GND), LED49.3 (GND), LED50.3 (GND), LED51.3 (GND), LED52.3 (GND), LED53.3 (GND), LED54.3 (GND), LED55.3 (GND), LED56.3 (GND), LED57.3 (GND), LED58.3 (GND), LED59.3 (GND), LED60.3 (GND), LED61.3 (GND), LED62.3 (GND), LED63.3 (GND), LED64.3 (GND), LED65.3 (GND), LED66.3 (GND), LED67.3 (GND), LED68.3 (GND), LED69.3 (GND), LED70.3 (GND), LED71.3 (GND), LED72.3 (GND), LED73.3 (GND), LED74.3 (GND), LED75.3 (GND), LED76.3 (GND), LED77.3 (GND), LED78.3 (GND), LED79.3 (GND), LED80.3 (GND), LED81.3 (GND), LED82.3 (GND), LED83.3 (GND), LED84.3 (GND), LED85.3 (GND), LED86.3 (GND), LED87.3 (GND), LED88.3 (GND), LED89.3 (GND), LED90.3 (GND), LED91.3 (GND), LED92.3 (GND), LED93.3 (GND), LED94.3 (GND), LED95.3 (GND), LED96.3 (GND), LED97.3 (GND), LED98.3 (GND), LED99.3 (GND)
- net at LED32.5 (CKO): now also LED33.2 (CKI)
- net at LED32.6 (SDO): now also LED33.1 (SDI)
- new net: LED33.5 (CKO), LED34.2 (CKI)
- new net: LED33.6 (SDO), LED34.1 (SDI)
- new net: LED34.5 (CKO), LED35.2 (CKI)
- new net: LED34.6 (SDO), LED35.1 (SDI)
- new net: LED35.5 (CKO), LED36.2 (CKI)
- new net: LED35.6 (SDO), LED36.1 (SDI)
- new net: LED36.5 (CKO), LED37.2 (CKI)
- new net: LED36.6 (SDO), LED37.1 (SDI)
- new net: LED37.5 (CKO), LED38.2 (CKI)
- new net: LED37.6 (SDO), LED38.1 (SDI)
- new net: LED38.5 (CKO), LED39.2 (CKI)
- new net: LED38.6 (SDO), LED39.1 (SDI)
- new net: LED39.5 (CKO), LED40.2 (CKI)
- new net: LED39.6 (SDO), LED40.1 (SDI)
- new net: LED40.5 (CKO), LED41.2 (CKI)
- new net: LED40.6 (SDO), LED41.1 (SDI)
- new net: LED41.5 (CKO), LED42.2 (CKI)
- new net: LED41.6 (SDO), LED42.1 (SDI)
- new net: LED42.5 (CKO), LED43.2 (CKI)
- new net: LED42.6 (SDO), LED43.1 (SDI)
- new net: LED43.5 (CKO), LED44.2 (CKI)
- new net: LED43.6 (SDO), LED44.1 (SDI)
- new net: LED44.5 (CKO), LED45.2 (CKI)
- new net: LED44.6 (SDO), LED45.1 (SDI)
- new net: LED45.5 (CKO), LED46.2 (CKI)
- new net: LED45.6 (SDO), LED46.1 (SDI)
- new net: LED46.5 (CKO), LED47.2 (CKI)
- new net: LED46.6 (SDO), LED47.1 (SDI)
- new net: LED47.5 (CKO), LED48.2 (CKI)
- new net: LED47.6 (SDO), LED48.1 (SDI)
- new net: LED48.5 (CKO), LED49.2 (CKI)
- new net: LED48.6 (SDO), LED49.1 (SDI)
- new net: LED49.5 (CKO), LED50.2 (CKI)
- new net: LED49.6 (SDO), LED50.1 (SDI)
- new net: LED50.5 (CKO), LED51.2 (CKI)
- new net: LED50.6 (SDO), LED51.1 (SDI)
- new net: LED51.5 (CKO), LED52.2 (CKI)
- new net: LED51.6 (SDO), LED52.1 (SDI)
- new net: LED52.5 (CKO), LED53.2 (CKI)
- new net: LED52.6 (SDO), LED53.1 (SDI)
- new net: LED53.5 (CKO), LED54.2 (CKI)
- new net: LED53.6 (SDO), LED54.1 (SDI)
- new net: LED54.5 (CKO), LED55.2 (CKI)
- new net: LED54.6 (SDO), LED55.1 (SDI)
- new net: LED55.5 (CKO), LED56.2 (CKI)
- new net: LED55.6 (SDO), LED56.1 (SDI)
- new net: LED56.5 (CKO), LED57.2 (CKI)
- new net: LED56.6 (SDO), LED57.1 (SDI)
- new net: LED57.5 (CKO), LED58.2 (CKI)
- new net: LED57.6 (SDO), LED58.1 (SDI)
- new net: LED58.5 (CKO), LED59.2 (CKI)
- new net: LED58.6 (SDO), LED59.1 (SDI)
- new net: LED59.5 (CKO), LED60.2 (CKI)
- new net: LED59.6 (SDO), LED60.1 (SDI)
- new net: LED60.5 (CKO), LED61.2 (CKI)
- new net: LED60.6 (SDO), LED61.1 (SDI)
- new net: LED61.5 (CKO), LED62.2 (CKI)
- new net: LED61.6 (SDO), LED62.1 (SDI)
- new net: LED62.5 (CKO), LED63.2 (CKI)
- new net: LED62.6 (SDO), LED63.1 (SDI)
- new net: LED63.5 (CKO), LED64.2 (CKI)
- new net: LED63.6 (SDO), LED64.1 (SDI)
- new net: LED64.5 (CKO), LED65.2 (CKI)
- new net: LED64.6 (SDO), LED65.1 (SDI)
- new net: LED65.5 (CKO), LED66.2 (CKI)
- new net: LED65.6 (SDO), LED66.1 (SDI)
- new net: LED66.5 (CKO), LED67.2 (CKI)
- new net: LED66.6 (SDO), LED67.1 (SDI)
- new net: LED67.5 (CKO), LED68.2 (CKI)
- new net: LED67.6 (SDO), LED68.1 (SDI)
- new net: LED68.5 (CKO), LED69.2 (CKI)
- new net: LED68.6 (SDO), LED69.1 (SDI)
- new net: LED69.5 (CKO), LED70.2 (CKI)
- new net: LED69.6 (SDO), LED70.1 (SDI)
- new net: LED70.5 (CKO), LED71.2 (CKI)
- new net: LED70.6 (SDO), LED71.1 (SDI)
- new net: LED71.5 (CKO), LED72.2 (CKI)
- new net: LED71.6 (SDO), LED72.1 (SDI)
- new net: LED72.5 (CKO), LED73.2 (CKI)
- new net: LED72.6 (SDO), LED73.1 (SDI)
- new net: LED73.5 (CKO), LED74.2 (CKI)
- new net: LED73.6 (SDO), LED74.1 (SDI)
- new net: LED74.5 (CKO), LED75.2 (CKI)
- new net: LED74.6 (SDO), LED75.1 (SDI)
- new net: LED75.5 (CKO), LED76.2 (CKI)
- new net: LED75.6 (SDO), LED76.1 (SDI)
- new net: LED76.5 (CKO), LED77.2 (CKI)
- new net: LED76.6 (SDO), LED77.1 (SDI)
- new net: LED77.5 (CKO), LED78.2 (CKI)
- new net: LED77.6 (SDO), LED78.1 (SDI)
- new net: LED78.5 (CKO), LED79.2 (CKI)
- new net: LED78.6 (SDO), LED79.1 (SDI)
- new net: LED79.5 (CKO), LED80.2 (CKI)
- new net: LED79.6 (SDO), LED80.1 (SDI)
- new net: LED80.5 (CKO), LED81.2 (CKI)
- new net: LED80.6 (SDO), LED81.1 (SDI)
- new net: LED81.5 (CKO), LED82.2 (CKI)
- new net: LED81.6 (SDO), LED82.1 (SDI)
- new net: LED82.5 (CKO), LED83.2 (CKI)
- new net: LED82.6 (SDO), LED83.1 (SDI)
- new net: LED83.5 (CKO), LED84.2 (CKI)
- new net: LED83.6 (SDO), LED84.1 (SDI)
- new net: LED84.5 (CKO), LED85.2 (CKI)
- new net: LED84.6 (SDO), LED85.1 (SDI)
- new net: LED85.5 (CKO), LED86.2 (CKI)
- new net: LED85.6 (SDO), LED86.1 (SDI)
- new net: LED86.5 (CKO), LED87.2 (CKI)
- new net: LED86.6 (SDO), LED87.1 (SDI)
- new net: LED87.5 (CKO), LED88.2 (CKI)
- new net: LED87.6 (SDO), LED88.1 (SDI)
- new net: LED88.5 (CKO), LED89.2 (CKI)
- new net: LED88.6 (SDO), LED89.1 (SDI)
- new net: LED89.5 (CKO), LED90.2 (CKI)
- new net: LED89.6 (SDO), LED90.1 (SDI)
- new net: LED90.5 (CKO), LED91.2 (CKI)
- new net: LED90.6 (SDO), LED91.1 (SDI)
- new net: LED91.5 (CKO), LED92.2 (CKI)
- new net: LED91.6 (SDO), LED92.1 (SDI)
- new net: LED92.5 (CKO), LED93.2 (CKI)
- new net: LED92.6 (SDO), LED93.1 (SDI)
- new net: LED93.5 (CKO), LED94.2 (CKI)
- new net: LED93.6 (SDO), LED94.1 (SDI)
- new net: LED94.5 (CKO), LED95.2 (CKI)
- new net: LED94.6 (SDO), LED95.1 (SDI)
- new net: LED95.5 (CKO), LED96.2 (CKI)
- new net: LED95.6 (SDO), LED96.1 (SDI)
- new net: LED96.5 (CKO), LED97.2 (CKI)
- new net: LED96.6 (SDO), LED97.1 (SDI)
- new net: LED97.5 (CKO), LED98.2 (CKI)
- new net: LED97.6 (SDO), LED98.1 (SDI)
- new net: LED98.5 (CKO), LED99.2 (CKI)
- new net: LED98.6 (SDO), LED99.1 (SDI)
- new net: LED100.2 (CKI), LED99.5 (CKO)
- new net: LED100.1 (SDI), LED99.6 (SDO)
Other:
- moved on the sheet: LED1, LED10, LED11, LED12, LED13, LED14, LED15, LED16, LED17, LED18, LED19, LED2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

Commit message: before something dies
Parts:
- added LED101, LED102, LED103: SK9822, MATHSTERK:LED_RGB_5050-6, symbol SK9822
- LED1, LED10, LED100, LED11, LED12, LED13, LED14, LED15, LED16, LED17, LED18, LED19, LED2, LED20, LED21, LED22, LED23, LED24, LED25, LED26, LED27, LED28, LED29, LED3, LED30, LED31, LED32, LED33, LED34, LED35, LED36, LED37, LED38, LED39, LED4, LED40, LED41, LED42, LED43, LED44, LED45, LED46, LED47, LED48, LED49, LED5, LED50, LED51, LED52, LED53, LED54, LED55, LED56, LED57, LED58, LED59, LED6, LED60, LED61, LED62, LED63, LED64, LED65, LED66, LED67, LED68, LED69, LED7, LED70, LED71, LED72, LED73, LED74, LED75, LED76, LED77, LED78, LED79, LED8, LED80, LED81, LED82, LED83, LED84, LED85, LED86, LED87, LED88, LED89, LED9, LED90, LED91, LED92, LED93, LED94, LED95, LED96, LED97, LED98, LED99: footprint LEDs:LED_RGB_5050-6 -> MATHSTERK:LED_RGB_5050-6
Connections:
- net +5V: now also LED101.4 (VCC), LED102.4 (VCC), LED103.4 (VCC)
- net GND: now also LED101.3 (GND), LED102.3 (GND), LED103.3 (GND)
- net at LED100.5 (CKO): now also LED101.2 (CKI)
- net at LED100.6 (SDO): now also LED101.1 (SDI)
- new net: LED101.5 (CKO), LED102.2 (CKI)
- new net: LED101.6 (SDO), LED102.1 (SDI)
- new net: LED102.5 (CKO), LED103.2 (CKI)
- new net: LED102.6 (SDO), LED103.1 (SDI)

Commit message: moar leds, more powah
Parts:
- added LED104, LED105, LED106, LED107, LED108, LED109, LED110: SK9822, MATHSTERK:LED_RGB_5050-6, symbol SK9822
Connections:
- net +5V: now also LED104.4 (VCC), LED105.4 (VCC), LED106.4 (VCC), LED107.4 (VCC), LED108.4 (VCC), LED109.4 (VCC), LED110.4 (VCC)
- net GND: now also LED104.3 (GND), LED105.3 (GND), LED106.3 (GND), LED107.3 (GND), LED108.3 (GND), LED109.3 (GND), LED110.3 (GND)
- net at LED103.5 (CKO): now also LED104.2 (CKI)
- net at LED103.6 (SDO): now also LED104.1 (SDI)
- new net: LED104.6 (SDO), LED105.1 (SDI)
- new net: LED104.5 (CKO), LED105.2 (CKI)
- new net: LED105.5 (CKO), LED106.2 (CKI)
- new net: LED105.6 (SDO), LED106.1 (SDI)
- new net: LED106.5 (CKO), LED107.2 (CKI)
- new net: LED106.6 (SDO), LED107.1 (SDI)
- new net: LED107.5 (CKO), LED108.2 (CKI)
- new net: LED107.6 (SDO), LED108.1 (SDI)
- new net: LED108.5 (CKO), LED109.2 (CKI)
- new net: LED108.6 (SDO), LED109.1 (SDI)
- new net: LED109.5 (CKO), LED110.2 (CKI)
- new net: LED109.6 (SDO), LED110.1 (SDI)
- no-connect marks 2 -> 0

Commit message: in case of emergency
Parts:
- added LED111, LED112, LED113, LED114, LED115, LED116: SK9822, MATHSTERK:LED_RGB_5050-6, symbol SK9822
Connections:
- net +5V: now also LED111.4 (VCC), LED112.4 (VCC), LED113.4 (VCC), LED114.4 (VCC), LED115.4 (VCC), LED116.4 (VCC)
- net GND: now also LED111.3 (GND), LED112.3 (GND), LED113.3 (GND), LED114.3 (GND), LED115.3 (GND), LED116.3 (GND)
- net at LED110.5 (CKO): now also LED111.2 (CKI)
- net at LED110.6 (SDO): now also LED111.1 (SDI)
- new net: LED111.5 (CKO), LED112.2 (CKI)
- new net: LED111.6 (SDO), LED112.1 (SDI)
- new net: LED112.5 (CKO), LED113.2 (CKI)
- new net: LED112.6 (SDO), LED113.1 (SDI)
- new net: LED113.5 (CKO), LED114.2 (CKI)
- new net: LED113.6 (SDO), LED114.1 (SDI)
- new net: LED114.5 (CKO), LED115.2 (CKI)
- new net: LED114.6 (SDO), LED115.1 (SDI)
- new net: LED115.5 (CKO), LED116.2 (CKI)
- new net: LED115.6 (SDO), LED116.1 (SDI)
- no-connect marks 0 -> 2

Commit message: testing
Parts:
- renumbered LED1 to LED601, LED9 to LED602, LED17 to LED603, LED25 to LED604, LED33 to LED605, LED41 to LED606, LED49 to LED607, LED57 to LED608, LED65 to LED609, LED73 to LED610, LED81 to LED611, LED89 to LED612, LED97 to LED613, LED105 to LED614, LED113 to LED615, LED2 to LED616, LED10 to LED617, LED18 to LED618, LED26 to LED619, LED34 to LED620, LED42 to LED621, LED50 to LED622, LED58 to LED623, LED66 to LED624, LED74 to LED625, LED82 to LED626, LED90 to LED627, LED98 to LED628, LED106 to LED629, LED114 to LED630, LED3 to LED631, LED11 to LED632, LED19 to LED633, LED27 to LED634, LED35 to LED635, LED43 to LED636, LED51 to LED637, LED59 to LED638, LED67 to LED639, LED75 to LED640, LED83 to LED641, LED91 to LED642, LED99 to LED643, LED107 to LED644, LED115 to LED645, LED4 to LED646, LED12 to LED647, LED20 to LED648, LED28 to LED649, LED36 to LED650, LED44 to LED651, LED52 to LED652, LED60 to LED653, LED68 to LED654, LED76 to LED655, LED84 to LED656, LED92 to LED657, LED100 to LED658, LED108 to LED659, LED116 to LED660, LED5 to LED661, LED13 to LED662, LED21 to LED663, LED29 to LED664, LED37 to LED665, LED45 to LED666, LED53 to LED667, LED61 to LED668, LED69 to LED669, LED77 to LED670, LED85 to LED671, LED93 to LED672, LED101 to LED673, LED109 to LED674, LED6 to LED675, LED14 to LED676, LED22 to LED677, LED30 to LED678, LED38 to LED679, LED46 to LED680, LED54 to LED681, LED62 to LED682, LED70 to LED683, LED78 to LED684, LED86 to LED685, LED94 to LED686, LED102 to LED687, LED110 to LED688, LED7 to LED689, LED15 to LED690, LED23 to LED691, LED31 to LED692, LED39 to LED693, LED47 to LED694, LED55 to LED695, LED63 to LED696, LED71 to LED697, LED79 to LED698, LED87 to LED699, LED95 to LED700, LED103 to LED701, LED111 to LED702, LED8 to LED703, LED16 to LED704, LED24 to LED705, LED32 to LED706, LED40 to LED707, LED48 to LED708, LED56 to LED709, LED64 to LED710, LED72 to LED711, LED80 to LED712, LED88 to LED713, LED96 to LED714, LED104 to LED715, LED112 to LED716
