File: Projects/Voicemeeter/file5AFAE97F.sch (KiCad schematic (older format))
At the start: 0 parts

Commit message: uuuuuugh
Parts:
- added J?: Screw_Terminal_01x06, symbol Screw_Terminal_01x06
- added PSU701: IRM-45, MATHSTERK:IRM-45, symbol IRM-45
Connections:
- new net: J?.6 (Pin_6), PSU701.1 (Live)
- new net: J?.5 (Pin_5), PSU701.2 (Neutral)
- new net: J?.1 (Pin_1), J?.4 (Pin_4)
- new net: J?.2 (Pin_2), J?.3 (Pin_3)
- new net +5V: PSU701.3 (5V)
- new net GND: PSU701.4 (GND)
Changed lines of the file:
@@
 $Descr A4 11693 8268
 encoding utf-8
-Sheet 1 7
+Sheet 7 7
 Title ""
-Date "2018-04-28"
+Date ""
 Rev ""
 Comp ""
@@
 Comment4 ""
 $EndDescr
-$Sheet
-S 2000 2750 1000 1050
-U 5AE49271
-F0 "Pot" 60
-F1 "file5AE49270.sch" 60
-F2 "HD[11..38]" O R 3000 2850 60
-F3 "DD[11..28]" O R 3000 2950 60
-F4 "OD[11..53]" O R 3000 3050 60
-F5 "OA[1..5]" O R 3000 3150 60
-F6 "DA[11..24]" O R 3000 3250 60
-F7 "HA[11..33]" O R 3000 3350 60
-$EndSheet
-$Sheet
-S 4000 3750 1000 400
-U 5AE5FE22
-F0 "Capacitors" 60
-F1 "file5AE5FE21.sch" 60
-F2 "HA[11..33]" B L 4000 4050 60
-F3 "DA[11..24]" B L 4000 3950 60
-F4 "OA[1..5]" B L 4000 3850 60
-$EndSheet
-$Sheet
-S 4000 2750 1450 700
-U 5AF6330D
-F0 "Mux" 60
-F1 "file5AF6330C.sch" 60
-F2 "HA[11..33]" I L 4000 3350 60
-F3 "OA[1..5]" I L 4000 3150 60
-F4 "DA[11..24]" I L 4000 3250 60
-F5 "M[1..27]" O R 5450 2950 60
-F6 "HD[11..38]" I L 4000 2850 60
-F7 "DD[11..28]" I L 4000 2950 60
-F8 "OD[11..53]" I L 4000 3050 60
-$EndSheet
-Wire Bus Line
-	4000 4050 3100 4050
-Wire Bus Line
-	3100 4050 3100 3350
-Wire Bus Line
-	3000 3350 4000 3350
-Wire Bus Line
-	3000 3250 4000 3250
-Wire Bus Line
-	3200 3250 3200 3950
-Wire Bus Line
-	3200 3950 4000 3950
-Wire Bus Line
-	4000 3850 3300 3850
-Wire Bus Line
-	3300 3850 3300 3150
-Wire Bus Line
-	3000 3150 4000 3150
-Wire Bus Line
-	4000 3050 3000 3050
-Wire Bus Line
-	3000 2850 4000 2850
-Wire Bus Line
-	3000 2950 4000 2950
-$Sheet
-S 6250 2750 1500 700
-U 5AE700A5
-F0 "STM" 60
-F1 "file5AE700A4.sch" 60
-F2 "M[1..27]" I L 6250 2950 60
-F3 "SK[1..2]" O R 7750 3100 60
-$EndSheet
-Connection ~ 3300 3150
-Connection ~ 3200 3250
-Connection ~ 3100 3350
-Wire Bus Line
-	5450 2950 6250 2950
-$Sheet
-S 8100 2900 1050 450
-U 5AE7739C
-F0 "LEDs" 60
-F1 "file5AE7739B.sch" 60
-F2 "SK[1..2]" I L 8100 3100 60
-$EndSheet
-Wire Bus Line
-	7750 3100 8100 3100
-$Sheet
-S 4000 1550 1450 750
-U 5AFAE980
-F0 "PSU" 60
-F1 "file5AFAE97F.sch" 60
-$EndSheet
+$Comp
+L IRM-45 PSU701
+U 1 1 5AFAEAD3
+P 4350 3000
+F 0 "PSU701" H 4250 2950 60  0000 C CNN
+F 1 "IRM-45" H 4250 2850 60  0000 C CNN
+F 2 "MATHSTERK:IRM-45" H 4350 3000 60  0001 C CNN
+F 3 "" H 4350 3000 60  0001 C CNN
+	1    4350 3000
+	1    0    0    -1
+$EndComp
+$Comp
+L +5V #PWR0119
+U 1 1 5AFAEB53
+P 4950 3100
+F 0 "#PWR0119" H 4950 2950 50  0001 C CNN
+F 1 "+5V" H 4950 3240 50  0000 C CNN
+F 2 "" H 4950 3100 50  0001 C CNN
+F 3 "" H 4950 3100 50  0001 C CNN
+	1    4950 3100
+	1    0    0    -1
+$EndComp
+Wire Wire Line
+	4950 3100 4950 3150
+Wire Wire Line
+	4950 3150 4900 3150
+$Comp
+L GND #PWR0120
+U 1 1 5AFAEB6C
+P 4950 3300
+F 0 "#PWR0120" H 4950 3050 50  0001 C CNN
+F 1 "GND" H 4950 3150 50  0000 C CNN
+F 2 "" H 4950 3300 50  0001 C CNN
+F 3 "" H 4950 3300 50  0001 C CNN
+	1    4950 3300
+	1    0    0    -1
+$EndComp
+Wire Wire Line
+	4900 3250 4950 3250
+Wire Wire Line
+	4950 3250 4950 3300
+$Comp
+L Screw_Terminal_01x06 J?
+U 1 1 5AFB15A4
+P 3250 3100
+F 0 "J?" H 3250 3400 50  0000 C CNN
+F 1 "Screw_Terminal_01x06" H 3250 2700 50  0000 C CNN
+F 2 "" H 3250 3100 50  0001 C CNN
+F 3 "" H 3250 3100 50  0001 C CNN
+	1    3250 3100
+	-1   0    0    1
+$EndComp
+Wire Wire Line
+	3450 2800 3800 2800
+Wire Wire Line
+	3800 2900 3450 2900
+Wire Wire Line
+	3450 3300 3650 3300
+Wire Wire Line
+	3650 3300 3650 3000
+Wire Wire Line
+	3650 3000 3450 3000
+Wire Wire Line
+	3450 3100 3550 3100
+Wire Wire Line
+	3550 3100 3550 3200
+Wire Wire Line
+	3550 3200 3450 3200
 $EndSCHEMATC

Commit message: yes
Parts:
- J701: renamed from J?; footprint (none) -> Connectors_Terminal_Blocks:TerminalBlock_bornier-6_P5.08mm
Changed lines of the file:
@@
 $EndComp
 $Comp
-L +5V #PWR0119
+L +5V #PWR0255
 U 1 1 5AFAEB53
 P 4950 3100
-F 0 "#PWR0119" H 4950 2950 50  0001 C CNN
+F 0 "#PWR0255" H 4950 2950 50  0001 C CNN
 F 1 "+5V" H 4950 3240 50  0000 C CNN
 F 2 "" H 4950 3100 50  0001 C CNN
@@
 	4950 3150 4900 3150
 $Comp
-L GND #PWR0120
+L GND #PWR0256
 U 1 1 5AFAEB6C
 P 4950 3300
-F 0 "#PWR0120" H 4950 3050 50  0001 C CNN
+F 0 "#PWR0256" H 4950 3050 50  0001 C CNN
 F 1 "GND" H 4950 3150 50  0000 C CNN
 F 2 "" H 4950 3300 50  0001 C CNN
@@
 	4950 3250 4950 3300
 $Comp
-L Screw_Terminal_01x06 J?
+L Screw_Terminal_01x06 J701
 U 1 1 5AFB15A4
 P 3250 3100
-F 0 "J?" H 3250 3400 50  0000 C CNN
+F 0 "J701" H 3250 3400 50  0000 C CNN
 F 1 "Screw_Terminal_01x06" H 3250 2700 50  0000 C CNN
-F 2 "" H 3250 3100 50  0001 C CNN
+F 2 "Connectors_Terminal_Blocks:TerminalBlock_bornier-6_P5.08mm" H 3250 3100 50  0001 C CNN
 F 3 "" H 3250 3100 50  0001 C CNN
 	1    3250 3100
