File: Projects/Voicemeeter/test.kicad_pcb (KiCad board)
At the start: 2 copper layers, 678.5 x 302.5 mm, 45 parts, among them J501 SPARE, J502 GS2, J503 GS2, J504 GS2, J505 MIDI OUT, J506 MIDI IN, SW501 PEC11R-4215F-S0024, U401 74HC4051, U402 74HC4051, U403 74HC4051, U404 74HC4051, U405 74HC4051, U406 74HC4051, U407 74HC4051, U408 74HC4051, U409 74HC4051, U410 74HC4051, U502 PC817

Commit message: yes
Parts:
- removed J503: GS2, Connectors_Terminal_Blocks:TerminalBlock_Altech_AK300-2_P5.00mm
- removed R501, R504, R505, R506, R507, R508, R509, R510, R511, R512, R513, R515, R516, R517, R518, R520, R522: 10K, Resistors_SMD:R_1206_HandSoldering
- removed R514, R521: 220R, Resistors_SMD:R_1206_HandSoldering
- removed R519: 330R, Resistors_SMD:R_1206_HandSoldering
- removed RESET501: SW_Push, Buttons_Switches_THT:SW_PUSH-12mm
- removed U402: 74HC4051, Housings_DIP:DIP-16_W7.62mm_LongPads
- U401, U403, U404, U405, U406, U407, U408, U409, U410: moved to B.Cu
- moved J502 216.3 mm to (100.0, 29.4)
- moved J501 201.6 mm to (90.0, 24.9), turned to 0 degrees
- moved J504 173.2 mm to (90.6, 40.0)
- moved J505 139.6 mm to (117.5, 30.0)
- moved D501 114.0 mm to (151.9, 37.3)
- moved J506 114.0 mm to (146.5, 24.6)
- moved U502 114.0 mm to (146.5, 36.5)
- moved C502 114.0 mm to (131.0, 27.1)
- moved R502 114.0 mm to (133.0, 34.1)
- moved R503 114.0 mm to (133.0, 36.8)
- moved OLED501 110.3 mm to (200.0, 60.0)
- moved C501 110.1 mm to (300.0, 115.0)
- moved U406 109.9 mm to (95.0, 115.0), turned to 270 degrees
- moved U407 109.3 mm to (130.0, 115.0), turned to 270 degrees
- moved U405 109.0 mm to (65.0, 115.0), turned to 270 degrees
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Connections:
- U401 pad 6: (no net) -> Net-(U401-Pad6)
- U401 pad 7: (no net) -> Net-(U401-Pad7)
- U403 pad 4: (no net) -> Net-(U403-Pad4)
- U403 pad 6: (no net) -> Net-(U403-Pad6)
- U403 pad 7: (no net) -> Net-(U403-Pad7)
- U404 pad 6: (no net) -> Net-(U404-Pad6)
- U404 pad 7: (no net) -> Net-(U404-Pad7)
- U405 pad 6: (no net) -> Net-(U405-Pad6)
- U405 pad 7: (no net) -> Net-(U405-Pad7)
- U406 pad 6: (no net) -> Net-(U406-Pad6)
- U406 pad 7: (no net) -> Net-(U406-Pad7)
- U407 pad 6: (no net) -> Net-(U407-Pad6)
- U407 pad 7: (no net) -> Net-(U407-Pad7)
- U408 pad 6: (no net) -> Net-(U408-Pad6)
- U408 pad 7: (no net) -> Net-(U408-Pad7)
- U409 pad 6: (no net) -> Net-(U409-Pad6)
- U409 pad 7: (no net) -> Net-(U409-Pad7)
- U410 pad 12: (no net) -> Net-(U410-Pad12)
- U410 pad 6: (no net) -> Net-(U410-Pad6)
- U410 pad 7: (no net) -> Net-(U410-Pad7)
- U502 pad 1: Net-(R519-Pad1) -> Net-(D501-Pad1)
- U502 pad 2: GND -> Net-(D501-Pad2)
- U502 pad 3: Net-(D501-Pad2) -> GND
- U502 pad 4: Net-(D501-Pad1) -> Net-(R519-Pad1)
Other:
- board size 678.5 x 302.5 mm -> 604.5 x 217 mm
