File: Projects/Voicemeeter/test.kicad_pcb (KiCad board)
At the start: 2 copper layers, 310 x 190 mm, 12 parts, among them J501 SPARE, J502 GS2, J504 GS2, J505 MIDI OUT, J506 MIDI IN, U502 PC817

Commit message: in case of emergency
Parts:
- moved J504 62.1 mm to (30.5, 24.8), turned to 0 degrees
Routing:
- added copper zone on B.Cu, net +3V3
- added copper zone on F.Cu, net GND

Commit message: gtg
Parts:
- C501, C502, D501, J505, J506, U502: moved to B.Cu
- moved J504 2.54 mm to (30.5, 27.3)
- turned J505 to 270 degrees
Routing:
- net /Capacitors/HA11: track 0.00 -> 125.2 mm
- net /Mux/HD18: track 0.00 -> 105.0 mm
- net /Mux/M3: track 0.00 -> 103.9 mm
- net /Mux/M1: track 0.00 -> 101.9 mm
- net /Mux/M2: track 0.00 -> 101.7 mm
- net /Mux/HD17: track 0.00 -> 95.0 mm
- net /Mux/HD16: track 0.00 -> 83.5 mm
- net /Mux/HD15: track 0.00 -> 75.7 mm
- net /Mux/HD14: track 0.00 -> 46.6 mm
- net /Mux/HD13: track 0.00 -> 36.5 mm
- net /Mux/HD12: track 0.00 -> 25.4 mm
- net /Mux/HD11: track 0.00 -> 11.5 mm
- net Net-(LED19-Pad6): track 0.00 -> 8.20 mm
- net Net-(LED19-Pad5): track 0.00 -> 8.20 mm
- net Net-(LED21-Pad6): track 0.00 -> 4.20 mm
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
Commit message: buh
Routing:
- net +5V: track 0.00 -> 158.6 mm
- net Net-(LED12-Pad5): track 0.00 -> 134.2 mm
- net Net-(LED12-Pad6): track 0.00 -> 131.3 mm
- net /Capacitors/HA11: track 125.2 -> 0.40 mm
- net Net-(LED10-Pad1): track 0.00 -> 37.3 mm
- net Net-(LED4-Pad6): track 0.00 -> 37.3 mm
- net Net-(LED6-Pad5): track 0.00 -> 36.0 mm
- net Net-(LED10-Pad2): track 0.00 -> 33.3 mm
- net Net-(LED4-Pad5): track 0.00 -> 33.3 mm
- net Net-(LED2-Pad5): track 0.00 -> 32.0 mm
- net Net-(LED6-Pad6): track 0.00 -> 28.8 mm
- net Net-(LED2-Pad6): track 0.00 -> 27.2 mm
- net Net-(LED13-Pad6): track 0.00 -> 26.0 mm
- net Net-(LED13-Pad5): track 0.00 -> 25.2 mm
- net Net-(LED14-Pad5): track 0.00 -> 24.1 mm
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
Commit message: zzzz
Routing:
- net /Capacitors/HA11: track 0.40 -> 58.0 mm, vias 0 -> 1
- net +5V: track 158.6 -> 176.0 mm, vias 0 -> 6
- net /Mux/M1: track 101.9 -> 108.0 mm
- net Net-(LED14-Pad6): track 16.6 -> 22.5 mm, vias 0 -> 2
- net /Mux/M2: track 101.7 -> 104.6 mm, vias 0 -> 1
- net /Mux/HD17: track 95.0 -> 97.5 mm
- net /Mux/HD16: track 83.5 -> 86.0 mm
- net /Mux/HD15: track 75.7 -> 78.2 mm
- net GND: track 1.62 -> 2.75 mm, vias 1 -> 2
- net /Mux/HD12: track 25.4 -> 26.5 mm
- net Net-(LED14-Pad5): track 24.1 -> 24.4 mm, vias 0 -> 2

Commit message: lol
Routing:
- net /Capacitors/HA11: track 58.0 -> 57.3 mm
- net (no net): track 0.00 -> 0.78 mm
Changed lines of the file:
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@@
   (general
     (links 1154)
-    (no_connects 541)
-    (area 15 15 348.564286 222.700001)
+    (no_connects 535)
+    (area 19.949999 19.949999 330.050001 210.050001)
     (thickness 1.6)
     (drawings 11)
@@
   )
   (setup
-    (last_trace_width 0.508)
+    (last_trace_width 0.25)
     (user_trace_width 0.1524)
     (user_trace_width 0.254)
@@
   (gr_line (start 330 210) (end 330 20) (angle 90) (layer Edge.Cuts) (width 0.1))
   (gr_line (start 20 210) (end 330 210) (angle 90) (layer Edge.Cuts) (width 0.1))
+  (segment (start 76.74 98.26) (end 76.74 97.88) (width 0.508) (layer F.Cu) (net 0))
+  (segment (start 90.04 54.72) (end 90.04 55.12) (width 0.508) (layer F.Cu) (net 0))
   (segment (start 63.05 128.5) (end 61.75 128.5) (width 0.508) (layer B.Cu) (net 1))
   (via (at 61.75 128.5) (size 0.6) (drill 0.4) (layers F.Cu B.Cu) (net 1))
@@
   (segment (start 28.5 117) (end 45.5 100) (width 0.508) (layer F.Cu) (net 80))
   (segment (start 45.5 100) (end 60 100) (width 0.508) (layer F.Cu) (net 80))
-  (segment (start 76.74 98.26) (end 76.74 97.88) (width 0.508) (layer F.Cu) (net 80))
   (segment (start 37.5 126) (end 36.499908 126) (width 0.508) (layer B.Cu) (net 80))
   (via (at 36.499908 126) (size 0.6) (drill 0.4) (layers F.Cu B.Cu) (net 80))
   (segment (start 37.5 128.5) (end 37.5 126) (width 0.508) (layer B.Cu) (net 80))
-  (segment (start 90.04 54.72) (end 90.04 55.12) (width 0.508) (layer F.Cu) (net 80))
   (segment (start 27.5 72.4) (end 27.5 87.6) (width 0.508) (layer F.Cu) (net 210))
   (segment (start 29.2 87.6) (end 29.2 72.4) (width 0.508) (layer F.Cu) (net 211))

Commit message: boop
Parts:
- moved C501 28.2 mm to (280.8, 110.0)
Routing:
- net +5V: track 176.0 -> 1846.7 mm, vias 6 -> 26
- net /Mux/HD28: track 0.00 -> 102.8 mm
- net /Mux/HD27: track 0.00 -> 95.2 mm
- net /Mux/M21: track 0.00 -> 91.7 mm, vias 0 -> 2
- net /Mux/HD26: track 0.00 -> 86.4 mm
- net /Mux/M1: track 108.0 -> 183.7 mm, vias 0 -> 1
- net /Mux/HD25: track 0.00 -> 74.9 mm
- net /Mux/M2: track 104.6 -> 177.1 mm, vias 1 -> 2
- net /Mux/M3: track 103.6 -> 164.9 mm
- net /Capacitors/HA23: track 0.00 -> 57.9 mm
- net /Capacitors/HA33: track 0.00 -> 47.3 mm
- net /Capacitors/HA13: track 0.00 -> 45.6 mm
- net /Mux/M11: track 0.00 -> 44.7 mm
- net /Mux/HD24: track 0.00 -> 44.3 mm
- net /Capacitors/HA32: track 0.00 -> 41.8 mm
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