File: Projects/Voicemeeter/test.kicad_pcb (KiCad board)
At the start: 2 copper layers, 310 x 190 mm, 12 parts, among them J501 SPARE, J502 GS2, J504 GS2, J505 MIDI OUT, J506 MIDI IN, U502 PC817

Commit message: vada
Routing:
- net +5V: track 1846.7 -> 2079.9 mm
- net /LEDs/SK2: track 0.00 -> 57.7 mm
- net /LEDs/SK1: track 0.00 -> 54.2 mm
- net /Capacitors/HA31: track 0.00 -> 47.1 mm, vias 0 -> 2
- net /Capacitors/HA21: track 0.00 -> 33.3 mm, vias 0 -> 2
- net Net-(LED81-Pad6): track 0.00 -> 25.2 mm
- net Net-(LED81-Pad5): track 0.00 -> 25.2 mm
- net GND: track 43.5 -> 48.2 mm, vias 2 -> 3

Commit message: starting to get bored
Parts:
- added RV210: POT, MATHSTERK:slidepot, F.Cu at (123.8, 163.5)
- added U403: 74HC4051, Housings_DIP:DIP-16_W7.62mm_LongPads, B.Cu at (136.4, 32.6)
Routing:
- net /Mux/M2: track 177.1 -> 393.3 mm, vias 2 -> 4
- net /Mux/M3: track 164.9 -> 380.7 mm, vias 0 -> 2
- net /Mux/M1: track 183.7 -> 388.3 mm, vias 1 -> 2
- net /Capacitors/DA11: track 0.00 -> 149.6 mm, vias 0 -> 5
- net /Capacitors/DA21: track 0.00 -> 119.0 mm, vias 0 -> 4
- net /Mux/HD38: track 0.00 -> 101.9 mm
- net /Mux/DD28: track 0.00 -> 101.3 mm
- net /Mux/DD18: track 0.00 -> 99.6 mm
- net /Mux/HD37: track 0.00 -> 94.3 mm
- net /Mux/DD27: track 0.00 -> 92.7 mm
- net /Mux/DD17: track 0.00 -> 92.0 mm
- net /Mux/HD36: track 0.00 -> 85.8 mm
- net /Mux/DD26: track 0.00 -> 84.2 mm
- net /Mux/DD16: track 0.00 -> 83.5 mm
- net /Mux/OD53: track 0.00 -> 78.8 mm
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
Commit message: asd
Parts:
- moved R502 36.0 mm to (66.0, 25.9), turned to 90 degrees
- moved R503 34.6 mm to (68.6, 25.9), turned to 90 degrees
Routing:
- net +5V: track 2102.8 -> 0.00 mm, vias 31 -> 0
- net /Mux/M2: track 393.3 -> 0.00 mm, vias 4 -> 0
- net /Mux/M1: track 388.3 -> 0.00 mm, vias 2 -> 0
- net /Mux/M3: track 380.7 -> 0.00 mm, vias 2 -> 0
- net /Capacitors/DA11: track 149.6 -> 0.00 mm, vias 5 -> 0
- net Net-(LED12-Pad5): track 134.2 -> 0.00 mm
- net Net-(LED12-Pad6): track 131.7 -> 0.00 mm
- net /Capacitors/DA21: track 119.0 -> 0.00 mm, vias 4 -> 0
- net /Mux/HD18: track 105.1 -> 0.00 mm
- net /Mux/HD28: track 102.8 -> 0.00 mm
- net /Mux/HD38: track 101.9 -> 0.00 mm
- net /Mux/DD28: track 101.3 -> 0.00 mm
- net /Mux/DD18: track 99.6 -> 0.00 mm
- net /Mux/HD17: track 97.5 -> 0.00 mm
- net /Mux/HD27: track 95.2 -> 0.00 mm
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- removed copper zone on B.Cu, net +3V3
- removed copper zone on F.Cu, net GND
Other:
- board outline removed

Commit message: before it's too late
Parts:
- moved U403 45.3 mm to (94.8, 50.6)
- moved J502 39.9 mm to (68.6, 54.0), turned to 180 degrees
Connections:
- U403 pad 1: /Capacitors/DA22 -> /Capacitors/DA24
- U403 pad 15: /Capacitors/DA13 -> /Capacitors/DA22
- U403 pad 2: /Capacitors/DA24 -> /Capacitors/DA23
- U403 pad 5: /Capacitors/DA23 -> /Capacitors/DA13
